File: hdw/AC_Power_Meter/USB_UART_Isolation.sch (KiCad schematic (older format))
At the start: 0 parts

Commit message: Populated USB circuit pages
Parts:
- added C? (x2): 0.1uF, symbol Custom_Library:C_Custom
- added R? (x4): 10k, symbol Custom_Library:R_Custom
- added U?: ISO7321C, Package_SO:SOIC-8_3.9x4.9mm_P1.27mm, symbol Isolator:ISO7321C
Connections:
- net labels added: +3.3V, +5V_USB, GND, GND_USB, USB_UART_RX, USB_UART_RX_ISO, USB_UART_TX, USB_UART_TX_ISO
- wire segments 0 -> 20
Other:
- note added: "USB UART Isolation"

Commit message: Added MU logo and titles to all sheets
Changed lines of the file:
@@
 Text GLabel 7730 3720 2    60   Input ~ 0
 USB_UART_RX_ISO
-Text Notes 4610 1130 0    100  ~ 20
+Text Notes 540  690  0    100  ~ 20
 USB UART Isolation
 $Comp
@@
 	1    0    0    -1
 $EndComp
+$Comp
+L Mu_Logo:LOGO #G?
+U 1 1 5BBF6DB0
+P 9900 1000
+F 0 "#G?" H 9900 670 60  0001 C CNN
+F 1 "LOGO" H 9900 1330 60  0001 C CNN
+F 2 "" H 9900 1000 50  0001 C CNN
+F 3 "" H 9900 1000 50  0001 C CNN
+	1    9900 1000
+	1    0    0    -1
+$EndComp

Commit message: Updated MU logo to crisper image
Changed lines of the file:
@@
 $EndComp
 $Comp
-L Mu_Logo:LOGO #G?
-U 1 1 5BBF6DB0
-P 9900 1000
-F 0 "#G?" H 9900 670 60  0001 C CNN
-F 1 "LOGO" H 9900 1330 60  0001 C CNN
-F 2 "" H 9900 1000 50  0001 C CNN
-F 3 "" H 9900 1000 50  0001 C CNN
-	1    9900 1000
+L Custom_Library:MU_Logo #G?
+U 1 1 5BB69DAE
+P 9900 1100
+F 0 "#G?" H 9900 614 60  0001 C CNN
+F 1 "MU_Logo" H 9900 1586 60  0001 C CNN
+F 2 "" H 9900 1100 50  0001 C CNN
+F 3 "" H 9900 1100 50  0001 C CNN
+	1    9900 1100
 	1    0    0    -1
 $EndComp

Commit message: Added ORing circuit to TRIAC page
Parts:
- added C?: C_Custom, symbol Custom_Library:C_Custom
Changed lines of the file:
@@
 	1    0    0    -1
 $EndComp
+$Comp
+L Custom_Library:C_Custom C?
+U 1 1 5BB59130
+P 5330 4740
+F 0 "C?" H 5355 4840 50  0000 L CNN
+F 1 "C_Custom" H 5355 4640 50  0000 L CNN
+F 2 "" H 5368 4590 50  0001 C CNN
+F 3 "" H 5355 4840 50  0001 C CNN
+F 4 "Foot" H 5180 4840 50  0000 R CNN "display_footprint"
+F 5 "V" H 5180 4740 50  0000 R CNN "Voltage"
+F 6 "Er" H 5180 4640 50  0000 R CNN "Dielectric"
+F 7 "PN" H 5755 5240 60  0001 C CNN "Digi-Key PN"
+	1    5330 4740
+	0    1    1    0
+$EndComp
 $EndSCHEMATC

Commit message: Added series resistor in ZCD circuit
Parts:
- C?: value C_Custom -> 0.056uF; Dielectric Er -> X7R; Voltage V -> 250VAC; display_footprint Foot -> 2220
Connections:
- wire segments 20 -> 24
Changed lines of the file:
@@
 U 1 1 5BB59130
 P 5330 4740
-F 0 "C?" H 5355 4840 50  0000 L CNN
-F 1 "C_Custom" H 5355 4640 50  0000 L CNN
+F 0 "C?" V 5380 4830 50  0000 L CNN
+F 1 "0.056uF" V 5380 4650 50  0000 R CNN
 F 2 "" H 5368 4590 50  0001 C CNN
 F 3 "" H 5355 4840 50  0001 C CNN
-F 4 "Foot" H 5180 4840 50  0000 R CNN "display_footprint"
-F 5 "V" H 5180 4740 50  0000 R CNN "Voltage"
-F 6 "Er" H 5180 4640 50  0000 R CNN "Dielectric"
+F 4 "2220" V 5190 4740 50  0000 C CNN "display_footprint"
+F 5 "250VAC" V 5110 4740 50  0000 C CNN "Voltage"
+F 6 "X7R" V 5020 4740 50  0000 C CNN "Dielectric"
 F 7 "PN" H 5755 5240 60  0001 C CNN "Digi-Key PN"
 	1    5330 4740
 	0    1    1    0
 $EndComp
+$Comp
+L Custom_Library:GND_USB #PWR?
+U 1 1 5BB6AFF1
+P 5850 4820
+F 0 "#PWR?" H 5850 4570 50  0001 C CNN
+F 1 "GND_USB" H 5850 4670 50  0000 C CNN
+F 2 "" H 5850 4820 50  0001 C CNN
+F 3 "" H 5850 4820 50  0001 C CNN
+	1    5850 4820
+	1    0    0    -1
+$EndComp
+Wire Wire Line
+	5850 4820 5850 4740
+Wire Wire Line
+	5850 4740 5480 4740
+$Comp
+L power:GND #PWR?
+U 1 1 5BB6B260
+P 4810 4820
+F 0 "#PWR?" H 4810 4570 50  0001 C CNN
+F 1 "GND" H 4810 4670 50  0000 C CNN
+F 2 "" H 4810 4820 50  0001 C CNN
+F 3 "" H 4810 4820 50  0001 C CNN
+	1    4810 4820
+	1    0    0    -1
+$EndComp
+Wire Wire Line
+	4810 4820 4810 4740
+Wire Wire Line
+	4810 4740 5180 4740
 $EndSCHEMATC
