File: hdw/AC_Power_Meter/USB_UART_Isolation.sch (KiCad schematic (older format))
At the start: 8 parts

Commit message: Rewired a few micro symbols, add FMW notes
Parts:
- gave numbers to parts that had none: 8
Changed lines of the file:
@@
 $Descr A 11000 8500
 encoding utf-8
-Sheet 11 17
+Sheet 11 18
 Title ""
 Date ""
@@
 USB UART Isolation
 $Comp
-L Isolator:ISO7321C U?
+L Isolator:ISO7321C U1101
 U 1 1 5BB52339
 P 5330 3620
-F 0 "U?" H 5330 4045 50  0000 C CNN
+F 0 "U1101" H 5330 4045 50  0000 C CNN
 F 1 "ISO7321C" H 5330 3970 50  0000 C CNN
 F 2 "Package_SO:SOIC-8_3.9x4.9mm_P1.27mm" H 5330 3270 50  0001 C CIN
@@
 $EndComp
 $Comp
-L Custom_Library:GND_USB #PWR?
+L Custom_Library:GND_USB #PWR01109
 U 1 1 5BB5259F
 P 5850 4050
-F 0 "#PWR?" H 5850 3800 50  0001 C CNN
+F 0 "#PWR01109" H 5850 3800 50  0001 C CNN
 F 1 "GND_USB" H 5850 3900 50  0000 C CNN
 F 2 "" H 5850 4050 50  0001 C CNN
@@
 $EndComp
 $Comp
-L power:GND #PWR?
+L power:GND #PWR01106
 U 1 1 5BB525D8
 P 4810 4050
-F 0 "#PWR?" H 4810 3800 50  0001 C CNN
+F 0 "#PWR01106" H 4810 3800 50  0001 C CNN
 F 1 "GND" H 4810 3900 50  0000 C CNN
 F 2 "" H 4810 4050 50  0001 C CNN
@@
 	4810 3520 4810 4050
 $Comp
-L Custom_Library:+5V_USB #PWR?
+L Custom_Library:+5V_USB #PWR01108
 U 1 1 5BB52829
 P 5850 3340
-F 0 "#PWR?" H 5850 3190 50  0001 C CNN
+F 0 "#PWR01108" H 5850 3190 50  0001 C CNN
 F 1 "+5V_USB" H 5850 3480 50  0000 C CNN
 F 2 "" H 5850 3340 50  0001 C CNN
@@
 	5850 3420 5730 3420
 $Comp
-L Custom_Library:+3.3V #PWR?
+L Custom_Library:+3.3V #PWR01105
 U 1 1 5BB5288C
 P 4810 3340
-F 0 "#PWR?" H 4810 3190 50  0001 C CNN
+F 0 "#PWR01105" H 4810 3190 50  0001 C CNN
 F 1 "+3.3V" H 4810 3480 50  0000 C CNN
 F 2 "" H 4810 3340 50  0000 C CNN
@@
 P 6520 4130
 AR Path="/5BB27BA3/5BB52E7F" Ref="R?"  Part="1"
-AR Path="/5BB27BE1/5BB52E7F" Ref="R?"  Part="1"
-F 0 "R?" H 6440 4130 50  0000 R CNN
+AR Path="/5BB27BE1/5BB52E7F" Ref="R1103"  Part="1"
+F 0 "R1103" H 6440 4130 50  0000 R CNN
 F 1 "10k" V 6520 4130 50  0000 C CNN
 F 2 "" H 6520 4130 50  0001 C CNN
@@
 P 4440 2620
 AR Path="/5BB27BA3/5BB52E90" Ref="C?"  Part="1"
-AR Path="/5BB27BE1/5BB52E90" Ref="C?"  Part="1"
-F 0 "C?" H 4465 2720 50  0000 L CNN
+AR Path="/5BB27BE1/5BB52E90" Ref="C1101"  Part="1"
+F 0 "C1101" H 4465 2720 50  0000 L CNN
 F 1 "0.1uF" H 4465 2520 50  0000 L CNN
 F 2 "" H 4478 2470 50  0001 C CNN
@@
 P 7450 4120
 AR Path="/5BB27BA3/5BB52FEA" Ref="R?"  Part="1"
-AR Path="/5BB27BE1/5BB52FEA" Ref="R?"  Part="1"
-F 0 "R?" H 7370 4120 50  0000 R CNN
+AR Path="/5BB27BE1/5BB52FEA" Ref="R1104"  Part="1"
+F 0 "R1104" H 7370 4120 50  0000 R CNN
 F 1 "10k" V 7450 4120 50  0000 C CNN
 F 2 "" H 7450 4120 50  0001 C CNN
@@
 	7450 3720 5730 3720
 $Comp
-L Custom_Library:GND_USB #PWR?
+L Custom_Library:GND_USB #PWR01113
 U 1 1 5BB53209
 P 6520 4280
-F 0 "#PWR?" H 6520 4030 50  0001 C CNN
+F 0 "#PWR01113" H 6520 4030 50  0001 C CNN
 F 1 "GND_USB" H 6520 4130 50  0000 C CNN
 F 2 "" H 6520 4280 50  0001 C CNN
@@
 $EndComp
 $Comp
-L Custom_Library:GND_USB #PWR?
+L Custom_Library:GND_USB #PWR01114
 U 1 1 5BB53223
 P 7450 4270
-F 0 "#PWR?" H 7450 4020 50  0001 C CNN
+F 0 "#PWR01114" H 7450 4020 50  0001 C CNN
 F 1 "GND_USB" H 7450 4120 50  0000 C CNN
 F 2 "" H 7450 4270 50  0001 C CNN
@@
 P 4140 4130
 AR Path="/5BB27BA3/5BB5328E" Ref="R?"  Part="1"
-AR Path="/5BB27BE1/5BB5328E" Ref="R?"  Part="1"
-F 0 "R?" H 4060 4130 50  0000 R CNN
+AR Path="/5BB27BE1/5BB5328E" Ref="R1102"  Part="1"
+F 0 "R1102" H 4060 4130 50  0000 R CNN
 F 1 "10k" V 4140 4130 50  0000 C CNN
 F 2 "" H 4140 4130 50  0001 C CNN
@@
 P 3210 4120
 AR Path="/5BB27BA3/5BB53299" Ref="R?"  Part="1"
-AR Path="/5BB27BE1/5BB53299" Ref="R?"  Part="1"
-F 0 "R?" H 3130 4120 50  0000 R CNN
+AR Path="/5BB27BE1/5BB53299" Ref="R1101"  Part="1"
+F 0 "R1101" H 3130 4120 50  0000 R CNN
 F 1 "10k" V 3210 4120 50  0000 C CNN
 F 2 "" H 3210 4120 50  0001 C CNN
@@
 P 5910 2620
 AR Path="/5BB27BA3/5BB53B36" Ref="C?"  Part="1"
-AR Path="/5BB27BE1/5BB53B36" Ref="C?"  Part="1"
-F 0 "C?" H 5935 2720 50  0000 L CNN
+AR Path="/5BB27BE1/5BB53B36" Ref="C1103"  Part="1"
+F 0 "C1103" H 5935 2720 50  0000 L CNN
 F 1 "0.1uF" H 5935 2520 50  0000 L CNN
 F 2 "" H 5948 2470 50  0001 C CNN
@@
 $EndComp
 $Comp
-L Custom_Library:+3.3V #PWR?
+L Custom_Library:+3.3V #PWR01103
 U 1 1 5BB53B62
 P 4440 2470
-F 0 "#PWR?" H 4440 2320 50  0001 C CNN
+F 0 "#PWR01103" H 4440 2320 50  0001 C CNN
 F 1 "+3.3V" H 4440 2610 50  0000 C CNN
 F 2 "" H 4440 2470 50  0000 C CNN
@@
 $EndComp
 $Comp
-L Custom_Library:+5V_USB #PWR?
+L Custom_Library:+5V_USB #PWR01111
 U 1 1 5BB53B89
 P 5910 2470
-F 0 "#PWR?" H 5910 2320 50  0001 C CNN
+F 0 "#PWR01111" H 5910 2320 50  0001 C CNN
 F 1 "+5V_USB" H 5910 2610 50  0000 C CNN
 F 2 "" H 5910 2470 50  0001 C CNN
@@
 $EndComp
 $Comp
-L power:GND #PWR?
+L power:GND #PWR01104
 U 1 1 5BB53BA2
 P 4440 2770
-F 0 "#PWR?" H 4440 2520 50  0001 C CNN
+F 0 "#PWR01104" H 4440 2520 50  0001 C CNN
 F 1 "GND" H 4440 2620 50  0000 C CNN
 F 2 "" H 4440 2770 50  0001 C CNN
@@
 $EndComp
 $Comp
-L Custom_Library:GND_USB #PWR?
+L Custom_Library:GND_USB #PWR01112
 U 1 1 5BB53BBB
 P 5910 2770
-F 0 "#PWR?" H 5910 2520 50  0001 C CNN
+F 0 "#PWR01112" H 5910 2520 50  0001 C CNN
 F 1 "GND_USB" H 5910 2620 50  0000 C CNN
 F 2 "" H 5910 2770 50  0001 C CNN
@@
 $EndComp
 $Comp
-L power:GND #PWR?
+L power:GND #PWR01102
 U 1 1 5BB53BEB
 P 4140 4280
-F 0 "#PWR?" H 4140 4030 50  0001 C CNN
+F 0 "#PWR01102" H 4140 4030 50  0001 C CNN
 F 1 "GND" H 4140 4130 50  0000 C CNN
 F 2 "" H 4140 4280 50  0001 C CNN
@@
 $EndComp
 $Comp
-L power:GND #PWR?
+L power:GND #PWR01101
 U 1 1 5BB53C20
 P 3210 4270
-F 0 "#PWR?" H 3210 4020 50  0001 C CNN
+F 0 "#PWR01101" H 3210 4020 50  0001 C CNN
 F 1 "GND" H 3210 4120 50  0000 C CNN
 F 2 "" H 3210 4270 50  0001 C CNN
@@
 $EndComp
 $Comp
-L Custom_Library:MU_Logo #G?
+L Custom_Library:MU_Logo #G1101
 U 1 1 5BB69DAE
 P 9900 1100
-F 0 "#G?" H 9900 614 60  0001 C CNN
+F 0 "#G1101" H 9900 614 60  0001 C CNN
 F 1 "MU_Logo" H 9900 1586 60  0001 C CNN
 F 2 "" H 9900 1100 50  0001 C CNN
@@
 $EndComp
 $Comp
-L Custom_Library:C_Custom C?
+L Custom_Library:C_Custom C1102
 U 1 1 5BB59130
 P 5330 4740
-F 0 "C?" V 5380 4830 50  0000 L CNN
+F 0 "C1102" V 5380 4830 50  0000 L CNN
 F 1 "0.056uF" V 5380 4650 50  0000 R CNN
 F 2 "" H 5368 4590 50  0001 C CNN
@@
 $EndComp
 $Comp
-L Custom_Library:GND_USB #PWR?
+L Custom_Library:GND_USB #PWR01110
 U 1 1 5BB6AFF1
 P 5850 4820
-F 0 "#PWR?" H 5850 4570 50  0001 C CNN
+F 0 "#PWR01110" H 5850 4570 50  0001 C CNN
 F 1 "GND_USB" H 5850 4670 50  0000 C CNN
 F 2 "" H 5850 4820 50  0001 C CNN
@@
 	5850 4740 5480 4740
 $Comp
-L power:GND #PWR?
+L power:GND #PWR01107
 U 1 1 5BB6B260
 P 4810 4820
-F 0 "#PWR?" H 4810 4570 50  0001 C CNN
+F 0 "#PWR01107" H 4810 4570 50  0001 C CNN
 F 1 "GND" H 4810 4670 50  0000 C CNN
 F 2 "" H 4810 4820 50  0001 C CNN

Commit message: Updated most footprints
Parts:
- C1101, C1103: footprint (none) -> Capacitors_SMD:C_0603; Digi-Key PN PN -> 490-8020-1-ND
- C1102: footprint (none) -> Capacitors_SMD:C_2220; Digi-Key PN PN -> 490-7747-1-ND
- R1101, R1102, R1103, R1104: footprint (none) -> Resistors_SMD:R_0603; Digi-Key PN PN -> RHM10KADCT-ND
Changed lines of the file:
@@
 F 0 "R1103" H 6440 4130 50  0000 R CNN
 F 1 "10k" V 6520 4130 50  0000 C CNN
-F 2 "" H 6520 4130 50  0001 C CNN
+F 2 "Resistors_SMD:R_0603" H 6520 4130 50  0001 C CNN
 F 3 "" H 6520 4130 50  0001 C CNN
 F 4 "0603" H 6620 4210 50  0000 L CNN "display_footprint"
 F 5 "1%" H 6620 4130 50  0000 L CNN "Tolerance"
 F 6 "1/10W" H 6630 4050 50  0000 L CNN "Wattage"
-F 7 "PN" H 6820 4530 60  0001 C CNN "Digi-Key PN"
+F 7 "RHM10KADCT-ND" H 6820 4530 60  0001 C CNN "Digi-Key PN"
 	1    6520 4130
 	1    0    0    -1
@@
 F 0 "C1101" H 4465 2720 50  0000 L CNN
 F 1 "0.1uF" H 4465 2520 50  0000 L CNN
-F 2 "" H 4478 2470 50  0001 C CNN
+F 2 "Capacitors_SMD:C_0603" H 4478 2470 50  0001 C CNN
 F 3 "" H 4465 2720 50  0001 C CNN
 F 4 "0603" H 4290 2720 50  0000 R CNN "display_footprint"
 F 5 "50V" H 4290 2620 50  0000 R CNN "Voltage"
 F 6 "X7R" H 4290 2520 50  0000 R CNN "Dielectric"
-F 7 "PN" H 4865 3120 60  0001 C CNN "Digi-Key PN"
+F 7 "490-8020-1-ND" H 4865 3120 60  0001 C CNN "Digi-Key PN"
 	1    4440 2620
 	-1   0    0    -1
@@
 F 0 "R1104" H 7370 4120 50  0000 R CNN
 F 1 "10k" V 7450 4120 50  0000 C CNN
-F 2 "" H 7450 4120 50  0001 C CNN
+F 2 "Resistors_SMD:R_0603" H 7450 4120 50  0001 C CNN
 F 3 "" H 7450 4120 50  0001 C CNN
 F 4 "0603" H 7550 4200 50  0000 L CNN "display_footprint"
 F 5 "1%" H 7550 4120 50  0000 L CNN "Tolerance"
 F 6 "1/10W" H 7560 4040 50  0000 L CNN "Wattage"
-F 7 "PN" H 7750 4520 60  0001 C CNN "Digi-Key PN"
+F 7 "RHM10KADCT-ND" H 7750 4520 60  0001 C CNN "Digi-Key PN"
 	1    7450 4120
 	1    0    0    -1
@@
 F 0 "R1102" H 4060 4130 50  0000 R CNN
 F 1 "10k" V 4140 4130 50  0000 C CNN
-F 2 "" H 4140 4130 50  0001 C CNN
+F 2 "Resistors_SMD:R_0603" H 4140 4130 50  0001 C CNN
 F 3 "" H 4140 4130 50  0001 C CNN
 F 4 "0603" H 4240 4210 50  0000 L CNN "display_footprint"
 F 5 "1%" H 4240 4130 50  0000 L CNN "Tolerance"
 F 6 "1/10W" H 4250 4050 50  0000 L CNN "Wattage"
-F 7 "PN" H 4440 4530 60  0001 C CNN "Digi-Key PN"
+F 7 "RHM10KADCT-ND" H 4440 4530 60  0001 C CNN "Digi-Key PN"
 	1    4140 4130
 	-1   0    0    -1
@@
 F 0 "R1101" H 3130 4120 50  0000 R CNN
 F 1 "10k" V 3210 4120 50  0000 C CNN
-F 2 "" H 3210 4120 50  0001 C CNN
+F 2 "Resistors_SMD:R_0603" H 3210 4120 50  0001 C CNN
 F 3 "" H 3210 4120 50  0001 C CNN
 F 4 "0603" H 3310 4200 50  0000 L CNN "display_footprint"
 F 5 "1%" H 3310 4120 50  0000 L CNN "Tolerance"
 F 6 "1/10W" H 3320 4040 50  0000 L CNN "Wattage"
-F 7 "PN" H 3510 4520 60  0001 C CNN "Digi-Key PN"
+F 7 "RHM10KADCT-ND" H 3510 4520 60  0001 C CNN "Digi-Key PN"
 	1    3210 4120
 	-1   0    0    -1
@@
 F 0 "C1103" H 5935 2720 50  0000 L CNN
 F 1 "0.1uF" H 5935 2520 50  0000 L CNN
-F 2 "" H 5948 2470 50  0001 C CNN
+F 2 "Capacitors_SMD:C_0603" H 5948 2470 50  0001 C CNN
 F 3 "" H 5935 2720 50  0001 C CNN
 F 4 "0603" H 5760 2720 50  0000 R CNN "display_footprint"
 F 5 "50V" H 5760 2620 50  0000 R CNN "Voltage"
 F 6 "X7R" H 5760 2520 50  0000 R CNN "Dielectric"
-F 7 "PN" H 6335 3120 60  0001 C CNN "Digi-Key PN"
+F 7 "490-8020-1-ND" H 6335 3120 60  0001 C CNN "Digi-Key PN"
 	1    5910 2620
 	-1   0    0    -1
@@
 F 0 "C1102" V 5380 4830 50  0000 L CNN
 F 1 "0.056uF" V 5380 4650 50  0000 R CNN
-F 2 "" H 5368 4590 50  0001 C CNN
+F 2 "Capacitors_SMD:C_2220" H 5368 4590 50  0001 C CNN
 F 3 "" H 5355 4840 50  0001 C CNN
 F 4 "2220" V 5190 4740 50  0000 C CNN "display_footprint"
 F 5 "250VAC" V 5110 4740 50  0000 C CNN "Voltage"
 F 6 "X7R" V 5020 4740 50  0000 C CNN "Dielectric"
-F 7 "PN" H 5755 5240 60  0001 C CNN "Digi-Key PN"
+F 7 "490-7747-1-ND" H 5755 5240 60  0001 C CNN "Digi-Key PN"
 	1    5330 4740
 	0    1    1    0

Commit message: Arranged a few pages of components
Parts:
- U1101: footprint Package_SO:SOIC-8_3.9x4.9mm_P1.27mm -> Housings_SOIC:SOIC-8_3.9x4.9mm_Pitch1.27mm
Changed lines of the file:
@@
 F 0 "U1101" H 5330 4045 50  0000 C CNN
 F 1 "ISO7321C" H 5330 3970 50  0000 C CNN
-F 2 "Package_SO:SOIC-8_3.9x4.9mm_P1.27mm" H 5330 3270 50  0001 C CIN
+F 2 "Housings_SOIC:SOIC-8_3.9x4.9mm_Pitch1.27mm" H 5330 3270 50  0001 C CIN
 F 3 "http://www.ti.com/general/docs/lit/getliterature.tsp?genericPartNumber=iso7321c&fileType=pdf" H 5330 3620 50  0001 C CNN
 F 4 "296-42102-1-ND" H 5330 3620 50  0001 C CNN "Digi-Key PN"

Commit message: Routed much more of the board, design rule fixes
Changed lines of the file:
@@
 L Custom_Library:R_Custom R?
 U 1 1 5BB52E7F
-P 6520 4130
+P 6520 3440
 AR Path="/5BB27BA3/5BB52E7F" Ref="R?"  Part="1"
 AR Path="/5BB27BE1/5BB52E7F" Ref="R1103"  Part="1"
-F 0 "R1103" H 6440 4130 50  0000 R CNN
-F 1 "10k" V 6520 4130 50  0000 C CNN
-F 2 "Resistors_SMD:R_0603" H 6520 4130 50  0001 C CNN
-F 3 "" H 6520 4130 50  0001 C CNN
-F 4 "0603" H 6620 4210 50  0000 L CNN "display_footprint"
-F 5 "1%" H 6620 4130 50  0000 L CNN "Tolerance"
-F 6 "1/10W" H 6630 4050 50  0000 L CNN "Wattage"
-F 7 "RHM10KADCT-ND" H 6820 4530 60  0001 C CNN "Digi-Key PN"
-	1    6520 4130
-	1    0    0    -1
+F 0 "R1103" H 6440 3440 50  0000 R CNN
+F 1 "10k" V 6520 3440 50  0000 C CNN
+F 2 "Resistors_SMD:R_0603" H 6520 3440 50  0001 C CNN
+F 3 "" H 6520 3440 50  0001 C CNN
+F 4 "0603" H 6620 3520 50  0000 L CNN "display_footprint"
+F 5 "1%" H 6620 3440 50  0000 L CNN "Tolerance"
+F 6 "1/10W" H 6630 3360 50  0000 L CNN "Wattage"
+F 7 "RHM10KADCT-ND" H 6820 3840 60  0001 C CNN "Digi-Key PN"
+	1    6520 3440
+	1    0    0    1
 $EndComp
 $Comp
@@
 L Custom_Library:R_Custom R?
 U 1 1 5BB52FEA
-P 7450 4120
+P 7450 3430
 AR Path="/5BB27BA3/5BB52FEA" Ref="R?"  Part="1"
 AR Path="/5BB27BE1/5BB52FEA" Ref="R1104"  Part="1"
-F 0 "R1104" H 7370 4120 50  0000 R CNN
-F 1 "10k" V 7450 4120 50  0000 C CNN
-F 2 "Resistors_SMD:R_0603" H 7450 4120 50  0001 C CNN
-F 3 "" H 7450 4120 50  0001 C CNN
-F 4 "0603" H 7550 4200 50  0000 L CNN "display_footprint"
-F 5 "1%" H 7550 4120 50  0000 L CNN "Tolerance"
-F 6 "1/10W" H 7560 4040 50  0000 L CNN "Wattage"
-F 7 "RHM10KADCT-ND" H 7750 4520 60  0001 C CNN "Digi-Key PN"
-	1    7450 4120
-	1    0    0    -1
-$EndComp
-Wire Wire Line
-	7730 3720 7450 3720
-Wire Wire Line
-	7730 3820 6520 3820
-Wire Wire Line
-	6520 3980 6520 3820
-Connection ~ 6520 3820
-Wire Wire Line
-	6520 3820 5730 3820
-Wire Wire Line
-	7450 3970 7450 3720
-Connection ~ 7450 3720
-Wire Wire Line
-	7450 3720 5730 3720
-$Comp
-L Custom_Library:GND_USB #PWR01113
-U 1 1 5BB53209
-P 6520 4280
-F 0 "#PWR01113" H 6520 4030 50  0001 C CNN
-F 1 "GND_USB" H 6520 4130 50  0000 C CNN
-F 2 "" H 6520 4280 50  0001 C CNN
-F 3 "" H 6520 4280 50  0001 C CNN
-	1    6520 4280
-	1    0    0    -1
-$EndComp
-$Comp
-L Custom_Library:GND_USB #PWR01114
-U 1 1 5BB53223
-P 7450 4270
-F 0 "#PWR01114" H 7450 4020 50  0001 C CNN
-F 1 "GND_USB" H 7450 4120 50  0000 C CNN
-F 2 "" H 7450 4270 50  0001 C CNN
-F 3 "" H 7450 4270 50  0001 C CNN
-	1    7450 4270
-	1    0    0    -1
+F 0 "R1104" H 7370 3430 50  0000 R CNN
+F 1 "10k" V 7450 3430 50  0000 C CNN
+F 2 "Resistors_SMD:R_0603" H 7450 3430 50  0001 C CNN
+F 3 "" H 7450 3430 50  0001 C CNN
+F 4 "0603" H 7550 3510 50  0000 L CNN "display_footprint"
+F 5 "1%" H 7550 3430 50  0000 L CNN "Tolerance"
+F 6 "1/10W" H 7560 3350 50  0000 L CNN "Wattage"
+F 7 "RHM10KADCT-ND" H 7750 3830 60  0001 C CNN "Digi-Key PN"
+	1    7450 3430
+	1    0    0    1
 $EndComp
 Text GLabel 2930 3820 0    60   Input ~ 0
@@
 L Custom_Library:R_Custom R?
 U 1 1 5BB5328E
-P 4140 4130
+P 4140 3440
 AR Path="/5BB27BA3/5BB5328E" Ref="R?"  Part="1"
 AR Path="/5BB27BE1/5BB5328E" Ref="R1102"  Part="1"
-F 0 "R1102" H 4060 4130 50  0000 R CNN
-F 1 "10k" V 4140 4130 50  0000 C CNN
-F 2 "Resistors_SMD:R_0603" H 4140 4130 50  0001 C CNN
-F 3 "" H 4140 4130 50  0001 C CNN
-F 4 "0603" H 4240 4210 50  0000 L CNN "display_footprint"
-F 5 "1%" H 4240 4130 50  0000 L CNN "Tolerance"
-F 6 "1/10W" H 4250 4050 50  0000 L CNN "Wattage"
-F 7 "RHM10KADCT-ND" H 4440 4530 60  0001 C CNN "Digi-Key PN"
-	1    4140 4130
-	-1   0    0    -1
+F 0 "R1102" H 4060 3440 50  0000 R CNN
+F 1 "10k" V 4140 3440 50  0000 C CNN
+F 2 "Resistors_SMD:R_0603" H 4140 3440 50  0001 C CNN
+F 3 "" H 4140 3440 50  0001 C CNN
+F 4 "0603" H 4240 3520 50  0000 L CNN "display_footprint"
+F 5 "1%" H 4240 3440 50  0000 L CNN "Tolerance"
+F 6 "1/10W" H 4250 3360 50  0000 L CNN "Wattage"
+F 7 "RHM10KADCT-ND" H 4440 3840 60  0001 C CNN "Digi-Key PN"
+	1    4140 3440
+	-1   0    0    1
 $EndComp
 $Comp
 L Custom_Library:R_Custom R?
 U 1 1 5BB53299
-P 3210 4120
+P 3210 3430
 AR Path="/5BB27BA3/5BB53299" Ref="R?"  Part="1"
 AR Path="/5BB27BE1/5BB53299" Ref="R1101"  Part="1"
-F 0 "R1101" H 3130 4120 50  0000 R CNN
-F 1 "10k" V 3210 4120 50  0000 C CNN
-F 2 "Resistors_SMD:R_0603" H 3210 4120 50  0001 C CNN
-F 3 "" H 3210 4120 50  0001 C CNN
-F 4 "0603" H 3310 4200 50  0000 L CNN "display_footprint"
-F 5 "1%" H 3310 4120 50  0000 L CNN "Tolerance"
-F 6 "1/10W" H 3320 4040 50  0000 L CNN "Wattage"
-F 7 "RHM10KADCT-ND" H 3510 4520 60  0001 C CNN "Digi-Key PN"
-	1    3210 4120
-	-1   0    0    -1
-$EndComp
-Wire Wire Line
-	2930 3720 3210 3720
-Wire Wire Line
-	2930 3820 4140 3820
-Wire Wire Line
-	4140 3980 4140 3820
-Connection ~ 4140 3820
-Wire Wire Line
-	4140 3820 4930 3820
-Wire Wire Line
-	3210 3970 3210 3720
-Connection ~ 3210 3720
-Wire Wire Line
-	3210 3720 4930 3720
+F 0 "R1101" H 3130 3430 50  0000 R CNN
+F 1 "10k" V 3210 3430 50  0000 C CNN
+F 2 "Resistors_SMD:R_0603" H 3210 3430 50  0001 C CNN
+F 3 "" H 3210 3430 50  0001 C CNN
+F 4 "0603" H 3310 3510 50  0000 L CNN "display_footprint"
+F 5 "1%" H 3310 3430 50  0000 L CNN "Tolerance"
+F 6 "1/10W" H 3320 3350 50  0000 L CNN "Wattage"
+F 7 "RHM10KADCT-ND" H 3510 3830 60  0001 C CNN "Digi-Key PN"
+	1    3210 3430
+	-1   0    0    1
+$EndComp
 $Comp
 L Custom_Library:C_Custom C?
@@
 $EndComp
 $Comp
-L power:GND #PWR01102
-U 1 1 5BB53BEB
-P 4140 4280
-F 0 "#PWR01102" H 4140 4030 50  0001 C CNN
-F 1 "GND" H 4140 4130 50  0000 C CNN
-F 2 "" H 4140 4280 50  0001 C CNN
-F 3 "" H 4140 4280 50  0001 C CNN
-	1    4140 4280
-	1    0    0    -1
-$EndComp
-$Comp
-L power:GND #PWR01101
-U 1 1 5BB53C20
-P 3210 4270
-F 0 "#PWR01101" H 3210 4020 50  0001 C CNN
-F 1 "GND" H 3210 4120 50  0000 C CNN
-F 2 "" H 3210 4270 50  0001 C CNN
-F 3 "" H 3210 4270 50  0001 C CNN
-	1    3210 4270
-	1    0    0    -1
-$EndComp
-$Comp
 L Custom_Library:MU_Logo #G1101
 U 1 1 5BB69DAE
@@
 Wire Wire Line
 	4810 4740 5180 4740
+Wire Wire Line
+	5730 3720 7450 3720
+Wire Wire Line
+	5730 3820 6520 3820
+Wire Wire Line
+	2930 3720 3210 3720
+Wire Wire Line
+	2930 3820 4140 3820
+Wire Wire Line
+	3210 3580 3210 3720
+Connection ~ 3210 3720
+Wire Wire Line
+	3210 3720 4930 3720
+Wire Wire Line
+	4140 3590 4140 3820
+Connection ~ 4140 3820
+Wire Wire Line
+	4140 3820 4930 3820
+Wire Wire Line
+	6520 3590 6520 3820
+Connection ~ 6520 3820
+Wire Wire Line
+	6520 3820 7730 3820
+Wire Wire Line
+	7450 3580 7450 3720
+Connection ~ 7450 3720
+Wire Wire Line
+	7450 3720 7730 3720
+$Comp
+L Custom_Library:+3.3V #PWR0101
+U 1 1 5BBABC36
+P 4140 3290
+F 0 "#PWR0101" H 4140 3140 50  0001 C CNN
+F 1 "+3.3V" H 4140 3430 50  0000 C CNN
+F 2 "" H 4140 3290 50  0000 C CNN
+F 3 "" H 4140 3290 50  0000 C CNN
+	1    4140 3290
+	1    0    0    -1
+$EndComp
+$Comp
+L Custom_Library:+3.3V #PWR0102
+U 1 1 5BBABC58
+P 3210 3280
+F 0 "#PWR0102" H 3210 3130 50  0001 C CNN
+F 1 "+3.3V" H 3210 3420 50  0000 C CNN
+F 2 "" H 3210 3280 50  0000 C CNN
+F 3 "" H 3210 3280 50  0000 C CNN
+	1    3210 3280
+	1    0    0    -1
+$EndComp
+$Comp
+L Custom_Library:+5V_USB #PWR0103
+U 1 1 5BBABCD5
+P 7450 3280
+F 0 "#PWR0103" H 7450 3130 50  0001 C CNN
+F 1 "+5V_USB" H 7450 3420 50  0000 C CNN
+F 2 "" H 7450 3280 50  0001 C CNN
+F 3 "" H 7450 3280 50  0001 C CNN
+	1    7450 3280
+	1    0    0    -1
+$EndComp
+$Comp
+L Custom_Library:+5V_USB #PWR0104
+U 1 1 5BBABCF7
+P 6520 3290
+F 0 "#PWR0104" H 6520 3140 50  0001 C CNN
+F 1 "+5V_USB" H 6520 3430 50  0000 C CNN
+F 2 "" H 6520 3290 50  0001 C CNN
+F 3 "" H 6520 3290 50  0001 C CNN
+	1    6520 3290
+	1    0    0    -1
+$EndComp
 $EndSCHEMATC

Commit message: Serious BOM scrubbing to drive price down
Parts:
- removed C1102: 0.056uF, Capacitors_SMD:C_2220, symbol Custom_Library:C_Custom
Connections:
- wire segments 24 -> 20
Changed lines of the file:
@@
 $Descr A 11000 8500
 encoding utf-8
-Sheet 11 18
+Sheet 11 17
 Title ""
 Date ""
@@
 	1    0    0    -1
 $EndComp
-$Comp
-L Custom_Library:C_Custom C1102
-U 1 1 5BB59130
-P 5330 4740
-F 0 "C1102" V 5380 4830 50  0000 L CNN
-F 1 "0.056uF" V 5380 4650 50  0000 R CNN
-F 2 "Capacitors_SMD:C_2220" H 5368 4590 50  0001 C CNN
-F 3 "" H 5355 4840 50  0001 C CNN
-F 4 "2220" V 5190 4740 50  0000 C CNN "display_footprint"
-F 5 "250VAC" V 5110 4740 50  0000 C CNN "Voltage"
-F 6 "X7R" V 5020 4740 50  0000 C CNN "Dielectric"
-F 7 "490-7747-1-ND" H 5755 5240 60  0001 C CNN "Digi-Key PN"
-	1    5330 4740
-	0    1    1    0
-$EndComp
-$Comp
-L Custom_Library:GND_USB #PWR01110
-U 1 1 5BB6AFF1
-P 5850 4820
-F 0 "#PWR01110" H 5850 4570 50  0001 C CNN
-F 1 "GND_USB" H 5850 4670 50  0000 C CNN
-F 2 "" H 5850 4820 50  0001 C CNN
-F 3 "" H 5850 4820 50  0001 C CNN
-	1    5850 4820
-	1    0    0    -1
-$EndComp
-Wire Wire Line
-	5850 4820 5850 4740
-Wire Wire Line
-	5850 4740 5480 4740
-$Comp
-L power:GND #PWR01107
-U 1 1 5BB6B260
-P 4810 4820
-F 0 "#PWR01107" H 4810 4570 50  0001 C CNN
-F 1 "GND" H 4810 4670 50  0000 C CNN
-F 2 "" H 4810 4820 50  0001 C CNN
-F 3 "" H 4810 4820 50  0001 C CNN
-	1    4810 4820
-	1    0    0    -1
-$EndComp
-Wire Wire Line
-	4810 4820 4810 4740
-Wire Wire Line
-	4810 4740 5180 4740
 Wire Wire Line
 	5730 3720 7450 3720
