File: hdw/AC_Power_Meter/AC_Current_Sensor.sch (KiCad schematic (older format))
At the start: 12 parts

Commit message: Added TRIAC circuit and POS12 AC/DC converter
Connections:
- net labels added: HT
- net labels removed: ISNS_HT_IN
- wire segments 34 -> 36
Changed lines of the file:
@@
 	1    0    0    -1
 $EndComp
-Text GLabel 3340 3410 0    50   Input ~ 0
-ISNS_HT_IN
 Text GLabel 3340 3710 0    50   Output ~ 0
 ISNS_HT_OUT
@@
 	7320 3510 7240 3510
 Connection ~ 7240 3510
+$Comp
+L power:HT #PWR?
+U 1 1 5BB463D5
+P 3260 3330
+F 0 "#PWR?" H 3260 3450 50  0001 C CNN
+F 1 "HT" H 3260 3420 50  0000 C CNN
+F 2 "" H 3260 3330 50  0001 C CNN
+F 3 "" H 3260 3330 50  0001 C CNN
+	1    3260 3330
+	1    0    0    -1
+$EndComp
+Wire Wire Line
+	3260 3330 3260 3410
+Wire Wire Line
+	3260 3410 3340 3410
 $EndSCHEMATC

Commit message: Added MU logo and titles to all sheets
Other:
- note added: "AC Current Sensor, Signal Buffer"
Changed lines of the file:
@@
 Wire Wire Line
 	3260 3410 3340 3410
+Text Notes 540  690  0    100  ~ 20
+AC Current Sensor, Signal Buffer
+$Comp
+L Mu_Logo:LOGO #G?
+U 1 1 5BBF1375
+P 9900 1000
+F 0 "#G?" H 9900 670 60  0001 C CNN
+F 1 "LOGO" H 9900 1330 60  0001 C CNN
+F 2 "" H 9900 1000 50  0001 C CNN
+F 3 "" H 9900 1000 50  0001 C CNN
+	1    9900 1000
+	1    0    0    -1
+$EndComp
 $EndSCHEMATC

Commit message: Updated MU logo to crisper image
Changed lines of the file:
@@
 AC Current Sensor, Signal Buffer
 $Comp
-L Mu_Logo:LOGO #G?
-U 1 1 5BBF1375
-P 9900 1000
-F 0 "#G?" H 9900 670 60  0001 C CNN
-F 1 "LOGO" H 9900 1330 60  0001 C CNN
-F 2 "" H 9900 1000 50  0001 C CNN
-F 3 "" H 9900 1000 50  0001 C CNN
-	1    9900 1000
+L Custom_Library:MU_Logo #G?
+U 1 1 5BB6B7BB
+P 9900 1100
+F 0 "#G?" H 9900 614 60  0001 C CNN
+F 1 "MU_Logo" H 9900 1586 60  0001 C CNN
+F 2 "" H 9900 1100 50  0001 C CNN
+F 3 "" H 9900 1100 50  0001 C CNN
+	1    9900 1100
 	1    0    0    -1
 $EndComp

Commit message: Revised signal conditioning, cleaned up a lot of pages
Parts:
- removed C?: 0.1uF, symbol Custom_Library:C_Custom
- removed C?: 10nF, symbol Custom_Library:C_Custom
- removed C?: 1nF, symbol Custom_Library:C_Custom
- removed C?: 10uF, symbol Custom_Library:C_Custom
- removed C?: 1uF, symbol Custom_Library:C_Custom
- removed U?: LTC6240IS5, Package_TO_SOT_SMD:SOT-23-5, symbol Custom_Library:LTC6240IS5
Connections:
- wire segments 36 -> 17
Other:
- note added: "10.7ARMS Max to support full output swing of conditioning stages"
- note added: "AC Current Sensor"
- note removed: "15A Max to support full output swing of conditioning stage"
- note removed: "AC Current Sensor, Signal Buffer"
- moved on the sheet: U?

Commit message: Rewired a few micro symbols, add FMW notes
Parts:
- gave numbers to parts that had none: 6
Changed lines of the file:
@@
 $Descr A 11000 8500
 encoding utf-8
-Sheet 3 17
+Sheet 3 18
 Title ""
 Date "2018-10-01"
@@
 AR Path="/5BB27BA3/5BB2A066" Ref="C?"  Part="1"
 AR Path="/5BB27B84/5BB2A066" Ref="C?"  Part="1"
-AR Path="/5BB27B24/5BB2A066" Ref="C?"  Part="1"
-F 0 "C?" H 4995 5170 50  0000 L CNN
+AR Path="/5BB27B24/5BB2A066" Ref="C301"  Part="1"
+F 0 "C301" H 4995 5170 50  0000 L CNN
 F 1 "0.1uF" H 4995 4970 50  0000 L CNN
 F 2 "" H 5008 4920 50  0001 C CNN
@@
 AR Path="/5BB27BA3/5BB2A071" Ref="C?"  Part="1"
 AR Path="/5BB27B84/5BB2A071" Ref="C?"  Part="1"
-AR Path="/5BB27B24/5BB2A071" Ref="C?"  Part="1"
-F 0 "C?" H 5345 5170 50  0000 L CNN
+AR Path="/5BB27B24/5BB2A071" Ref="C302"  Part="1"
+F 0 "C302" H 5345 5170 50  0000 L CNN
 F 1 "10nF" H 5345 4970 50  0000 L CNN
 F 2 "" H 5358 4920 50  0001 C CNN
@@
 AR Path="/5BB27BA3/5BB2A07C" Ref="C?"  Part="1"
 AR Path="/5BB27B84/5BB2A07C" Ref="C?"  Part="1"
-AR Path="/5BB27B24/5BB2A07C" Ref="C?"  Part="1"
-F 0 "C?" H 5695 5170 50  0000 L CNN
+AR Path="/5BB27B24/5BB2A07C" Ref="C303"  Part="1"
+F 0 "C303" H 5695 5170 50  0000 L CNN
 F 1 "1nF" H 5695 4970 50  0000 L CNN
 F 2 "" H 5708 4920 50  0001 C CNN
@@
 P 5320 5300
 AR Path="/5BB27B84/5BB2A083" Ref="#PWR?"  Part="1"
-AR Path="/5BB27B24/5BB2A083" Ref="#PWR?"  Part="1"
-F 0 "#PWR?" H 5320 5050 50  0001 C CNN
+AR Path="/5BB27B24/5BB2A083" Ref="#PWR0303"  Part="1"
+F 0 "#PWR0303" H 5320 5050 50  0001 C CNN
 F 1 "GND" H 5320 5150 50  0000 C CNN
 F 2 "" H 5320 5300 50  0001 C CNN
@@
 P 5320 4840
 AR Path="/5BB27B84/5BB2A089" Ref="#PWR?"  Part="1"
-AR Path="/5BB27B24/5BB2A089" Ref="#PWR?"  Part="1"
-F 0 "#PWR?" H 5320 4690 50  0001 C CNN
+AR Path="/5BB27B24/5BB2A089" Ref="#PWR0302"  Part="1"
+F 0 "#PWR0302" H 5320 4690 50  0001 C CNN
 F 1 "+3.3V" H 5320 4980 50  0000 C CNN
 F 2 "" H 5320 4840 50  0000 C CNN
@@
 	4970 5260 4970 5220
 $Comp
-L power:GND #PWR?
+L power:GND #PWR0305
 U 1 1 5BB2AB7D
 P 5350 4040
-F 0 "#PWR?" H 5350 3790 50  0001 C CNN
+F 0 "#PWR0305" H 5350 3790 50  0001 C CNN
 F 1 "GND" H 5350 3890 50  0000 C CNN
 F 2 "" H 5350 4040 50  0001 C CNN
@@
 P 5350 3240
 AR Path="/5BB27B84/5BB2ABA3" Ref="#PWR?"  Part="1"
-AR Path="/5BB27B24/5BB2ABA3" Ref="#PWR?"  Part="1"
-F 0 "#PWR?" H 5350 3090 50  0001 C CNN
+AR Path="/5BB27B24/5BB2ABA3" Ref="#PWR0304"  Part="1"
+F 0 "#PWR0304" H 5350 3090 50  0001 C CNN
 F 1 "+3.3V" H 5350 3380 50  0000 C CNN
 F 2 "" H 5350 3240 50  0000 C CNN
@@
 P 6670 3060
 AR Path="/5BB27B84/5BB2B17F" Ref="#PWR?"  Part="1"
-AR Path="/5BB27B24/5BB2B17F" Ref="#PWR?"  Part="1"
-F 0 "#PWR?" H 6670 2910 50  0001 C CNN
+AR Path="/5BB27B24/5BB2B17F" Ref="#PWR0306"  Part="1"
+F 0 "#PWR0306" H 6670 2910 50  0001 C CNN
 F 1 "+3.3V" H 6670 3200 50  0000 C CNN
 F 2 "" H 6670 3060 50  0000 C CNN
@@
 P 6670 3210
 AR Path="/5BB27BA3/5BB2B40B" Ref="R?"  Part="1"
-AR Path="/5BB27B24/5BB2B40B" Ref="R?"  Part="1"
-F 0 "R?" H 6590 3210 50  0000 R CNN
+AR Path="/5BB27B24/5BB2B40B" Ref="R301"  Part="1"
+F 0 "R301" H 6590 3210 50  0000 R CNN
 F 1 "10k" V 6670 3210 50  0000 C CNN
 F 2 "" H 6670 3210 50  0001 C CNN
@@
 P 6670 4050
 AR Path="/5BB27BA3/5BB2B41F" Ref="R?"  Part="1"
-AR Path="/5BB27B24/5BB2B41F" Ref="R?"  Part="1"
-F 0 "R?" H 6590 4050 50  0000 R CNN
+AR Path="/5BB27B24/5BB2B41F" Ref="R302"  Part="1"
+F 0 "R302" H 6590 4050 50  0000 R CNN
 F 1 "0" V 6670 4050 50  0000 C CNN
 F 2 "" H 6670 4050 50  0001 C CNN
@@
 Connection ~ 6670 3740
 $Comp
-L power:GND #PWR?
+L power:GND #PWR0307
 U 1 1 5BB2B800
 P 6670 4200
-F 0 "#PWR?" H 6670 3950 50  0001 C CNN
+F 0 "#PWR0307" H 6670 3950 50  0001 C CNN
 F 1 "GND" H 6670 4050 50  0000 C CNN
 F 2 "" H 6670 4200 50  0001 C CNN
@@
 $EndComp
 $Comp
-L Sensor_Current:ACS722xLCTR-20AB U?
+L Sensor_Current:ACS722xLCTR-20AB U301
 U 1 1 5BB31C32
 P 5350 3640
-F 0 "U?" H 5450 4090 50  0000 L CNN
+F 0 "U301" H 5450 4090 50  0000 L CNN
 F 1 "ACS722LLCTR-20AB" H 5450 3990 50  0000 L CNN
 F 2 "" H 5450 3290 50  0001 L CIN
@@
 10.7ARMS Max to support full output swing of conditioning stages
 $Comp
-L power:HT #PWR?
+L power:HT #PWR0301
 U 1 1 5BB463D5
 P 4870 3360
-F 0 "#PWR?" H 4870 3480 50  0001 C CNN
+F 0 "#PWR0301" H 4870 3480 50  0001 C CNN
 F 1 "HT" H 4870 3450 50  0000 C CNN
 F 2 "" H 4870 3360 50  0001 C CNN
@@
 AC Current Sensor
 $Comp
-L Custom_Library:MU_Logo #G?
+L Custom_Library:MU_Logo #G301
 U 1 1 5BB6B7BB
 P 9900 1100
-F 0 "#G?" H 9900 614 60  0001 C CNN
+F 0 "#G301" H 9900 614 60  0001 C CNN
 F 1 "MU_Logo" H 9900 1586 60  0001 C CNN
 F 2 "" H 9900 1100 50  0001 C CNN
