File: hdw/AC_Power_Meter/AC_Current_Sensor.sch (KiCad schematic (older format))
At the start: 6 parts, among them U301 ACS722LLCTR-20AB

Commit message: Placed a lot more parts, netlist cleanup
Changed lines of the file:
@@
 	1    0    0    -1
 $EndComp
-Text GLabel 4950 3740 0    50   Output ~ 0
+Text GLabel 4950 3440 0    50   Output ~ 0
 ISNS_HT_OUT
 $Comp
@@
 L power:HT #PWR0301
 U 1 1 5BB463D5
-P 4870 3360
-F 0 "#PWR0301" H 4870 3480 50  0001 C CNN
-F 1 "HT" H 4870 3450 50  0000 C CNN
-F 2 "" H 4870 3360 50  0001 C CNN
-F 3 "" H 4870 3360 50  0001 C CNN
-	1    4870 3360
+P 4870 3660
+F 0 "#PWR0301" H 4870 3780 50  0001 C CNN
+F 1 "HT" H 4870 3750 50  0000 C CNN
+F 2 "" H 4870 3660 50  0001 C CNN
+F 3 "" H 4870 3660 50  0001 C CNN
+	1    4870 3660
 	1    0    0    -1
 $EndComp
 Wire Wire Line
-	4870 3360 4870 3440
+	4870 3660 4870 3740
 Wire Wire Line
-	4870 3440 4950 3440
+	4870 3740 4950 3740
 Text Notes 540  690  0    100  ~ 20
 AC Current Sensor

Commit message: MOAR ROUTING
Changed lines of the file:
@@
 	1    0    0    -1
 $EndComp
-Text GLabel 4950 3440 0    50   Output ~ 0
+Text GLabel 4950 3740 0    50   Output ~ 0
 ISNS_HT_OUT
 $Comp
@@
 L power:HT #PWR0301
 U 1 1 5BB463D5
-P 4870 3660
-F 0 "#PWR0301" H 4870 3780 50  0001 C CNN
-F 1 "HT" H 4870 3750 50  0000 C CNN
-F 2 "" H 4870 3660 50  0001 C CNN
-F 3 "" H 4870 3660 50  0001 C CNN
-	1    4870 3660
+P 4870 3360
+F 0 "#PWR0301" H 4870 3480 50  0001 C CNN
+F 1 "HT" H 4870 3450 50  0000 C CNN
+F 2 "" H 4870 3360 50  0001 C CNN
+F 3 "" H 4870 3360 50  0001 C CNN
+	1    4870 3360
 	1    0    0    -1
 $EndComp
 Wire Wire Line
-	4870 3660 4870 3740
+	4870 3360 4870 3440
 Wire Wire Line
-	4870 3740 4950 3740
+	4870 3440 4950 3440
 Text Notes 540  690  0    100  ~ 20
 AC Current Sensor
