File: hdw/AC_Power_Meter/AC_Current_Sensor.sch (KiCad schematic (older format))
At the start: 6 parts, among them U301 ACS722LLCTR-20AB

Commit message: Updated most footprints
Parts:
- C301: footprint (none) -> Capacitors_SMD:C_0603; Digi-Key PN PN -> 490-8020-1-ND
- C302: footprint (none) -> Capacitors_SMD:C_0603; Digi-Key PN PN -> 1276-1921-1-ND
- C303: footprint (none) -> Capacitors_SMD:C_0603; Digi-Key PN PN -> 478-1215-1-ND
- R301: footprint (none) -> Resistors_SMD:R_0603; Digi-Key PN PN -> RHM10KADCT-ND
- R302: footprint (none) -> Resistors_SMD:R_0603; Digi-Key PN PN -> (none)
- U301: footprint (none) -> Housings_SOIC:SOIC-8_3.9x4.9mm_Pitch1.27mm
Changed lines of the file:
@@
 F 0 "C301" H 4995 5170 50  0000 L CNN
 F 1 "0.1uF" H 4995 4970 50  0000 L CNN
-F 2 "" H 5008 4920 50  0001 C CNN
+F 2 "Capacitors_SMD:C_0603" H 5008 4920 50  0001 C CNN
 F 3 "" H 4995 5170 50  0001 C CNN
 F 4 "0603" H 4820 5170 50  0000 R CNN "display_footprint"
 F 5 "50V" H 4820 5070 50  0000 R CNN "Voltage"
 F 6 "X7R" H 4820 4970 50  0000 R CNN "Dielectric"
-F 7 "PN" H 5395 5570 60  0001 C CNN "Digi-Key PN"
+F 7 "490-8020-1-ND" H 5395 5570 60  0001 C CNN "Digi-Key PN"
 	1    4970 5070
 	1    0    0    -1
@@
 F 0 "C302" H 5345 5170 50  0000 L CNN
 F 1 "10nF" H 5345 4970 50  0000 L CNN
-F 2 "" H 5358 4920 50  0001 C CNN
+F 2 "Capacitors_SMD:C_0603" H 5358 4920 50  0001 C CNN
 F 3 "" H 5345 5170 50  0001 C CNN
 F 4 "0603" H 5170 5170 50  0001 R CNN "display_footprint"
 F 5 "50V" H 5170 5070 50  0001 R CNN "Voltage"
 F 6 "X7R" H 5170 4970 50  0001 R CNN "Dielectric"
-F 7 "PN" H 5745 5570 60  0001 C CNN "Digi-Key PN"
+F 7 "1276-1921-1-ND" H 5745 5570 60  0001 C CNN "Digi-Key PN"
 	1    5320 5070
 	1    0    0    -1
@@
 F 0 "C303" H 5695 5170 50  0000 L CNN
 F 1 "1nF" H 5695 4970 50  0000 L CNN
-F 2 "" H 5708 4920 50  0001 C CNN
+F 2 "Capacitors_SMD:C_0603" H 5708 4920 50  0001 C CNN
 F 3 "" H 5695 5170 50  0001 C CNN
 F 4 "0603" H 5520 5170 50  0001 R CNN "display_footprint"
 F 5 "50V" H 5520 5070 50  0001 R CNN "Voltage"
 F 6 "X7R" H 5520 4970 50  0001 R CNN "Dielectric"
-F 7 "PN" H 6095 5570 60  0001 C CNN "Digi-Key PN"
+F 7 "478-1215-1-ND" H 6095 5570 60  0001 C CNN "Digi-Key PN"
 	1    5670 5070
 	1    0    0    -1
@@
 F 0 "R301" H 6590 3210 50  0000 R CNN
 F 1 "10k" V 6670 3210 50  0000 C CNN
-F 2 "" H 6670 3210 50  0001 C CNN
+F 2 "Resistors_SMD:R_0603" H 6670 3210 50  0001 C CNN
 F 3 "" H 6670 3210 50  0001 C CNN
 F 4 "0603" H 6770 3290 50  0000 L CNN "display_footprint"
 F 5 "1%" H 6770 3210 50  0000 L CNN "Tolerance"
 F 6 "1/10W" H 6780 3130 50  0000 L CNN "Wattage"
-F 7 "PN" H 6970 3610 60  0001 C CNN "Digi-Key PN"
+F 7 "RHM10KADCT-ND" H 6970 3610 60  0001 C CNN "Digi-Key PN"
 	1    6670 3210
 	-1   0    0    -1
@@
 F 0 "R302" H 6590 4050 50  0000 R CNN
 F 1 "0" V 6670 4050 50  0000 C CNN
-F 2 "" H 6670 4050 50  0001 C CNN
+F 2 "Resistors_SMD:R_0603" H 6670 4050 50  0001 C CNN
 F 3 "" H 6670 4050 50  0001 C CNN
 F 4 "None" H 6590 4130 50  0000 R CNN "Config"
@@
 F 6 "1%" H 6770 4050 50  0000 L CNN "Tolerance"
 F 7 "1/10W" H 6780 3970 50  0000 L CNN "Wattage"
-F 8 "PN" H 6970 4450 60  0001 C CNN "Digi-Key PN"
+F 8 "" H 6970 4450 60  0001 C CNN "Digi-Key PN"
 	1    6670 4050
 	-1   0    0    1
@@
 F 0 "U301" H 5450 4090 50  0000 L CNN
 F 1 "ACS722LLCTR-20AB" H 5450 3990 50  0000 L CNN
-F 2 "" H 5450 3290 50  0001 L CIN
+F 2 "Housings_SOIC:SOIC-8_3.9x4.9mm_Pitch1.27mm" H 5450 3290 50  0001 L CIN
 F 3 "http://www.allegromicro.com/~/media/Files/Datasheets/ACS722-Datasheet.ashx?la=en" H 5350 3640 50  0001 C CNN
 F 4 "620-1637-1-ND" H 5350 3640 50  0001 C CNN "Digi-Key PN"

Commit message: Modified schematic and board files slightly
Parts:
- removed U301: ACS722LLCTR-20AB, Housings_SOIC:SOIC-8_3.9x4.9mm_Pitch1.27mm, symbol Sensor_Current:ACS722xLCTR-20AB
- added U301: ACS722LLCTR-05AB, Package_SO:SOIC-8_3.9x4.9mm_P1.27mm, symbol Sensor_Current:ACS722xLCTR-05AB
Other:
- note added: "5.35 ARMS Max to support full output swing of conditioning stages"
- note removed: "10.7ARMS Max to support full output swing of conditioning stages"
Changed lines of the file:
@@
-	1    0    0    -1
-$EndComp
-$Comp
-L Sensor_Current:ACS722xLCTR-20AB U301
-U 1 1 5BB31C32
-P 5350 3640
-F 0 "U301" H 5450 4090 50  0000 L CNN
-F 1 "ACS722LLCTR-20AB" H 5450 3990 50  0000 L CNN
-F 2 "Housings_SOIC:SOIC-8_3.9x4.9mm_Pitch1.27mm" H 5450 3290 50  0001 L CIN
-F 3 "http://www.allegromicro.com/~/media/Files/Datasheets/ACS722-Datasheet.ashx?la=en" H 5350 3640 50  0001 C CNN
-F 4 "620-1637-1-ND" H 5350 3640 50  0001 C CNN "Digi-Key PN"
-	1    5350 3640
 	1    0    0    -1
 $EndComp
 Text Notes 3530 4440 0    50   ~ 0
-10.7ARMS Max to support full output swing of conditioning stages
+5.35 ARMS Max to support full output swing of conditioning stages
 $Comp
 L power:HT #PWR0301
@@
 Text GLabel 5750 3440 2    50   Output ~ 0
 ISNS_OUT
+$Comp
+L Sensor_Current:ACS722xLCTR-05AB U301
+U 1 1 5BD3627A
+P 5350 3640
+F 0 "U301" H 5450 4090 50  0000 L CNN
+F 1 "ACS722LLCTR-05AB" H 5450 3990 50  0000 L CNN
+F 2 "Package_SO:SOIC-8_3.9x4.9mm_P1.27mm" H 5450 3290 50  0001 L CIN
+F 3 "http://www.allegromicro.com/~/media/Files/Datasheets/ACS722-Datasheet.ashx?la=en" H 5350 3640 50  0001 C CNN
+F 4 "620-1634-1-ND" H 5350 3640 50  0001 C CNN "Digi-Key PN"
+	1    5350 3640
+	1    0    0    -1
+$EndComp
 $EndSCHEMATC

Commit message: Added a lot of functionality in formware
Other:
- note added: "3.787 Peak Amps Max to support full output swing of conditioning stages"
- note removed: "5.35 ARMS Max to support full output swing of conditioning stages"
Changed lines of the file:
@@
 $EndComp
 Text Notes 3530 4440 0    50   ~ 0
-5.35 ARMS Max to support full output swing of conditioning stages
+3.787 Peak Amps Max to support full output swing of conditioning stages
 $Comp
 L power:HT #PWR0301
