File: hdw/AC_Power_Meter/AC_Input.sch (KiCad schematic (older format))
At the start: 5 parts, among them J201 HT_IN, J202 NEUT_IN, J203 EARTH_IN, P201 AC In Socket

Commit message: Updated most footprints
Parts:
- J201, J202, J203: Digi-Key PN (none) -> 732-3214-ND
- P201: Digi-Key PN (none) -> Q223-ND
Changed lines of the file:
@@
 F 2 "" H 4610 3240 50  0001 C CNN
 F 3 "~" H 4610 3240 50  0001 C CNN
+F 4 "732-3214-ND" H 4610 3240 50  0001 C CNN "Digi-Key PN"
 	1    4610 3240
 	-1   0    0    -1
@@
 F 2 "" H 4610 3640 50  0001 C CNN
 F 3 "~" H 4610 3640 50  0001 C CNN
+F 4 "732-3214-ND" H 4610 3640 50  0001 C CNN "Digi-Key PN"
 	1    4610 3640
 	-1   0    0    -1
@@
 F 2 "" H 4610 4040 50  0001 C CNN
 F 3 "~" H 4610 4040 50  0001 C CNN
+F 4 "732-3214-ND" H 4610 4040 50  0001 C CNN "Digi-Key PN"
 	1    4610 4040
 	-1   0    0    -1
@@
 F 2 "" H 2920 3560 50  0001 C CNN
 F 3 "~" H 2920 3560 50  0001 C CNN
+F 4 "Q223-ND" H 2520 3560 50  0001 C CNN "Digi-Key PN"
 	1    2520 3560
 	1    0    0    -1

Commit message: Finished assigning footprints, added netlist
Parts:
- J201, J202, J203: footprint (none) -> Custom Footprints Library:Wuerth_7461096_M4_Shank_9pos
Changed lines of the file:
@@
 F 0 "J201" H 4610 3340 50  0000 C CNN
 F 1 "HT_IN" H 4610 3140 50  0000 C CNN
-F 2 "" H 4610 3240 50  0001 C CNN
+F 2 "Custom Footprints Library:Wuerth_7461096_M4_Shank_9pos" H 4610 3240 50  0001 C CNN
 F 3 "~" H 4610 3240 50  0001 C CNN
 F 4 "732-3214-ND" H 4610 3240 50  0001 C CNN "Digi-Key PN"
@@
 F 0 "J202" H 4610 3740 50  0000 C CNN
 F 1 "NEUT_IN" H 4610 3540 50  0000 C CNN
-F 2 "" H 4610 3640 50  0001 C CNN
+F 2 "Custom Footprints Library:Wuerth_7461096_M4_Shank_9pos" H 4610 3640 50  0001 C CNN
 F 3 "~" H 4610 3640 50  0001 C CNN
 F 4 "732-3214-ND" H 4610 3640 50  0001 C CNN "Digi-Key PN"
@@
 F 0 "J203" H 4610 4140 50  0000 C CNN
 F 1 "EARTH_IN" H 4610 3940 50  0000 C CNN
-F 2 "" H 4610 4040 50  0001 C CNN
+F 2 "Custom Footprints Library:Wuerth_7461096_M4_Shank_9pos" H 4610 4040 50  0001 C CNN
 F 3 "~" H 4610 4040 50  0001 C CNN
 F 4 "732-3214-ND" H 4610 4040 50  0001 C CNN "Digi-Key PN"

Commit message: Made a fw minor adjustments to PCB
Parts:
- added MK201, MK203: 4-40 Screw, symbol Custom_Library:Screw
- added MK202, MK204: Nut, symbol Custom_Library:Nut
Changed lines of the file:
@@
 	5310 4040 4890 4040
 Connection ~ 4890 4040
+$Comp
+L Custom_Library:Screw MK?
+U 1 1 5BBA935B
+P 2020 2100
+AR Path="/5BB27C33/5BBA935B" Ref="MK?"  Part="1"
+AR Path="/5BB27B1A/5BBA935B" Ref="MK201"  Part="1"
+F 0 "MK201" H 2020 2200 50  0000 C CNN
+F 1 "4-40 Screw" H 2020 2300 50  0000 C CNN
+F 2 "" H 2020 2350 50  0001 C CNN
+F 3 "" H 2020 2350 50  0001 C CNN
+F 4 "36-9502-ND" H 2020 2100 50  0001 C CNN "Digi-Key PN"
+	1    2020 2100
+	1    0    0    -1
+$EndComp
+$Comp
+L Custom_Library:Screw MK?
+U 1 1 5BBA9363
+P 2770 2100
+AR Path="/5BB27C33/5BBA9363" Ref="MK?"  Part="1"
+AR Path="/5BB27B1A/5BBA9363" Ref="MK203"  Part="1"
+F 0 "MK203" H 2770 2200 50  0000 C CNN
+F 1 "4-40 Screw" H 2770 2300 50  0000 C CNN
+F 2 "" H 2770 2350 50  0001 C CNN
+F 3 "" H 2770 2350 50  0001 C CNN
+F 4 "36-9502-ND" H 2770 2100 50  0001 C CNN "Digi-Key PN"
+	1    2770 2100
+	1    0    0    -1
+$EndComp
+$Comp
+L Custom_Library:Nut MK202
+U 1 1 5BBAE4E8
+P 2020 2520
+F 0 "MK202" H 2020 2570 50  0000 C CNN
+F 1 "Nut" H 2020 2670 50  0000 C CNN
+F 2 "" H 2020 2870 50  0001 C CNN
+F 3 "" H 2020 2870 50  0001 C CNN
+F 4 "36-4694-ND" H 2020 2520 50  0001 C CNN "Digi-Key PN"
+	1    2020 2520
+	1    0    0    -1
+$EndComp
+$Comp
+L Custom_Library:Nut MK204
+U 1 1 5BBAEFC1
+P 2770 2520
+F 0 "MK204" H 2770 2570 50  0000 C CNN
+F 1 "Nut" H 2770 2670 50  0000 C CNN
+F 2 "" H 2770 2870 50  0001 C CNN
+F 3 "" H 2770 2870 50  0001 C CNN
+F 4 "36-4694-ND" H 2770 2520 50  0001 C CNN "Digi-Key PN"
+	1    2770 2520
+	1    0    0    -1
+$EndComp
 $EndSCHEMATC

Commit message: Serious BOM scrubbing to drive price down
Parts:
- J201, J202, J203: footprint Custom Footprints Library:Wuerth_7461096_M4_Shank_9pos -> Custom Footprints Library:Keystone_8191; Digi-Key PN 732-3214-ND -> 36-8191-ND
Changed lines of the file:
@@
 $Descr A 11000 8500
 encoding utf-8
-Sheet 2 18
+Sheet 2 17
 Title ""
 Date "2018-10-01"
@@
 F 0 "J201" H 4610 3340 50  0000 C CNN
 F 1 "HT_IN" H 4610 3140 50  0000 C CNN
-F 2 "Custom Footprints Library:Wuerth_7461096_M4_Shank_9pos" H 4610 3240 50  0001 C CNN
+F 2 "Custom Footprints Library:Keystone_8191" H 4610 3240 50  0001 C CNN
 F 3 "~" H 4610 3240 50  0001 C CNN
-F 4 "732-3214-ND" H 4610 3240 50  0001 C CNN "Digi-Key PN"
+F 4 "36-8191-ND" H 4610 3240 50  0001 C CNN "Digi-Key PN"
 	1    4610 3240
 	-1   0    0    -1
@@
 F 0 "J202" H 4610 3740 50  0000 C CNN
 F 1 "NEUT_IN" H 4610 3540 50  0000 C CNN
-F 2 "Custom Footprints Library:Wuerth_7461096_M4_Shank_9pos" H 4610 3640 50  0001 C CNN
+F 2 "Custom Footprints Library:Keystone_8191" H 4610 3640 50  0001 C CNN
 F 3 "~" H 4610 3640 50  0001 C CNN
-F 4 "732-3214-ND" H 4610 3640 50  0001 C CNN "Digi-Key PN"
+F 4 "36-8191-ND" H 4610 3640 50  0001 C CNN "Digi-Key PN"
 	1    4610 3640
 	-1   0    0    -1
@@
 F 0 "J203" H 4610 4140 50  0000 C CNN
 F 1 "EARTH_IN" H 4610 3940 50  0000 C CNN
-F 2 "Custom Footprints Library:Wuerth_7461096_M4_Shank_9pos" H 4610 4040 50  0001 C CNN
+F 2 "Custom Footprints Library:Keystone_8191" H 4610 4040 50  0001 C CNN
 F 3 "~" H 4610 4040 50  0001 C CNN
-F 4 "732-3214-ND" H 4610 4040 50  0001 C CNN "Digi-Key PN"
+F 4 "36-8191-ND" H 4610 4040 50  0001 C CNN "Digi-Key PN"
 	1    4610 4040
 	-1   0    0    -1
