File: hdw/AC_Power_Meter/AC_Output.sch (KiCad schematic (older format))
At the start: 5 parts, among them J401 HT_OUT, J402 NEUT_OUT, J403 EARTH_OUT, J404 Output Socket

Commit message: Updated most footprints
Parts:
- J401, J402, J403: Digi-Key PN (none) -> 732-3214-ND
- J404: Digi-Key PN (none) -> Q337-ND
Changed lines of the file:
@@
 F 2 "" H 5640 3390 50  0001 C CNN
 F 3 "~" H 5640 3390 50  0001 C CNN
+F 4 "732-3214-ND" H 5640 3390 50  0001 C CNN "Digi-Key PN"
 	1    5640 3390
 	1    0    0    -1
@@
 F 2 "" H 5640 3790 50  0001 C CNN
 F 3 "~" H 5640 3790 50  0001 C CNN
+F 4 "732-3214-ND" H 5640 3790 50  0001 C CNN "Digi-Key PN"
 	1    5640 3790
 	1    0    0    -1
@@
 F 2 "" H 5640 4190 50  0001 C CNN
 F 3 "~" H 5640 4190 50  0001 C CNN
+F 4 "732-3214-ND" H 5640 4190 50  0001 C CNN "Digi-Key PN"
 	1    5640 4190
 	1    0    0    -1
@@
 F 2 "" H 7970 3890 50  0001 C CNN
 F 3 "~" H 7970 3890 50  0001 C CNN
+F 4 "Q337-ND" H 8270 3790 50  0001 C CNN "Digi-Key PN"
 	1    8270 3790
 	1    0    0    -1

Commit message: Finished assigning footprints, added netlist
Parts:
- J401, J402, J403: footprint (none) -> Custom Footprints Library:Wuerth_7461096_M4_Shank_9pos
Changed lines of the file:
@@
 F 0 "J401" H 5640 3490 50  0000 C CNN
 F 1 "HT_OUT" H 5640 3290 50  0000 C CNN
-F 2 "" H 5640 3390 50  0001 C CNN
+F 2 "Custom Footprints Library:Wuerth_7461096_M4_Shank_9pos" H 5640 3390 50  0001 C CNN
 F 3 "~" H 5640 3390 50  0001 C CNN
 F 4 "732-3214-ND" H 5640 3390 50  0001 C CNN "Digi-Key PN"
@@
 F 0 "J402" H 5640 3890 50  0000 C CNN
 F 1 "NEUT_OUT" H 5640 3690 50  0000 C CNN
-F 2 "" H 5640 3790 50  0001 C CNN
+F 2 "Custom Footprints Library:Wuerth_7461096_M4_Shank_9pos" H 5640 3790 50  0001 C CNN
 F 3 "~" H 5640 3790 50  0001 C CNN
 F 4 "732-3214-ND" H 5640 3790 50  0001 C CNN "Digi-Key PN"
@@
 F 0 "J403" H 5640 4290 50  0000 C CNN
 F 1 "EARTH_OUT" H 5640 4090 50  0000 C CNN
-F 2 "" H 5640 4190 50  0001 C CNN
+F 2 "Custom Footprints Library:Wuerth_7461096_M4_Shank_9pos" H 5640 4190 50  0001 C CNN
 F 3 "~" H 5640 4190 50  0001 C CNN
 F 4 "732-3214-ND" H 5640 4190 50  0001 C CNN "Digi-Key PN"

Commit message: Serious BOM scrubbing to drive price down
Parts:
- J401, J402, J403: footprint Custom Footprints Library:Wuerth_7461096_M4_Shank_9pos -> Custom Footprints Library:Keystone_8191; Digi-Key PN 732-3214-ND -> 36-8191-ND
Changed lines of the file:
@@
 $Descr A 11000 8500
 encoding utf-8
-Sheet 4 18
+Sheet 4 17
 Title ""
 Date "2018-10-01"
@@
 F 0 "J401" H 5640 3490 50  0000 C CNN
 F 1 "HT_OUT" H 5640 3290 50  0000 C CNN
-F 2 "Custom Footprints Library:Wuerth_7461096_M4_Shank_9pos" H 5640 3390 50  0001 C CNN
+F 2 "Custom Footprints Library:Keystone_8191" H 5640 3390 50  0001 C CNN
 F 3 "~" H 5640 3390 50  0001 C CNN
-F 4 "732-3214-ND" H 5640 3390 50  0001 C CNN "Digi-Key PN"
+F 4 "36-8191-ND" H 5640 3390 50  0001 C CNN "Digi-Key PN"
 	1    5640 3390
 	1    0    0    -1
@@
 F 0 "J402" H 5640 3890 50  0000 C CNN
 F 1 "NEUT_OUT" H 5640 3690 50  0000 C CNN
-F 2 "Custom Footprints Library:Wuerth_7461096_M4_Shank_9pos" H 5640 3790 50  0001 C CNN
+F 2 "Custom Footprints Library:Keystone_8191" H 5640 3790 50  0001 C CNN
 F 3 "~" H 5640 3790 50  0001 C CNN
-F 4 "732-3214-ND" H 5640 3790 50  0001 C CNN "Digi-Key PN"
+F 4 "36-8191-ND" H 5640 3790 50  0001 C CNN "Digi-Key PN"
 	1    5640 3790
 	1    0    0    -1
@@
 F 0 "J403" H 5640 4290 50  0000 C CNN
 F 1 "EARTH_OUT" H 5640 4090 50  0000 C CNN
-F 2 "Custom Footprints Library:Wuerth_7461096_M4_Shank_9pos" H 5640 4190 50  0001 C CNN
+F 2 "Custom Footprints Library:Keystone_8191" H 5640 4190 50  0001 C CNN
 F 3 "~" H 5640 4190 50  0001 C CNN
-F 4 "732-3214-ND" H 5640 4190 50  0001 C CNN "Digi-Key PN"
+F 4 "36-8191-ND" H 5640 4190 50  0001 C CNN "Digi-Key PN"
 	1    5640 4190
 	1    0    0    -1
 $EndComp
-Text GLabel 4840 3390 0    50   Input ~ 0
-TRIAC_HT_OUT
 Text Notes 6460 3820 0    50   ~ 0
 -> To Panel AC Output Socket
@@
 NoConn ~ 8070 3790
 NoConn ~ 8070 3990
+Text GLabel 4840 3390 0    50   Input ~ 0
+TRIAC_HT_OUT
 $EndSCHEMATC
