File: hdw/AC_Power_Meter/POS12_Power_Supply.sch (KiCad schematic (older format))
At the start: 0 parts

Commit message: Added TRIAC circuit and POS12 AC/DC converter
Parts:
- added C?: 0.1uF, symbol Custom_Library:C_Custom
- added C?: 47uF, symbol Custom_Library:CP_Tant_Custom
- added F?: 3.15A, symbol Device:Fuse
- added PS?: TMLM04112, Converters_DCDC_ACDC:ACDC-Conv_Traco-TMLM-04, symbol Converter_ACDC:TMLM04112
Connections:
- net labels added: +12V, GND, HT, NEUT
- wire segments 0 -> 12
Other:
- note added: "Maximum Output Current: 333mA"
Changed lines of the file:
@@
 Comment4 ""
 $EndDescr
+$Comp
+L Custom_Library:C_Custom C?
+U 1 1 5BB476E0
+P 6520 3540
+AR Path="/5BB27BA3/5BB476E0" Ref="C?"  Part="1"
+AR Path="/5BB27B84/5BB476E0" Ref="C?"  Part="1"
+AR Path="/5BB27B24/5BB476E0" Ref="C?"  Part="1"
+AR Path="/5BB27B51/5BB476E0" Ref="C?"  Part="1"
+F 0 "C?" H 6545 3640 50  0000 L CNN
+F 1 "0.1uF" H 6545 3440 50  0000 L CNN
+F 2 "" H 6558 3390 50  0001 C CNN
+F 3 "" H 6545 3640 50  0001 C CNN
+F 4 "0603" H 6370 3640 50  0000 R CNN "display_footprint"
+F 5 "50V" H 6370 3540 50  0000 R CNN "Voltage"
+F 6 "X7R" H 6370 3440 50  0000 R CNN "Dielectric"
+F 7 "PN" H 6945 4040 60  0001 C CNN "Digi-Key PN"
+	1    6520 3540
+	1    0    0    -1
+$EndComp
+$Comp
+L Converter_ACDC:TMLM04112 PS?
+U 1 1 5BB47753
+P 5240 3410
+F 0 "PS?" H 5040 3610 50  0000 C CNN
+F 1 "TMLM04112" H 5240 3210 50  0000 C CNN
+F 2 "Converters_DCDC_ACDC:ACDC-Conv_Traco-TMLM-04" H 5240 3110 50  0001 C CNN
+F 3 "https://www.tracopower.com/products/tmlm.pdf" H 5240 3410 50  0001 C CNN
+F 4 "1951-1352-ND" H 5240 3410 50  0001 C CNN "Digi-Key PN"
+	1    5240 3410
+	1    0    0    -1
+$EndComp
+$Comp
+L Device:Fuse F?
+U 1 1 5BB4775A
+P 4300 3310
+F 0 "F?" V 4380 3310 50  0000 C CNN
+F 1 "3.15A" V 4225 3310 50  0000 C CNN
+F 2 "" V 4230 3310 50  0001 C CNN
+F 3 "~" H 4300 3310 50  0001 C CNN
+	1    4300 3310
+	0    1    1    0
+$EndComp
+Wire Wire Line
+	4450 3310 4840 3310
+$Comp
+L power:GND #PWR?
+U 1 1 5BB47762
+P 5720 3590
+AR Path="/5BB27B1A/5BB47762" Ref="#PWR?"  Part="1"
+AR Path="/5BB27B51/5BB47762" Ref="#PWR?"  Part="1"
+F 0 "#PWR?" H 5720 3340 50  0001 C CNN
+F 1 "GND" H 5720 3440 50  0000 C CNN
+F 2 "" H 5720 3590 50  0001 C CNN
+F 3 "" H 5720 3590 50  0001 C CNN
+	1    5720 3590
+	1    0    0    -1
+$EndComp
+Wire Wire Line
+	5720 3590 5720 3510
+Wire Wire Line
+	5720 3510 5640 3510
+Wire Wire Line
+	6520 3390 6520 3310
+Wire Wire Line
+	6520 3310 5640 3310
+$Comp
+L power:GND #PWR?
+U 1 1 5BB477D9
+P 6520 3690
+AR Path="/5BB27B1A/5BB477D9" Ref="#PWR?"  Part="1"
+AR Path="/5BB27B51/5BB477D9" Ref="#PWR?"  Part="1"
+F 0 "#PWR?" H 6520 3440 50  0001 C CNN
+F 1 "GND" H 6520 3540 50  0000 C CNN
+F 2 "" H 6520 3690 50  0001 C CNN
+F 3 "" H 6520 3690 50  0001 C CNN
+	1    6520 3690
+	1    0    0    -1
+$EndComp
+$Comp
+L Custom_Library:CP_Tant_Custom C?
+U 1 1 5BB47B13
+P 7250 3540
+F 0 "C?" H 7275 3640 50  0000 L CNN
+F 1 "47uF" H 7275 3440 50  0000 L CNN
+F 2 "" H 7288 3390 50  0001 C CNN
+F 3 "" H 7275 3640 50  0001 C CNN
+F 4 "478-3938-1-ND" H 7250 3540 50  0001 C CNN "Digi-Key PN"
+F 5 "7343" H 7100 3640 50  0000 R CNN "display_footprint"
+F 6 "16V" H 7100 3540 50  0000 R CNN "Voltage"
+F 7 "10%" H 7100 3440 50  0000 R CNN "Tolerance"
+	1    7250 3540
+	1    0    0    -1
+$EndComp
+Wire Wire Line
+	7250 3390 7250 3310
+Wire Wire Line
+	7250 3310 6520 3310
+Connection ~ 6520 3310
+$Comp
+L power:GND #PWR?
+U 1 1 5BB47B87
+P 7250 3690
+AR Path="/5BB27B1A/5BB47B87" Ref="#PWR?"  Part="1"
+AR Path="/5BB27B51/5BB47B87" Ref="#PWR?"  Part="1"
+F 0 "#PWR?" H 7250 3440 50  0001 C CNN
+F 1 "GND" H 7250 3540 50  0000 C CNN
+F 2 "" H 7250 3690 50  0001 C CNN
+F 3 "" H 7250 3690 50  0001 C CNN
+	1    7250 3690
+	1    0    0    -1
+$EndComp
+$Comp
+L power:+12V #PWR?
+U 1 1 5BB484FE
+P 7250 3230
+F 0 "#PWR?" H 7250 3080 50  0001 C CNN
+F 1 "+12V" H 7250 3370 50  0000 C CNN
+F 2 "" H 7250 3230 50  0001 C CNN
+F 3 "" H 7250 3230 50  0001 C CNN
+	1    7250 3230
+	1    0    0    -1
+$EndComp
+Wire Wire Line
+	7250 3230 7250 3310
+Connection ~ 7250 3310
+Text Notes 7620 3470 0    50   ~ 0
+Maximum Output Current: 333mA
+$Comp
+L power:HT #PWR?
+U 1 1 5BB48B61
+P 4070 3230
+F 0 "#PWR?" H 4070 3350 50  0001 C CNN
+F 1 "HT" H 4070 3320 50  0000 C CNN
+F 2 "" H 4070 3230 50  0001 C CNN
+F 3 "" H 4070 3230 50  0001 C CNN
+	1    4070 3230
+	1    0    0    -1
+$EndComp
+Wire Wire Line
+	4070 3230 4070 3310
+Wire Wire Line
+	4070 3310 4150 3310
+$Comp
+L power:NEUT #PWR?
+U 1 1 5BB48BFF
+P 4070 3590
+F 0 "#PWR?" H 4070 3440 50  0001 C CNN
+F 1 "NEUT" H 4070 3740 50  0000 C CNN
+F 2 "" H 4070 3590 50  0001 C CNN
+F 3 "" H 4070 3590 50  0001 C CNN
+	1    4070 3590
+	-1   0    0    1
+$EndComp
+Wire Wire Line
+	4070 3590 4070 3510
+Wire Wire Line
+	4070 3510 4840 3510
 $EndSCHEMATC

Commit message: Added AC input and output connections, added mechanical components
Parts:
- F?: footprint (none) -> Fuse_Holders_and_Fuses:Fuse_CB61F; Digi-Key PN (none) -> 283-4107-1-ND
Changed lines of the file:
@@
 U 1 1 5BB47753
 P 5240 3410
+AR Path="/5BB27B1A/5BB47753" Ref="PS?"  Part="1"
+AR Path="/5BB27B51/5BB47753" Ref="PS?"  Part="1"
 F 0 "PS?" H 5040 3610 50  0000 C CNN
 F 1 "TMLM04112" H 5240 3210 50  0000 C CNN
@@
 U 1 1 5BB4775A
 P 4300 3310
+AR Path="/5BB27B1A/5BB4775A" Ref="F?"  Part="1"
+AR Path="/5BB27B51/5BB4775A" Ref="F?"  Part="1"
 F 0 "F?" V 4380 3310 50  0000 C CNN
 F 1 "3.15A" V 4225 3310 50  0000 C CNN
-F 2 "" V 4230 3310 50  0001 C CNN
+F 2 "Fuse_Holders_and_Fuses:Fuse_CB61F" V 4230 3310 50  0001 C CNN
 F 3 "~" H 4300 3310 50  0001 C CNN
+F 4 "283-4107-1-ND" H 4300 3310 50  0001 C CNN "Digi-Key PN"
 	1    4300 3310
 	0    1    1    0

Commit message: Added +3.3V power supply, +12V window comparator, a few design files
Parts:
- added C? (x2): 0.1uF, symbol Custom_Library:C_Custom
- added C?: 10nF, symbol Custom_Library:C_Custom
- added C?: 1nF, symbol Custom_Library:C_Custom
- added F?: 3.15A, Fuse_Holders_and_Fuses:Fuse_CB61F, symbol Device:Fuse
- added J?: AUX_IN, symbol Connector:Barrel_Jack_Switch
- added R? (x3): R, symbol Custom_Library:R_Custom
- added R? (x2): 10k, symbol Custom_Library:R_Custom
- added TP?: TP, symbol Custom_Library:TP
- added U?: 74LVC1G17, TO_SOT_Packages_SMD:SOT-353_SC-70-5, symbol Custom_Library:74LVC1G17_Power
- added U?: LT6700-1-S6, TO_SOT_Packages_SMD:TSOT-23-6, symbol Custom_Library:LT6700-1-S6
Connections:
- net labels added: +3.3V, POS12_PGOOD
- wire segments 12 -> 46
- no-connect marks 0 -> 1
Other:
- moved on the sheet: PS?

Commit message: Added MU logo and titles to all sheets
Other:
- note added: "+12V 4W Isolated AC/DC Converter, +12V PGOOD Window Comparator"
Changed lines of the file:
@@
 Wire Wire Line
 	5370 2910 5040 2910
+Text Notes 540  690  0    100  ~ 20
++12V 4W Isolated AC/DC Converter, +12V PGOOD Window Comparator
+$Comp
+L Mu_Logo:LOGO #G?
+U 1 1 5BBF23CB
+P 9900 1000
+F 0 "#G?" H 9900 670 60  0001 C CNN
+F 1 "LOGO" H 9900 1330 60  0001 C CNN
+F 2 "" H 9900 1000 50  0001 C CNN
+F 3 "" H 9900 1000 50  0001 C CNN
+	1    9900 1000
+	1    0    0    -1
+$EndComp
 $EndSCHEMATC

Commit message: Updated MU logo to crisper image
Changed lines of the file:
@@
 +12V 4W Isolated AC/DC Converter, +12V PGOOD Window Comparator
 $Comp
-L Mu_Logo:LOGO #G?
-U 1 1 5BBF23CB
-P 9900 1000
-F 0 "#G?" H 9900 670 60  0001 C CNN
-F 1 "LOGO" H 9900 1330 60  0001 C CNN
-F 2 "" H 9900 1000 50  0001 C CNN
-F 3 "" H 9900 1000 50  0001 C CNN
-	1    9900 1000
+L Custom_Library:MU_Logo #G?
+U 1 1 5BB684EA
+P 9900 1100
+F 0 "#G?" H 9900 614 60  0001 C CNN
+F 1 "MU_Logo" H 9900 1586 60  0001 C CNN
+F 2 "" H 9900 1100 50  0001 C CNN
+F 3 "" H 9900 1100 50  0001 C CNN
+	1    9900 1100
 	1    0    0    -1
 $EndComp

Commit message: Revised signal conditioning, cleaned up a lot of pages
Parts:
- added Q?: BSS83P, Package_TO_SOT_SMD:SOT-23, symbol Transistor_FET:BSS83P
- added R?: 10k, symbol Custom_Library:R_Custom
- added Z?: UDZSTE-175.1B, symbol Custom_Library:ZENER_Custom
- J?: Config None -> (none)
- R?: value R -> 10.5k
- R?: value R -> 42.3k
- R?: value R -> 1.4M; Digi-Key PN PN -> P3.3MGCT-ND
Connections:
- wire segments 46 -> 52
Other:
- moved on the sheet: PS?

Commit message: Added pushbuttons sheet, prelim wiring on micro
Parts:
- added R?: 3.3k, symbol Custom_Library:R_Custom
- added R?: 10k, symbol Custom_Library:R_Custom
Connections:
- net labels added: POS12_ADC
- wire segments 52 -> 55
Changed lines of the file:
@@
 $Descr A 11000 8500
 encoding utf-8
-Sheet 5 16
+Sheet 5 17
 Title ""
 Date "2018-10-01"
@@
 	9070 2890 9070 2970
 Connection ~ 9070 2970
+$Comp
+L Custom_Library:R_Custom R?
+U 1 1 5BC1F9F5
+P 1190 6950
+AR Path="/5BB27BA3/5BC1F9F5" Ref="R?"  Part="1"
+AR Path="/5BB27B24/5BC1F9F5" Ref="R?"  Part="1"
+AR Path="/5BB27BB5/5BC1F9F5" Ref="R?"  Part="1"
+F 0 "R?" H 1110 6950 50  0000 R CNN
+F 1 "3.3k" V 1190 6950 40  0000 C CNN
+F 2 "" H 1190 6950 50  0001 C CNN
+F 3 "" H 1190 6950 50  0001 C CNN
+F 4 "0603" H 1290 7030 50  0000 L CNN "display_footprint"
+F 5 "1%" H 1290 6950 50  0000 L CNN "Tolerance"
+F 6 "1/10W" H 1300 6870 50  0000 L CNN "Wattage"
+F 7 "PN" H 1490 7350 60  0001 C CNN "Digi-Key PN"
+	1    1190 6950
+	-1   0    0    -1
+$EndComp
+$Comp
+L power:GND #PWR?
+U 1 1 5BC1F9FC
+P 1190 7100
+AR Path="/5BB27B24/5BC1F9FC" Ref="#PWR?"  Part="1"
+AR Path="/5BB27BB5/5BC1F9FC" Ref="#PWR?"  Part="1"
+F 0 "#PWR?" H 1190 6850 50  0001 C CNN
+F 1 "GND" H 1190 6950 50  0000 C CNN
+F 2 "" H 1190 7100 50  0001 C CNN
+F 3 "" H 1190 7100 50  0001 C CNN
+	1    1190 7100
+	1    0    0    -1
+$EndComp
+$Comp
+L Custom_Library:R_Custom R?
+U 1 1 5BC1FA08
+P 1190 6310
+AR Path="/5BB27BA3/5BC1FA08" Ref="R?"  Part="1"
+AR Path="/5BB27B24/5BC1FA08" Ref="R?"  Part="1"
+AR Path="/5BB27BB5/5BC1FA08" Ref="R?"  Part="1"
+F 0 "R?" H 1110 6310 50  0000 R CNN
+F 1 "10k" V 1190 6310 50  0000 C CNN
+F 2 "" H 1190 6310 50  0001 C CNN
+F 3 "" H 1190 6310 50  0001 C CNN
+F 4 "0603" H 1290 6390 50  0000 L CNN "display_footprint"
+F 5 "1%" H 1290 6310 50  0000 L CNN "Tolerance"
+F 6 "1/10W" H 1300 6230 50  0000 L CNN "Wattage"
+F 7 "PN" H 1490 6710 60  0001 C CNN "Digi-Key PN"
+	1    1190 6310
+	-1   0    0    -1
+$EndComp
+$Comp
+L power:+12V #PWR?
+U 1 1 5BC2065A
+P 1190 6160
+F 0 "#PWR?" H 1190 6010 50  0001 C CNN
+F 1 "+12V" H 1190 6300 50  0000 C CNN
+F 2 "" H 1190 6160 50  0001 C CNN
+F 3 "" H 1190 6160 50  0001 C CNN
+	1    1190 6160
+	1    0    0    -1
+$EndComp
+Wire Wire Line
+	1190 6460 1190 6630
+Text GLabel 1320 6630 2    50   Output ~ 0
+POS12_ADC
+Wire Wire Line
+	1320 6630 1190 6630
+Connection ~ 1190 6630
+Wire Wire Line
+	1190 6630 1190 6800
 $EndSCHEMATC

Commit message: Rewired a few micro symbols, add FMW notes
Parts:
- gave numbers to parts that had none: 23
Connections:
- wire segments 55 -> 57
