File: hdw/AC_Power_Meter/POS12_Power_Supply.sch (KiCad schematic (older format))
At the start: 23 parts, among them J501 AUX_IN, Q501 BSS83P, U501 LT6700-1-S6, U502 74LVC1G17

Commit message: Updated most footprints
Parts:
- C501, C504, C506: footprint (none) -> Capacitors_SMD:C_0603; Digi-Key PN PN -> 490-8020-1-ND
- C502: footprint (none) -> Capacitors_SMD:C_0603; Digi-Key PN PN -> 1276-1921-1-ND
- C503: footprint (none) -> Capacitors_SMD:C_0603; Digi-Key PN PN -> 478-1215-1-ND
- C505: footprint (none) -> Capacitors_Tantalum_SMD:CP_Tantalum_Case-X_EIA-7343-43_Reflow
- J501: footprint (none) -> Connectors:BARREL_JACK
- Q501: value BSS83P -> DMP3099L-7; Digi-Key PN (none) -> DMP3099L-7DICT-ND
- R501, R506, R507, R508: footprint (none) -> Resistors_SMD:R_0603; Digi-Key PN PN -> RHM10KADCT-ND
- R502: footprint (none) -> Resistors_SMD:R_0603; Digi-Key PN PN -> 311-3.30KHRCT-ND
- R503: footprint (none) -> Resistors_SMD:R_0603
- R504: footprint (none) -> Resistors_SMD:R_0603; Digi-Key PN PN -> 311-2399-1-ND
- R505: value 42.3k -> 43.2k; footprint (none) -> Resistors_SMD:R_0603; Digi-Key PN PN -> P43.2KHCT-ND
- TP501: footprint (none) -> Measurement_Points:Measurement_Point_Round-SMD-Pad_Small
- Z501: footprint (none) -> Diodes_SMD:D_SOD-523
Changed lines of the file:
@@
 F 0 "C504" H 4145 3240 50  0000 L CNN
 F 1 "0.1uF" H 4145 3040 50  0000 L CNN
-F 2 "" H 4158 2990 50  0001 C CNN
+F 2 "Capacitors_SMD:C_0603" H 4158 2990 50  0001 C CNN
 F 3 "" H 4145 3240 50  0001 C CNN
 F 4 "0603" H 3970 3240 50  0000 R CNN "display_footprint"
 F 5 "50V" H 3970 3140 50  0000 R CNN "Voltage"
 F 6 "X7R" H 3970 3040 50  0000 R CNN "Dielectric"
-F 7 "PN" H 4545 3640 60  0001 C CNN "Digi-Key PN"
+F 7 "490-8020-1-ND" H 4545 3640 60  0001 C CNN "Digi-Key PN"
 	1    4120 3140
 	1    0    0    -1
@@
 F 0 "C505" H 4875 3240 50  0000 L CNN
 F 1 "47uF" H 4875 3040 50  0000 L CNN
-F 2 "" H 4888 2990 50  0001 C CNN
+F 2 "Capacitors_Tantalum_SMD:CP_Tantalum_Case-X_EIA-7343-43_Reflow" H 4888 2990 50  0001 C CNN
 F 3 "" H 4875 3240 50  0001 C CNN
 F 4 "478-3938-1-ND" H 4850 3140 50  0001 C CNN "Digi-Key PN"
@@
 F 0 "R504" H 2770 5160 50  0000 R CNN
 F 1 "10.5k" V 2850 5160 40  0000 C CNN
-F 2 "" H 2850 5160 50  0001 C CNN
+F 2 "Resistors_SMD:R_0603" H 2850 5160 50  0001 C CNN
 F 3 "" H 2850 5160 50  0001 C CNN
 F 4 "0603" H 2950 5240 50  0000 L CNN "display_footprint"
 F 5 "1%" H 2950 5160 50  0000 L CNN "Tolerance"
 F 6 "1/10W" H 2960 5080 50  0000 L CNN "Wattage"
-F 7 "PN" H 3150 5560 60  0001 C CNN "Digi-Key PN"
+F 7 "311-2399-1-ND" H 3150 5560 60  0001 C CNN "Digi-Key PN"
 	1    2850 5160
 	1    0    0    -1
@@
 AR Path="/5BB27B51/5BB52432" Ref="R505"  Part="1"
 F 0 "R505" H 2770 5640 50  0000 R CNN
-F 1 "42.3k" V 2850 5640 40  0000 C CNN
-F 2 "" H 2850 5640 50  0001 C CNN
+F 1 "43.2k" V 2850 5640 40  0000 C CNN
+F 2 "Resistors_SMD:R_0603" H 2850 5640 50  0001 C CNN
 F 3 "" H 2850 5640 50  0001 C CNN
 F 4 "0603" H 2950 5720 50  0000 L CNN "display_footprint"
 F 5 "1%" H 2950 5640 50  0000 L CNN "Tolerance"
 F 6 "1/10W" H 2960 5560 50  0000 L CNN "Wattage"
-F 7 "PN" H 3150 6040 60  0001 C CNN "Digi-Key PN"
+F 7 "P43.2KHCT-ND" H 3150 6040 60  0001 C CNN "Digi-Key PN"
 	1    2850 5640
 	1    0    0    -1
@@
 F 0 "R503" H 2770 4670 50  0000 R CNN
 F 1 "1.4M" V 2850 4670 40  0000 C CNN
-F 2 "" H 2850 4670 50  0001 C CNN
+F 2 "Resistors_SMD:R_0603" H 2850 4670 50  0001 C CNN
 F 3 "" H 2850 4670 50  0001 C CNN
 F 4 "P3.3MGCT-ND" H 3150 5070 60  0001 C CNN "Digi-Key PN"
@@
 F 0 "R506" H 4670 4680 50  0000 R CNN
 F 1 "10k" V 4750 4680 50  0000 C CNN
-F 2 "" H 4750 4680 50  0001 C CNN
+F 2 "Resistors_SMD:R_0603" H 4750 4680 50  0001 C CNN
 F 3 "" H 4750 4680 50  0001 C CNN
 F 4 "0603" H 4850 4760 50  0000 L CNN "display_footprint"
 F 5 "1%" H 4850 4680 50  0000 L CNN "Tolerance"
 F 6 "1/10W" H 4860 4600 50  0000 L CNN "Wattage"
-F 7 "PN" H 5050 5080 60  0001 C CNN "Digi-Key PN"
+F 7 "RHM10KADCT-ND" H 5050 5080 60  0001 C CNN "Digi-Key PN"
 	1    4750 4680
 	1    0    0    -1
@@
 F 0 "R507" H 6780 5740 50  0000 R CNN
 F 1 "10k" V 6860 5740 50  0000 C CNN
-F 2 "" H 6860 5740 50  0001 C CNN
+F 2 "Resistors_SMD:R_0603" H 6860 5740 50  0001 C CNN
 F 3 "" H 6860 5740 50  0001 C CNN
 F 4 "0603" H 6960 5820 50  0000 L CNN "display_footprint"
 F 5 "1%" H 6960 5740 50  0000 L CNN "Tolerance"
 F 6 "1/10W" H 6970 5660 50  0000 L CNN "Wattage"
-F 7 "PN" H 7160 6140 60  0001 C CNN "Digi-Key PN"
+F 7 "RHM10KADCT-ND" H 7160 6140 60  0001 C CNN "Digi-Key PN"
 	1    6860 5740
 	1    0    0    -1
@@
 F 0 "C506" H 6055 6100 50  0000 L CNN
 F 1 "0.1uF" H 6055 5900 50  0000 L CNN
-F 2 "" H 6068 5850 50  0001 C CNN
+F 2 "Capacitors_SMD:C_0603" H 6068 5850 50  0001 C CNN
 F 3 "" H 6055 6100 50  0001 C CNN
 F 4 "0603" H 5880 6100 50  0000 R CNN "display_footprint"
 F 5 "50V" H 5880 6000 50  0000 R CNN "Voltage"
 F 6 "X7R" H 5880 5900 50  0000 R CNN "Dielectric"
-F 7 "PN" H 6455 6500 60  0001 C CNN "Digi-Key PN"
+F 7 "490-8020-1-ND" H 6455 6500 60  0001 C CNN "Digi-Key PN"
 	1    6030 6000
 	1    0    0    -1
@@
 F 0 "J501" H 7240 3280 50  0000 C CNN
 F 1 "AUX_IN" H 7240 2870 50  0000 C CNN
-F 2 "" H 7290 3030 50  0001 C CNN
+F 2 "Connectors:BARREL_JACK" H 7290 3030 50  0001 C CNN
 F 3 "~" H 7290 3030 50  0001 C CNN
 F 4 "" H 7240 2780 50  0001 C CNN "Config"
@@
 F 0 "C501" H 3425 6680 50  0000 L CNN
 F 1 "0.1uF" H 3425 6480 50  0000 L CNN
-F 2 "" H 3438 6430 50  0001 C CNN
+F 2 "Capacitors_SMD:C_0603" H 3438 6430 50  0001 C CNN
 F 3 "" H 3425 6680 50  0001 C CNN
 F 4 "0603" H 3250 6680 50  0000 R CNN "display_footprint"
 F 5 "50V" H 3250 6580 50  0000 R CNN "Voltage"
 F 6 "X7R" H 3250 6480 50  0000 R CNN "Dielectric"
-F 7 "PN" H 3825 7080 60  0001 C CNN "Digi-Key PN"
+F 7 "490-8020-1-ND" H 3825 7080 60  0001 C CNN "Digi-Key PN"
 	1    3400 6580
 	1    0    0    -1
@@
 F 0 "C502" H 3775 6680 50  0000 L CNN
 F 1 "10nF" H 3775 6480 50  0000 L CNN
-F 2 "" H 3788 6430 50  0001 C CNN
+F 2 "Capacitors_SMD:C_0603" H 3788 6430 50  0001 C CNN
 F 3 "" H 3775 6680 50  0001 C CNN
 F 4 "0603" H 3600 6680 50  0001 R CNN "display_footprint"
 F 5 "50V" H 3600 6580 50  0001 R CNN "Voltage"
 F 6 "X7R" H 3600 6480 50  0001 R CNN "Dielectric"
-F 7 "PN" H 4175 7080 60  0001 C CNN "Digi-Key PN"
+F 7 "1276-1921-1-ND" H 4175 7080 60  0001 C CNN "Digi-Key PN"
 	1    3750 6580
 	1    0    0    -1
@@
 F 0 "C503" H 4125 6680 50  0000 L CNN
 F 1 "1nF" H 4125 6480 50  0000 L CNN
-F 2 "" H 4138 6430 50  0001 C CNN
+F 2 "Capacitors_SMD:C_0603" H 4138 6430 50  0001 C CNN
 F 3 "" H 4125 6680 50  0001 C CNN
 F 4 "0603" H 3950 6680 50  0001 R CNN "display_footprint"
 F 5 "50V" H 3950 6580 50  0001 R CNN "Voltage"
 F 6 "X7R" H 3950 6480 50  0001 R CNN "Dielectric"
-F 7 "PN" H 4525 7080 60  0001 C CNN "Digi-Key PN"
+F 7 "478-1215-1-ND" H 4525 7080 60  0001 C CNN "Digi-Key PN"
 	1    4100 6580
 	1    0    0    -1
@@
 F 0 "TP501" H 3570 2980 50  0000 C CNN
 F 1 "TP" H 3570 2980 50  0001 C CNN
-F 2 "" H 3570 2830 60  0000 C CNN
+F 2 "Measurement_Points:Measurement_Point_Round-SMD-Pad_Small" H 3570 2830 60  0001 C CNN
 F 3 "" H 3570 2830 60  0000 C CNN
 	1    3570 2830
@@
 P 8500 3070
 F 0 "Q501" V 8830 3070 50  0000 C CNN
-F 1 "BSS83P" V 8730 3070 50  0000 C CNN
+F 1 "DMP3099L-7" V 8730 3070 50  0000 C CNN
 F 2 "Package_TO_SOT_SMD:SOT-23" H 8700 2995 50  0001 L CIN
 F 3 "http://www.farnell.com/datasheets/1835997.pdf" H 8500 3070 50  0001 L CNN
+F 4 "DMP3099L-7DICT-ND" H 8500 3070 50  0001 C CNN "Digi-Key PN"
 	1    8500 3070
 	0    -1   -1   0
@@
 F 0 "R508" H 8420 3760 50  0000 R CNN
 F 1 "10k" V 8500 3760 50  0000 C CNN
-F 2 "" H 8500 3760 50  0001 C CNN
+F 2 "Resistors_SMD:R_0603" H 8500 3760 50  0001 C CNN
 F 3 "" H 8500 3760 50  0001 C CNN
 F 4 "0603" H 8600 3840 50  0000 L CNN "display_footprint"
 F 5 "1%" H 8600 3760 50  0000 L CNN "Tolerance"
 F 6 "1/10W" H 8610 3680 50  0000 L CNN "Wattage"
-F 7 "PN" H 8800 4160 60  0001 C CNN "Digi-Key PN"
+F 7 "RHM10KADCT-ND" H 8800 4160 60  0001 C CNN "Digi-Key PN"
 	1    8500 3760
 	1    0    0    -1
@@
 F 0 "Z501" V 9070 3430 50  0000 C CNN
 F 1 "UDZSTE-175.1B" V 8970 3130 50  0000 R CNN
-F 2 "" H 9070 3230 60  0000 C CNN
+F 2 "Diodes_SMD:D_SOD-523" H 9070 3230 60  0001 C CNN
 F 3 "" H 9070 3230 60  0000 C CNN
 F 4 "UDZSTE-175.1BCT-ND" H 9070 3230 50  0001 C CNN "Digi-Key PN"
@@
 F 0 "R502" H 1110 6950 50  0000 R CNN
 F 1 "3.3k" V 1190 6950 40  0000 C CNN
-F 2 "" H 1190 6950 50  0001 C CNN
+F 2 "Resistors_SMD:R_0603" H 1190 6950 50  0001 C CNN
 F 3 "" H 1190 6950 50  0001 C CNN
 F 4 "0603" H 1290 7030 50  0000 L CNN "display_footprint"
 F 5 "1%" H 1290 6950 50  0000 L CNN "Tolerance"
 F 6 "1/10W" H 1300 6870 50  0000 L CNN "Wattage"
-F 7 "PN" H 1490 7350 60  0001 C CNN "Digi-Key PN"
+F 7 "311-3.30KHRCT-ND" H 1490 7350 60  0001 C CNN "Digi-Key PN"
 	1    1190 6950
 	-1   0    0    -1
@@
 F 0 "R501" H 1110 6310 50  0000 R CNN
 F 1 "10k" V 1190 6310 50  0000 C CNN
-F 2 "" H 1190 6310 50  0001 C CNN
+F 2 "Resistors_SMD:R_0603" H 1190 6310 50  0001 C CNN
 F 3 "" H 1190 6310 50  0001 C CNN
 F 4 "0603" H 1290 6390 50  0000 L CNN "display_footprint"
 F 5 "1%" H 1290 6310 50  0000 L CNN "Tolerance"
 F 6 "1/10W" H 1300 6230 50  0000 L CNN "Wattage"
-F 7 "PN" H 1490 6710 60  0001 C CNN "Digi-Key PN"
+F 7 "RHM10KADCT-ND" H 1490 6710 60  0001 C CNN "Digi-Key PN"
 	1    1190 6310
 	-1   0    0    -1

Commit message: Nailed down board outline, placed a few sections
Parts:
- Q501: footprint Package_TO_SOT_SMD:SOT-23 -> TO_SOT_Packages_SMD:SOT-23
Connections:
- wire segments 57 -> 59
- no-connect marks 1 -> 0
Changed lines of the file:
@@
 Wire Wire Line
 	7620 3170 7540 3170
-NoConn ~ 7540 3070
 $Comp
 L Custom_Library:C_Custom C?
@@
 F 0 "Q501" V 8830 3070 50  0000 C CNN
 F 1 "DMP3099L-7" V 8730 3070 50  0000 C CNN
-F 2 "Package_TO_SOT_SMD:SOT-23" H 8700 2995 50  0001 L CIN
+F 2 "TO_SOT_Packages_SMD:SOT-23" H 8700 2995 50  0001 L CIN
 F 3 "http://www.farnell.com/datasheets/1835997.pdf" H 8500 3070 50  0001 L CNN
 F 4 "DMP3099L-7DICT-ND" H 8500 3070 50  0001 C CNN "Digi-Key PN"
@@
 Wire Wire Line
 	1700 2910 1870 2910
+Wire Wire Line
+	7540 3070 7620 3070
+Wire Wire Line
+	7620 3070 7620 3170
+Connection ~ 7620 3170
 $EndSCHEMATC

Commit message: Finished routing, adding bells and whistles
Parts:
- added TP502: TP, Pin_Headers:Pin_Header_Angled_1x01_Pitch2.54mm, symbol Custom_Library:TP
Changed lines of the file:
@@
 	7620 3070 7620 3170
 Connection ~ 7620 3170
+$Comp
+L power:GND #PWR0524
+U 1 1 5BBBF15B
+P 5440 3300
+F 0 "#PWR0524" H 5440 3050 50  0001 C CNN
+F 1 "GND" H 5440 3150 50  0000 C CNN
+F 2 "" H 5440 3300 50  0001 C CNN
+F 3 "" H 5440 3300 50  0001 C CNN
+	1    5440 3300
+	1    0    0    -1
+$EndComp
+$Comp
+L Custom_Library:TP TP502
+U 1 1 5BBBF1B9
+P 5440 3300
+F 0 "TP502" H 5440 3450 50  0000 C CNN
+F 1 "TP" H 5440 3450 50  0001 C CNN
+F 2 "Pin_Headers:Pin_Header_Angled_1x01_Pitch2.54mm" H 5440 3300 60  0001 C CNN
+F 3 "" H 5440 3300 60  0000 C CNN
+	1    5440 3300
+	1    0    0    -1
+$EndComp
 $EndSCHEMATC

Commit message: Serious BOM scrubbing to drive price down
Parts:
- removed C501, C506: 0.1uF, Capacitors_SMD:C_0603, symbol Custom_Library:C_Custom
- removed C502: 10nF, Capacitors_SMD:C_0603, symbol Custom_Library:C_Custom
- removed C503: 1nF, Capacitors_SMD:C_0603, symbol Custom_Library:C_Custom
- removed R503: 1.4M, Resistors_SMD:R_0603, symbol Custom_Library:R_Custom
- removed R504: 10.5k, Resistors_SMD:R_0603, symbol Custom_Library:R_Custom
- removed R505: 43.2k, Resistors_SMD:R_0603, symbol Custom_Library:R_Custom
- removed R506, R507: 10k, Resistors_SMD:R_0603, symbol Custom_Library:R_Custom
- removed U501: LT6700-1-S6, TO_SOT_Packages_SMD:TSOT-23-6, symbol Custom_Library:LT6700-1-S6
- removed U502: 74LVC1G17, TO_SOT_Packages_SMD:SOT-353_SC-70-5, symbol Custom_Library:74LVC1G17_Power
Connections:
- net labels removed: +3.3V, POS12_PGOOD
- wire segments 59 -> 33
