File: hdw/AC_Power_Meter/USB_UART_Bridge.sch (KiCad schematic (older format))
At the start: 0 parts

Commit message: Populated USB circuit pages
Parts:
- added C? (x5): 0.1uF, symbol Custom_Library:C_Custom
- added C? (x2): 47pF, symbol Custom_Library:C_Custom
- added D?: Yellow, symbol Device:LED_ALT
- added J?: USB_B_Mini, symbol Connector:USB_B_Mini
- added L?: 600R 0.5A, Inductors_SMD:L_0603, symbol Device:Ferrite_Bead
- added R? (x2): 27, Resistors_SMD:R_0603, symbol Device:R
- added R?: 10k, symbol Custom_Library:R_Custom
- added R?: 1k, symbol Custom_Library:R_Custom
- added TP?: TP, Pin_Headers:Pin_Header_Straight_1x01_Pitch2.54mm, symbol Custom_Library:TP
- added TP?: TP, symbol Custom_Library:TP
- added U?: FT234XD, Housings_DFN_QFN:DFN-12-1EP_3x3mm_Pitch0.45mm, symbol Custom_Library:FT234XD
- added U?: TPD3S014DBVR, TO_SOT_Packages_SMD:SOT-23-6, symbol Custom_Library:TPD3S014DBVR
Connections:
- net labels added: +5V_USB, BRIDGE_USB+, BRIDGE_USB-, CONN_USB+, CONN_USB-, GND_USB, USB_UART_RX_ISO, USB_UART_TX_ISO, ~USB_ACTIVE
- wire segments 0 -> 47
- no-connect marks 0 -> 4
Other:
- note added: "UART to USB Bridge"

Commit message: Added zero cross detect circuit
Parts:
- added C? (x2): 0.1uF, symbol Custom_Library:C_Custom
- added C?: 4.7uF, symbol Custom_Library:C_Custom
Changed lines of the file:
@@
 $Descr A 11000 8500
 encoding utf-8
-Sheet 10 13
+Sheet 10 15
 Title ""
 Date ""
@@
 	1    0    0    -1
 $EndComp
+$Comp
+L Custom_Library:C_Custom C?
+U 1 1 5BB2F222
+P 2910 4810
+AR Path="/5BB27BA3/5BB2F222" Ref="C?"  Part="1"
+AR Path="/5BB27B84/5BB2F222" Ref="C?"  Part="1"
+AR Path="/5BB27BCC/5BB2F222" Ref="C?"  Part="1"
+F 0 "C?" H 2935 4910 50  0000 L CNN
+F 1 "0.1uF" H 2935 4710 50  0000 L CNN
+F 2 "" H 2948 4660 50  0001 C CNN
+F 3 "" H 2935 4910 50  0001 C CNN
+F 4 "0603" H 2760 4910 50  0000 R CNN "display_footprint"
+F 5 "50V" H 2760 4810 50  0000 R CNN "Voltage"
+F 6 "X7R" H 2760 4710 50  0000 R CNN "Dielectric"
+F 7 "PN" H 3335 5310 60  0001 C CNN "Digi-Key PN"
+	1    2910 4810
+	1    0    0    -1
+$EndComp
+$Comp
+L Custom_Library:C_Custom C?
+U 1 1 5BB2F482
+P 3540 4800
+AR Path="/5BB27BA3/5BB2F482" Ref="C?"  Part="1"
+AR Path="/5BB27B84/5BB2F482" Ref="C?"  Part="1"
+AR Path="/5BB27BCC/5BB2F482" Ref="C?"  Part="1"
+F 0 "C?" H 3565 4900 50  0000 L CNN
+F 1 "0.1uF" H 3565 4700 50  0000 L CNN
+F 2 "" H 3578 4650 50  0001 C CNN
+F 3 "" H 3565 4900 50  0001 C CNN
+F 4 "0603" H 3390 4900 50  0000 R CNN "display_footprint"
+F 5 "50V" H 3390 4800 50  0000 R CNN "Voltage"
+F 6 "X7R" H 3390 4700 50  0000 R CNN "Dielectric"
+F 7 "PN" H 3965 5300 60  0001 C CNN "Digi-Key PN"
+	1    3540 4800
+	1    0    0    -1
+$EndComp
+$Comp
+L Custom_Library:C_Custom C?
+U 1 1 5BB2F4D0
+P 4170 4790
+AR Path="/5BB27BA3/5BB2F4D0" Ref="C?"  Part="1"
+AR Path="/5BB27B84/5BB2F4D0" Ref="C?"  Part="1"
+AR Path="/5BB27BCC/5BB2F4D0" Ref="C?"  Part="1"
+F 0 "C?" H 4195 4890 50  0000 L CNN
+F 1 "4.7uF" H 4195 4690 50  0000 L CNN
+F 2 "" H 4208 4640 50  0001 C CNN
+F 3 "" H 4195 4890 50  0001 C CNN
+F 4 "0805" H 4020 4890 50  0000 R CNN "display_footprint"
+F 5 "10V" H 4020 4790 50  0000 R CNN "Voltage"
+F 6 "X7R" H 4020 4690 50  0000 R CNN "Dielectric"
+F 7 "PN" H 4595 5290 60  0001 C CNN "Digi-Key PN"
+	1    4170 4790
+	1    0    0    -1
+$EndComp
+$Comp
+L Custom_Library:GND_USB #PWR?
+U 1 1 5BB2F9DC
+P 2910 4960
+F 0 "#PWR?" H 2910 4710 50  0001 C CNN
+F 1 "GND_USB" H 2910 4810 50  0000 C CNN
+F 2 "" H 2910 4960 50  0001 C CNN
+F 3 "" H 2910 4960 50  0001 C CNN
+	1    2910 4960
+	1    0    0    -1
+$EndComp
+$Comp
+L Custom_Library:GND_USB #PWR?
+U 1 1 5BB2FA18
+P 3540 4950
+F 0 "#PWR?" H 3540 4700 50  0001 C CNN
+F 1 "GND_USB" H 3540 4800 50  0000 C CNN
+F 2 "" H 3540 4950 50  0001 C CNN
+F 3 "" H 3540 4950 50  0001 C CNN
+	1    3540 4950
+	1    0    0    -1
+$EndComp
+$Comp
+L Custom_Library:GND_USB #PWR?
+U 1 1 5BB2FA4D
+P 4170 4940
+F 0 "#PWR?" H 4170 4690 50  0001 C CNN
+F 1 "GND_USB" H 4170 4790 50  0000 C CNN
+F 2 "" H 4170 4940 50  0001 C CNN
+F 3 "" H 4170 4940 50  0001 C CNN
+	1    4170 4940
+	1    0    0    -1
+$EndComp
+$Comp
+L Custom_Library:+5V_USB #PWR?
+U 1 1 5BB2FAC3
+P 4170 4640
+F 0 "#PWR?" H 4170 4490 50  0001 C CNN
+F 1 "+5V_USB" H 4170 4780 50  0000 C CNN
+F 2 "" H 4170 4640 50  0001 C CNN
+F 3 "" H 4170 4640 50  0001 C CNN
+	1    4170 4640
+	1    0    0    -1
+$EndComp
+$Comp
+L Custom_Library:+5V_USB #PWR?
+U 1 1 5BB2FAFF
+P 3540 4650
+F 0 "#PWR?" H 3540 4500 50  0001 C CNN
+F 1 "+5V_USB" H 3540 4790 50  0000 C CNN
+F 2 "" H 3540 4650 50  0001 C CNN
+F 3 "" H 3540 4650 50  0001 C CNN
+	1    3540 4650
+	1    0    0    -1
+$EndComp
+$Comp
+L Custom_Library:+5V_USB #PWR?
+U 1 1 5BB2FB34
+P 2910 4660
+F 0 "#PWR?" H 2910 4510 50  0001 C CNN
+F 1 "+5V_USB" H 2910 4800 50  0000 C CNN
+F 2 "" H 2910 4660 50  0001 C CNN
+F 3 "" H 2910 4660 50  0001 C CNN
+	1    2910 4660
+	1    0    0    -1
+$EndComp

Commit message: Added MU logo and titles to all sheets
Parts:
- removed D?: Yellow, symbol Device:LED_ALT
- added C? (x2): 0.1uF, symbol Custom_Library:C_Custom
- added C?: 10nF, symbol Custom_Library:C_Custom
- added C?: 1nF, symbol Custom_Library:C_Custom
- added D?: Green, symbol Custom_Library:LED_ALT_Custom
- added D?: Yellow, symbol Custom_Library:LED_ALT_Custom
- added R?: 6.04k, symbol Custom_Library:R_Custom
- added R?: 40.2k, symbol Custom_Library:R_Custom
- added R?: 487k, symbol Custom_Library:R_Custom
- added R?: 10k, symbol Custom_Library:R_Custom
- added R?: 1k, symbol Custom_Library:R_Custom
- added U?: LT6700-1-S6, TO_SOT_Packages_SMD:TSOT-23-6, symbol Custom_Library:LT6700-1-S6
- added U?: 74LVC1G06, TO_SOT_Packages_SMD:SOT-353_SC-70-5, symbol Custom_Library:74LVC1G06_Power
Connections:
- wire segments 47 -> 72
Other:
- note added: "UART to USB Bridge, +5V USB Window Comparator"
- note removed: "UART to USB Bridge"

Commit message: Updated MU logo to crisper image
Changed lines of the file:
@@
 $EndComp
 $Comp
-L Mu_Logo:LOGO #G?
-U 1 1 5BBF67B7
-P 9900 1000
-F 0 "#G?" H 9900 670 60  0001 C CNN
-F 1 "LOGO" H 9900 1330 60  0001 C CNN
-F 2 "" H 9900 1000 50  0001 C CNN
-F 3 "" H 9900 1000 50  0001 C CNN
-	1    9900 1000
+L Custom_Library:MU_Logo #G?
+U 1 1 5BB69985
+P 9900 1100
+F 0 "#G?" H 9900 614 60  0001 C CNN
+F 1 "MU_Logo" H 9900 1586 60  0001 C CNN
+F 2 "" H 9900 1100 50  0001 C CNN
+F 3 "" H 9900 1100 50  0001 C CNN
+	1    9900 1100
 	1    0    0    -1
 $EndComp

Commit message: Added ORing circuit to TRIAC page
Parts:
- added L?: 600R 0.5A, Inductors_SMD:L_0603, symbol Device:Ferrite_Bead
Connections:
- wire segments 72 -> 76
- no-connect marks 4 -> 3
Changed lines of the file:
@@
 Wire Wire Line
 	8680 2060 8680 2140
-NoConn ~ 9600 3580
 Wire Wire Line
 	8190 2060 8190 2980
@@
 	1    0    0    -1
 $EndComp
+$Comp
+L Device:Ferrite_Bead L?
+U 1 1 5BB59622
+P 9980 3630
+F 0 "L?" V 9830 3655 50  0000 C CNN
+F 1 "600R 0.5A" V 10130 3630 50  0000 C CNN
+F 2 "Inductors_SMD:L_0603" V 9910 3630 50  0001 C CNN
+F 3 "~" H 9980 3630 50  0001 C CNN
+F 4 "732-1593-1-ND" V 9980 3630 50  0001 C CNN "Digi-Key PN"
+	1    9980 3630
+	0    -1   -1   0
+$EndComp
+$Comp
+L Custom_Library:GND_USB #PWR?
+U 1 1 5BB59B66
+P 10210 3710
+F 0 "#PWR?" H 10210 3460 50  0001 C CNN
+F 1 "GND_USB" H 10210 3560 50  0000 C CNN
+F 2 "" H 10210 3710 50  0001 C CNN
+F 3 "" H 10210 3710 50  0001 C CNN
+	1    10210 3710
+	1    0    0    -1
+$EndComp
+Wire Wire Line
+	10210 3710 10210 3630
+Wire Wire Line
+	10210 3630 10130 3630
+Wire Wire Line
+	9830 3630 9600 3630
+Wire Wire Line
+	9600 3630 9600 3580
 $EndSCHEMATC

Commit message: Rewired a few micro symbols, add FMW notes
Parts:
- gave numbers to parts that had none: 34
