File: hdw/AC_Power_Meter/Mechanical.sch (KiCad schematic (older format))
At the start: 0 parts

Commit message: Added AC input and output connections, added mechanical components
Parts:
- added MH? (x8): MountingHole, symbol Mechanical:MountingHole_Pad
- added MK? (x8): 4-40 Standoff, symbol Mechanical:Housing
- added MK? (x8): 4-40 Screw, symbol Mechanical:Housing
Connections:
- net labels added: Earth_Protective

Commit message: Added MU logo and titles to all sheets
Other:
- note added: "Mounting Holes and Mechanical Components"

Commit message: Updated MU logo to crisper image
Changed lines of the file:
@@
 Mounting Holes and Mechanical Components
 $Comp
-L Mu_Logo:LOGO #G?
-U 1 1 5BBF76AD
-P 9900 1000
-F 0 "#G?" H 9900 670 60  0001 C CNN
-F 1 "LOGO" H 9900 1330 60  0001 C CNN
-F 2 "" H 9900 1000 50  0001 C CNN
-F 3 "" H 9900 1000 50  0001 C CNN
-	1    9900 1000
+L Custom_Library:MU_Logo #G?
+U 1 1 5BB6A5D4
+P 9900 1100
+F 0 "#G?" H 9900 614 60  0001 C CNN
+F 1 "MU_Logo" H 9900 1586 60  0001 C CNN
+F 2 "" H 9900 1100 50  0001 C CNN
+F 3 "" H 9900 1100 50  0001 C CNN
+	1    9900 1100
 	1    0    0    -1
 $EndComp

Commit message: Added pushbuttons sheet, prelim wiring on micro
Parts:
- removed MK? (x8): 4-40 Standoff, symbol Mechanical:Housing
- removed MK? (x8): 4-40 Screw, symbol Mechanical:Housing
- added MK? (x8): 4-40 Screw, symbol Custom_Library:Screw
- added MK? (x8): 4-40 Standoff, symbol Custom_Library:Standoff
- added MK?: Housing, symbol Mechanical:Housing
- added MK?: Lid, symbol Mechanical:Housing

Commit message: Rewired a few micro symbols, add FMW notes
Parts:
- gave numbers to parts that had none: 26
Changed lines of the file:
@@
 $Descr A 11000 8500
 encoding utf-8
-Sheet 13 17
+Sheet 13 18
 Title ""
 Date "2018-10-01"
@@
 $EndDescr
 $Comp
-L Mechanical:MountingHole_Pad MH?
+L Mechanical:MountingHole_Pad MH1301
 U 1 1 5BB4FCC8
 P 1490 2140
-F 0 "MH?" H 1490 2390 50  0000 C CNN
+F 0 "MH1301" H 1490 2390 50  0000 C CNN
 F 1 "MountingHole" H 1490 2315 50  0000 C CNN
 F 2 "" H 1490 2140 50  0001 C CNN
@@
 $EndComp
 $Comp
-L power:Earth_Protective #PWR?
+L power:Earth_Protective #PWR01301
 U 1 1 5BB5004B
 P 1490 2240
-F 0 "#PWR?" H 1740 1990 50  0001 C CNN
+F 0 "#PWR01301" H 1740 1990 50  0001 C CNN
 F 1 "Earth_Protective" H 1940 2090 50  0001 C CNN
 F 2 "" H 1490 2140 50  0001 C CNN
@@
 $EndComp
 $Comp
-L Mechanical:MountingHole_Pad MH?
+L Mechanical:MountingHole_Pad MH1303
 U 1 1 5BB5039D
 P 2490 2140
-F 0 "MH?" H 2490 2390 50  0000 C CNN
+F 0 "MH1303" H 2490 2390 50  0000 C CNN
 F 1 "MountingHole" H 2490 2315 50  0000 C CNN
 F 2 "" H 2490 2140 50  0001 C CNN
@@
 $EndComp
 $Comp
-L power:Earth_Protective #PWR?
+L power:Earth_Protective #PWR01303
 U 1 1 5BB503A4
 P 2490 2240
-F 0 "#PWR?" H 2740 1990 50  0001 C CNN
+F 0 "#PWR01303" H 2740 1990 50  0001 C CNN
 F 1 "Earth_Protective" H 2940 2090 50  0001 C CNN
 F 2 "" H 2490 2140 50  0001 C CNN
@@
 $EndComp
 $Comp
-L Mechanical:MountingHole_Pad MH?
+L Mechanical:MountingHole_Pad MH1305
 U 1 1 5BB5043A
 P 3490 2140
-F 0 "MH?" H 3490 2390 50  0000 C CNN
+F 0 "MH1305" H 3490 2390 50  0000 C CNN
 F 1 "MountingHole" H 3490 2315 50  0000 C CNN
 F 2 "" H 3490 2140 50  0001 C CNN
@@
 $EndComp
 $Comp
-L power:Earth_Protective #PWR?
+L power:Earth_Protective #PWR01305
 U 1 1 5BB50441
 P 3490 2240
-F 0 "#PWR?" H 3740 1990 50  0001 C CNN
+F 0 "#PWR01305" H 3740 1990 50  0001 C CNN
 F 1 "Earth_Protective" H 3940 2090 50  0001 C CNN
 F 2 "" H 3490 2140 50  0001 C CNN
@@
 $EndComp
 $Comp
-L Mechanical:MountingHole_Pad MH?
+L Mechanical:MountingHole_Pad MH1307
 U 1 1 5BB50447
 P 4490 2140
-F 0 "MH?" H 4490 2390 50  0000 C CNN
+F 0 "MH1307" H 4490 2390 50  0000 C CNN
 F 1 "MountingHole" H 4490 2315 50  0000 C CNN
 F 2 "" H 4490 2140 50  0001 C CNN
@@
 $EndComp
 $Comp
-L power:Earth_Protective #PWR?
+L power:Earth_Protective #PWR01307
 U 1 1 5BB5044E
 P 4490 2240
-F 0 "#PWR?" H 4740 1990 50  0001 C CNN
+F 0 "#PWR01307" H 4740 1990 50  0001 C CNN
 F 1 "Earth_Protective" H 4940 2090 50  0001 C CNN
 F 2 "" H 4490 2140 50  0001 C CNN
@@
 $EndComp
 $Comp
-L Mechanical:MountingHole_Pad MH?
+L Mechanical:MountingHole_Pad MH1302
 U 1 1 5BB5087C
 P 1490 3140
-F 0 "MH?" H 1490 3390 50  0000 C CNN
+F 0 "MH1302" H 1490 3390 50  0000 C CNN
 F 1 "MountingHole" H 1490 3315 50  0000 C CNN
 F 2 "" H 1490 3140 50  0001 C CNN
@@
 $EndComp
 $Comp
-L power:Earth_Protective #PWR?
+L power:Earth_Protective #PWR01302
 U 1 1 5BB50883
 P 1490 3240
-F 0 "#PWR?" H 1740 2990 50  0001 C CNN
+F 0 "#PWR01302" H 1740 2990 50  0001 C CNN
 F 1 "Earth_Protective" H 1940 3090 50  0001 C CNN
 F 2 "" H 1490 3140 50  0001 C CNN
@@
 $EndComp
 $Comp
-L Mechanical:MountingHole_Pad MH?
+L Mechanical:MountingHole_Pad MH1304
 U 1 1 5BB50889
 P 2490 3140
-F 0 "MH?" H 2490 3390 50  0000 C CNN
+F 0 "MH1304" H 2490 3390 50  0000 C CNN
 F 1 "MountingHole" H 2490 3315 50  0000 C CNN
 F 2 "" H 2490 3140 50  0001 C CNN
@@
 $EndComp
 $Comp
-L power:Earth_Protective #PWR?
+L power:Earth_Protective #PWR01304
 U 1 1 5BB50890
 P 2490 3240
-F 0 "#PWR?" H 2740 2990 50  0001 C CNN
+F 0 "#PWR01304" H 2740 2990 50  0001 C CNN
 F 1 "Earth_Protective" H 2940 3090 50  0001 C CNN
 F 2 "" H 2490 3140 50  0001 C CNN
@@
 $EndComp
 $Comp
-L Mechanical:MountingHole_Pad MH?
+L Mechanical:MountingHole_Pad MH1306
 U 1 1 5BB50896
 P 3490 3140
-F 0 "MH?" H 3490 3390 50  0000 C CNN
+F 0 "MH1306" H 3490 3390 50  0000 C CNN
 F 1 "MountingHole" H 3490 3315 50  0000 C CNN
 F 2 "" H 3490 3140 50  0001 C CNN
@@
 $EndComp
 $Comp
-L power:Earth_Protective #PWR?
+L power:Earth_Protective #PWR01306
 U 1 1 5BB5089D
 P 3490 3240
-F 0 "#PWR?" H 3740 2990 50  0001 C CNN
+F 0 "#PWR01306" H 3740 2990 50  0001 C CNN
 F 1 "Earth_Protective" H 3940 3090 50  0001 C CNN
 F 2 "" H 3490 3140 50  0001 C CNN
@@
 $EndComp
 $Comp
-L Mechanical:MountingHole_Pad MH?
+L Mechanical:MountingHole_Pad MH1308
 U 1 1 5BB508A3
 P 4490 3140
-F 0 "MH?" H 4490 3390 50  0000 C CNN
+F 0 "MH1308" H 4490 3390 50  0000 C CNN
 F 1 "MountingHole" H 4490 3315 50  0000 C CNN
 F 2 "" H 4490 3140 50  0001 C CNN
@@
 $EndComp
 $Comp
-L power:Earth_Protective #PWR?
+L power:Earth_Protective #PWR01308
 U 1 1 5BB508AA
 P 4490 3240
-F 0 "#PWR?" H 4740 2990 50  0001 C CNN
+F 0 "#PWR01308" H 4740 2990 50  0001 C CNN
 F 1 "Earth_Protective" H 4940 3090 50  0001 C CNN
 F 2 "" H 4490 3140 50  0001 C CNN
@@
 Mounting Holes and Mechanical Components
 $Comp
-L Custom_Library:MU_Logo #G?
+L Custom_Library:MU_Logo #G1301
 U 1 1 5BB6A5D4
 P 9900 1100
-F 0 "#G?" H 9900 614 60  0001 C CNN
+F 0 "#G1301" H 9900 614 60  0001 C CNN
 F 1 "MU_Logo" H 9900 1586 60  0001 C CNN
 F 2 "" H 9900 1100 50  0001 C CNN
@@
 $EndComp
 $Comp
-L Custom_Library:Screw MK?
+L Custom_Library:Screw MK1303
 U 1 1 5BC10ED5
 P 6470 2210
-F 0 "MK?" H 6470 2310 50  0000 C CNN
+F 0 "MK1303" H 6470 2310 50  0000 C CNN
 F 1 "4-40 Screw" H 6470 2410 50  0000 C CNN
 F 2 "" H 6470 2460 50  0001 C CNN
@@
 $EndComp
 $Comp
-L Custom_Library:Screw MK?
+L Custom_Library:Screw MK1307
 U 1 1 5BC1118A
 P 7220 2210
-F 0 "MK?" H 7220 2310 50  0000 C CNN
+F 0 "MK1307" H 7220 2310 50  0000 C CNN
 F 1 "4-40 Screw" H 7220 2410 50  0000 C CNN
 F 2 "" H 7220 2460 50  0001 C CNN
@@
 $EndComp
 $Comp
-L Custom_Library:Screw MK?
+L Custom_Library:Screw MK1311
 U 1 1 5BC11270
 P 7970 2210
-F 0 "MK?" H 7970 2310 50  0000 C CNN
+F 0 "MK1311" H 7970 2310 50  0000 C CNN
 F 1 "4-40 Screw" H 7970 2410 50  0000 C CNN
 F 2 "" H 7970 2460 50  0001 C CNN
@@
 $EndComp
 $Comp
-L Custom_Library:Screw MK?
+L Custom_Library:Screw MK1315
 U 1 1 5BC11277
 P 8720 2210
-F 0 "MK?" H 8720 2310 50  0000 C CNN
+F 0 "MK1315" H 8720 2310 50  0000 C CNN
 F 1 "4-40 Screw" H 8720 2410 50  0000 C CNN
 F 2 "" H 8720 2460 50  0001 C CNN
@@
 $EndComp
 $Comp
-L Custom_Library:Screw MK?
+L Custom_Library:Screw MK1304
 U 1 1 5BC113EE
 P 6470 2960
-F 0 "MK?" H 6470 3060 50  0000 C CNN
+F 0 "MK1304" H 6470 3060 50  0000 C CNN
 F 1 "4-40 Screw" H 6470 3160 50  0000 C CNN
 F 2 "" H 6470 3210 50  0001 C CNN
@@
 $EndComp
 $Comp
-L Custom_Library:Screw MK?
+L Custom_Library:Screw MK1308
 U 1 1 5BC113F5
 P 7220 2960
-F 0 "MK?" H 7220 3060 50  0000 C CNN
+F 0 "MK1308" H 7220 3060 50  0000 C CNN
 F 1 "4-40 Screw" H 7220 3160 50  0000 C CNN
 F 2 "" H 7220 3210 50  0001 C CNN
@@
 $EndComp
 $Comp
-L Custom_Library:Screw MK?
+L Custom_Library:Screw MK1312
 U 1 1 5BC113FC
 P 7970 2960
-F 0 "MK?" H 7970 3060 50  0000 C CNN
+F 0 "MK1312" H 7970 3060 50  0000 C CNN
 F 1 "4-40 Screw" H 7970 3160 50  0000 C CNN
 F 2 "" H 7970 3210 50  0001 C CNN
@@
 $EndComp
 $Comp
-L Custom_Library:Screw MK?
+L Custom_Library:Screw MK1316
 U 1 1 5BC11403
 P 8720 2960
-F 0 "MK?" H 8720 3060 50  0000 C CNN
+F 0 "MK1316" H 8720 3060 50  0000 C CNN
 F 1 "4-40 Screw" H 8720 3160 50  0000 C CNN
 F 2 "" H 8720 3210 50  0001 C CNN
@@
 $EndComp
 $Comp
-L Custom_Library:Standoff MK?
+L Custom_Library:Standoff MK1305
 U 1 1 5BC1193F
 P 6470 3720
-F 0 "MK?" H 6470 3870 50  0000 C CNN
+F 0 "MK1305" H 6470 3870 50  0000 C CNN
 F 1 "4-40 Standoff" H 6470 3970 50  0000 C CNN
 F 2 "" H 6470 4070 50  0001 C CNN
@@
 $EndComp
 $Comp
-L Custom_Library:Standoff MK?
+L Custom_Library:Standoff MK1309
 U 1 1 5BC12310
 P 7220 3720
-F 0 "MK?" H 7220 3870 50  0000 C CNN
+F 0 "MK1309" H 7220 3870 50  0000 C CNN
 F 1 "4-40 Standoff" H 7220 3970 50  0000 C CNN
 F 2 "" H 7220 4070 50  0001 C CNN
@@
 $EndComp
 $Comp
-L Custom_Library:Standoff MK?
+L Custom_Library:Standoff MK1313
 U 1 1 5BC1235A
 P 7970 3720
-F 0 "MK?" H 7970 3870 50  0000 C CNN
+F 0 "MK1313" H 7970 3870 50  0000 C CNN
 F 1 "4-40 Standoff" H 7970 3970 50  0000 C CNN
 F 2 "" H 7970 4070 50  0001 C CNN
@@
 $EndComp
 $Comp
-L Custom_Library:Standoff MK?
+L Custom_Library:Standoff MK1317
 U 1 1 5BC123B2
 P 8720 3720
-F 0 "MK?" H 8720 3870 50  0000 C CNN
+F 0 "MK1317" H 8720 3870 50  0000 C CNN
 F 1 "4-40 Standoff" H 8720 3970 50  0000 C CNN
 F 2 "" H 8720 4070 50  0001 C CNN
@@
 $EndComp
 $Comp
-L Custom_Library:Standoff MK?
+L Custom_Library:Standoff MK1306
 U 1 1 5BC12534
 P 6470 4470
-F 0 "MK?" H 6470 4620 50  0000 C CNN
+F 0 "MK1306" H 6470 4620 50  0000 C CNN
 F 1 "4-40 Standoff" H 6470 4720 50  0000 C CNN
 F 2 "" H 6470 4820 50  0001 C CNN
@@
 $EndComp
 $Comp
-L Custom_Library:Standoff MK?
+L Custom_Library:Standoff MK1310
 U 1 1 5BC1253B
 P 7220 4470
-F 0 "MK?" H 7220 4620 50  0000 C CNN
+F 0 "MK1310" H 7220 4620 50  0000 C CNN
 F 1 "4-40 Standoff" H 7220 4720 50  0000 C CNN
 F 2 "" H 7220 4820 50  0001 C CNN
@@
 $EndComp
 $Comp
-L Custom_Library:Standoff MK?
+L Custom_Library:Standoff MK1314
 U 1 1 5BC12542
 P 7970 4470
-F 0 "MK?" H 7970 4620 50  0000 C CNN
+F 0 "MK1314" H 7970 4620 50  0000 C CNN
 F 1 "4-40 Standoff" H 7970 4720 50  0000 C CNN
 F 2 "" H 7970 4820 50  0001 C CNN
@@
 $EndComp
 $Comp
-L Custom_Library:Standoff MK?
+L Custom_Library:Standoff MK1318
 U 1 1 5BC12549
 P 8720 4470
-F 0 "MK?" H 8720 4620 50  0000 C CNN
+F 0 "MK1318" H 8720 4620 50  0000 C CNN
 F 1 "4-40 Standoff" H 8720 4720 50  0000 C CNN
 F 2 "" H 8720 4820 50  0001 C CNN
@@
 $EndComp
 $Comp
-L Mechanical:Housing MK?
+L Mechanical:Housing MK1301
 U 1 1 5BC1C7F0
 P 2840 5410
-F 0 "MK?" H 2990 5410 50  0000 L CNN
+F 0 "MK1301" H 2990 5410 50  0000 L CNN
 F 1 "Housing" H 2990 5335 50  0000 L CNN
 F 2 "" H 2890 5460 50  0001 C CNN
@@
 $EndComp
 $Comp
-L Mechanical:Housing MK?
+L Mechanical:Housing MK1302
 U 1 1 5BC1D3DD
 P 4090 5410
-F 0 "MK?" H 4240 5410 50  0000 L CNN
+F 0 "MK1302" H 4240 5410 50  0000 L CNN
 F 1 "Lid" H 4240 5335 50  0000 L CNN
 F 2 "" H 4140 5460 50  0001 C CNN

Commit message: Updated most footprints
Parts:
- MH1301, MH1302, MH1303, MH1304, MH1305, MH1306, MH1307, MH1308: footprint (none) -> Mounting_Holes:MountingHole_3mm_Pad_Via
- MK1303, MK1304, MK1307, MK1308, MK1311, MK1312, MK1315, MK1316: Digi-Key PN (none) -> 36-9900-ND
- MK1305, MK1306, MK1309, MK1310, MK1313, MK1314, MK1317, MK1318: Digi-Key PN (none) -> 36-8400-ND
Changed lines of the file:
@@
 F 0 "MH1301" H 1490 2390 50  0000 C CNN
 F 1 "MountingHole" H 1490 2315 50  0000 C CNN
-F 2 "" H 1490 2140 50  0001 C CNN
+F 2 "Mounting_Holes:MountingHole_3mm_Pad_Via" H 1490 2140 50  0001 C CNN
 F 3 "~" H 1490 2140 50  0001 C CNN
 	1    1490 2140
@@
 F 0 "MH1303" H 2490 2390 50  0000 C CNN
 F 1 "MountingHole" H 2490 2315 50  0000 C CNN
-F 2 "" H 2490 2140 50  0001 C CNN
+F 2 "Mounting_Holes:MountingHole_3mm_Pad_Via" H 2490 2140 50  0001 C CNN
 F 3 "~" H 2490 2140 50  0001 C CNN
 	1    2490 2140
@@
 F 0 "MH1305" H 3490 2390 50  0000 C CNN
 F 1 "MountingHole" H 3490 2315 50  0000 C CNN
-F 2 "" H 3490 2140 50  0001 C CNN
+F 2 "Mounting_Holes:MountingHole_3mm_Pad_Via" H 3490 2140 50  0001 C CNN
 F 3 "~" H 3490 2140 50  0001 C CNN
 	1    3490 2140
@@
 F 0 "MH1307" H 4490 2390 50  0000 C CNN
 F 1 "MountingHole" H 4490 2315 50  0000 C CNN
-F 2 "" H 4490 2140 50  0001 C CNN
+F 2 "Mounting_Holes:MountingHole_3mm_Pad_Via" H 4490 2140 50  0001 C CNN
 F 3 "~" H 4490 2140 50  0001 C CNN
 	1    4490 2140
@@
 F 0 "MH1302" H 1490 3390 50  0000 C CNN
 F 1 "MountingHole" H 1490 3315 50  0000 C CNN
-F 2 "" H 1490 3140 50  0001 C CNN
+F 2 "Mounting_Holes:MountingHole_3mm_Pad_Via" H 1490 3140 50  0001 C CNN
 F 3 "~" H 1490 3140 50  0001 C CNN
 	1    1490 3140
@@
 F 0 "MH1304" H 2490 3390 50  0000 C CNN
 F 1 "MountingHole" H 2490 3315 50  0000 C CNN
-F 2 "" H 2490 3140 50  0001 C CNN
+F 2 "Mounting_Holes:MountingHole_3mm_Pad_Via" H 2490 3140 50  0001 C CNN
 F 3 "~" H 2490 3140 50  0001 C CNN
 	1    2490 3140
@@
 F 0 "MH1306" H 3490 3390 50  0000 C CNN
 F 1 "MountingHole" H 3490 3315 50  0000 C CNN
-F 2 "" H 3490 3140 50  0001 C CNN
+F 2 "Mounting_Holes:MountingHole_3mm_Pad_Via" H 3490 3140 50  0001 C CNN
 F 3 "~" H 3490 3140 50  0001 C CNN
 	1    3490 3140
@@
 F 0 "MH1308" H 4490 3390 50  0000 C CNN
 F 1 "MountingHole" H 4490 3315 50  0000 C CNN
-F 2 "" H 4490 3140 50  0001 C CNN
+F 2 "Mounting_Holes:MountingHole_3mm_Pad_Via" H 4490 3140 50  0001 C CNN
 F 3 "~" H 4490 3140 50  0001 C CNN
 	1    4490 3140
@@
 F 2 "" H 6470 2460 50  0001 C CNN
 F 3 "" H 6470 2460 50  0001 C CNN
+F 4 "36-9900-ND" H 0   0   50  0001 C CNN "Digi-Key PN"
 	1    6470 2210
 	1    0    0    -1
@@
 F 2 "" H 7220 2460 50  0001 C CNN
 F 3 "" H 7220 2460 50  0001 C CNN
+F 4 "36-9900-ND" H 0   0   50  0001 C CNN "Digi-Key PN"
 	1    7220 2210
 	1    0    0    -1
@@
 F 2 "" H 7970 2460 50  0001 C CNN
 F 3 "" H 7970 2460 50  0001 C CNN
+F 4 "36-9900-ND" H 0   0   50  0001 C CNN "Digi-Key PN"
 	1    7970 2210
 	1    0    0    -1
@@
 F 2 "" H 8720 2460 50  0001 C CNN
 F 3 "" H 8720 2460 50  0001 C CNN
+F 4 "36-9900-ND" H 0   0   50  0001 C CNN "Digi-Key PN"
 	1    8720 2210
 	1    0    0    -1
@@
 F 2 "" H 6470 3210 50  0001 C CNN
 F 3 "" H 6470 3210 50  0001 C CNN
+F 4 "36-9900-ND" H 0   0   50  0001 C CNN "Digi-Key PN"
 	1    6470 2960
 	1    0    0    -1
@@
 F 2 "" H 7220 3210 50  0001 C CNN
 F 3 "" H 7220 3210 50  0001 C CNN
+F 4 "36-9900-ND" H 0   0   50  0001 C CNN "Digi-Key PN"
 	1    7220 2960
 	1    0    0    -1
@@
 F 2 "" H 7970 3210 50  0001 C CNN
 F 3 "" H 7970 3210 50  0001 C CNN
+F 4 "36-9900-ND" H 0   0   50  0001 C CNN "Digi-Key PN"
 	1    7970 2960
 	1    0    0    -1
@@
 F 2 "" H 8720 3210 50  0001 C CNN
 F 3 "" H 8720 3210 50  0001 C CNN
+F 4 "36-9900-ND" H 0   0   50  0001 C CNN "Digi-Key PN"
 	1    8720 2960
 	1    0    0    -1
@@
 F 2 "" H 6470 4070 50  0001 C CNN
 F 3 "" H 6470 4070 50  0001 C CNN
+F 4 "36-8400-ND" H 0   0   50  0001 C CNN "Digi-Key PN"
 	1    6470 3720
 	1    0    0    -1
@@
 F 2 "" H 7220 4070 50  0001 C CNN
 F 3 "" H 7220 4070 50  0001 C CNN
+F 4 "36-8400-ND" H 0   0   50  0001 C CNN "Digi-Key PN"
 	1    7220 3720
 	1    0    0    -1
@@
 F 2 "" H 7970 4070 50  0001 C CNN
 F 3 "" H 7970 4070 50  0001 C CNN
+F 4 "36-8400-ND" H 0   0   50  0001 C CNN "Digi-Key PN"
 	1    7970 3720
 	1    0    0    -1
@@
 F 2 "" H 8720 4070 50  0001 C CNN
 F 3 "" H 8720 4070 50  0001 C CNN
+F 4 "36-8400-ND" H 0   0   50  0001 C CNN "Digi-Key PN"
 	1    8720 3720
 	1    0    0    -1
@@
 F 2 "" H 6470 4820 50  0001 C CNN
 F 3 "" H 6470 4820 50  0001 C CNN
+F 4 "36-8400-ND" H 0   0   50  0001 C CNN "Digi-Key PN"
 	1    6470 4470
 	1    0    0    -1
@@
 F 2 "" H 7220 4820 50  0001 C CNN
 F 3 "" H 7220 4820 50  0001 C CNN
+F 4 "36-8400-ND" H 0   0   50  0001 C CNN "Digi-Key PN"
 	1    7220 4470
 	1    0    0    -1
@@
 F 2 "" H 7970 4820 50  0001 C CNN
 F 3 "" H 7970 4820 50  0001 C CNN
+F 4 "36-8400-ND" H 0   0   50  0001 C CNN "Digi-Key PN"
 	1    7970 4470
 	1    0    0    -1
@@
 F 2 "" H 8720 4820 50  0001 C CNN
 F 3 "" H 8720 4820 50  0001 C CNN
+F 4 "36-8400-ND" H 0   0   50  0001 C CNN "Digi-Key PN"
 	1    8720 4470
 	1    0    0    -1
