File: hdw/AC_Power_Meter/Mechanical.sch (KiCad schematic (older format))
At the start: 26 parts

Commit message: Nailed down board outline, placed a few sections
Parts:
- removed MH1301, MH1302, MH1303, MH1304, MH1305, MH1306, MH1307, MH1308: MountingHole, Mounting_Holes:MountingHole_3mm_Pad_Via, symbol Mechanical:MountingHole_Pad
- added MH1301, MH1302, MH1303, MH1305, MH1306, MH1307, MH1308: MountingHole, Mounting_Holes:MountingHole_3mm, symbol Mechanical:MountingHole
Connections:
- net labels removed: Earth_Protective
Changed lines of the file:
@@
 Comment4 ""
 $EndDescr
-$Comp
-L Mechanical:MountingHole_Pad MH1301
-U 1 1 5BB4FCC8
-P 1490 2140
-F 0 "MH1301" H 1490 2390 50  0000 C CNN
-F 1 "MountingHole" H 1490 2315 50  0000 C CNN
-F 2 "Mounting_Holes:MountingHole_3mm_Pad_Via" H 1490 2140 50  0001 C CNN
-F 3 "~" H 1490 2140 50  0001 C CNN
-	1    1490 2140
-	1    0    0    -1
-$EndComp
-$Comp
-L power:Earth_Protective #PWR01301
-U 1 1 5BB5004B
-P 1490 2240
-F 0 "#PWR01301" H 1740 1990 50  0001 C CNN
-F 1 "Earth_Protective" H 1940 2090 50  0001 C CNN
-F 2 "" H 1490 2140 50  0001 C CNN
-F 3 "~" H 1490 2140 50  0001 C CNN
-	1    1490 2240
-	1    0    0    -1
-$EndComp
-$Comp
-L Mechanical:MountingHole_Pad MH1303
-U 1 1 5BB5039D
-P 2490 2140
-F 0 "MH1303" H 2490 2390 50  0000 C CNN
-F 1 "MountingHole" H 2490 2315 50  0000 C CNN
-F 2 "Mounting_Holes:MountingHole_3mm_Pad_Via" H 2490 2140 50  0001 C CNN
-F 3 "~" H 2490 2140 50  0001 C CNN
-	1    2490 2140
-	1    0    0    -1
-$EndComp
-$Comp
-L power:Earth_Protective #PWR01303
-U 1 1 5BB503A4
-P 2490 2240
-F 0 "#PWR01303" H 2740 1990 50  0001 C CNN
-F 1 "Earth_Protective" H 2940 2090 50  0001 C CNN
-F 2 "" H 2490 2140 50  0001 C CNN
-F 3 "~" H 2490 2140 50  0001 C CNN
-	1    2490 2240
-	1    0    0    -1
-$EndComp
-$Comp
-L Mechanical:MountingHole_Pad MH1305
-U 1 1 5BB5043A
-P 3490 2140
-F 0 "MH1305" H 3490 2390 50  0000 C CNN
-F 1 "MountingHole" H 3490 2315 50  0000 C CNN
-F 2 "Mounting_Holes:MountingHole_3mm_Pad_Via" H 3490 2140 50  0001 C CNN
-F 3 "~" H 3490 2140 50  0001 C CNN
-	1    3490 2140
-	1    0    0    -1
-$EndComp
-$Comp
-L power:Earth_Protective #PWR01305
-U 1 1 5BB50441
-P 3490 2240
-F 0 "#PWR01305" H 3740 1990 50  0001 C CNN
-F 1 "Earth_Protective" H 3940 2090 50  0001 C CNN
-F 2 "" H 3490 2140 50  0001 C CNN
-F 3 "~" H 3490 2140 50  0001 C CNN
-	1    3490 2240
-	1    0    0    -1
-$EndComp
-$Comp
-L Mechanical:MountingHole_Pad MH1307
-U 1 1 5BB50447
-P 4490 2140
-F 0 "MH1307" H 4490 2390 50  0000 C CNN
-F 1 "MountingHole" H 4490 2315 50  0000 C CNN
-F 2 "Mounting_Holes:MountingHole_3mm_Pad_Via" H 4490 2140 50  0001 C CNN
-F 3 "~" H 4490 2140 50  0001 C CNN
-	1    4490 2140
-	1    0    0    -1
-$EndComp
-$Comp
-L power:Earth_Protective #PWR01307
-U 1 1 5BB5044E
-P 4490 2240
-F 0 "#PWR01307" H 4740 1990 50  0001 C CNN
-F 1 "Earth_Protective" H 4940 2090 50  0001 C CNN
-F 2 "" H 4490 2140 50  0001 C CNN
-F 3 "~" H 4490 2140 50  0001 C CNN
-	1    4490 2240
-	1    0    0    -1
-$EndComp
-$Comp
-L Mechanical:MountingHole_Pad MH1302
-U 1 1 5BB5087C
-P 1490 3140
-F 0 "MH1302" H 1490 3390 50  0000 C CNN
-F 1 "MountingHole" H 1490 3315 50  0000 C CNN
-F 2 "Mounting_Holes:MountingHole_3mm_Pad_Via" H 1490 3140 50  0001 C CNN
-F 3 "~" H 1490 3140 50  0001 C CNN
-	1    1490 3140
-	1    0    0    -1
-$EndComp
-$Comp
-L power:Earth_Protective #PWR01302
-U 1 1 5BB50883
-P 1490 3240
-F 0 "#PWR01302" H 1740 2990 50  0001 C CNN
-F 1 "Earth_Protective" H 1940 3090 50  0001 C CNN
-F 2 "" H 1490 3140 50  0001 C CNN
-F 3 "~" H 1490 3140 50  0001 C CNN
-	1    1490 3240
-	1    0    0    -1
-$EndComp
-$Comp
-L Mechanical:MountingHole_Pad MH1304
-U 1 1 5BB50889
-P 2490 3140
-F 0 "MH1304" H 2490 3390 50  0000 C CNN
-F 1 "MountingHole" H 2490 3315 50  0000 C CNN
-F 2 "Mounting_Holes:MountingHole_3mm_Pad_Via" H 2490 3140 50  0001 C CNN
-F 3 "~" H 2490 3140 50  0001 C CNN
-	1    2490 3140
-	1    0    0    -1
-$EndComp
-$Comp
-L power:Earth_Protective #PWR01304
-U 1 1 5BB50890
-P 2490 3240
-F 0 "#PWR01304" H 2740 2990 50  0001 C CNN
-F 1 "Earth_Protective" H 2940 3090 50  0001 C CNN
-F 2 "" H 2490 3140 50  0001 C CNN
-F 3 "~" H 2490 3140 50  0001 C CNN
-	1    2490 3240
-	1    0    0    -1
-$EndComp
-$Comp
-L Mechanical:MountingHole_Pad MH1306
-U 1 1 5BB50896
-P 3490 3140
-F 0 "MH1306" H 3490 3390 50  0000 C CNN
-F 1 "MountingHole" H 3490 3315 50  0000 C CNN
-F 2 "Mounting_Holes:MountingHole_3mm_Pad_Via" H 3490 3140 50  0001 C CNN
-F 3 "~" H 3490 3140 50  0001 C CNN
-	1    3490 3140
-	1    0    0    -1
-$EndComp
-$Comp
-L power:Earth_Protective #PWR01306
-U 1 1 5BB5089D
-P 3490 3240
-F 0 "#PWR01306" H 3740 2990 50  0001 C CNN
-F 1 "Earth_Protective" H 3940 3090 50  0001 C CNN
-F 2 "" H 3490 3140 50  0001 C CNN
-F 3 "~" H 3490 3140 50  0001 C CNN
-	1    3490 3240
-	1    0    0    -1
-$EndComp
-$Comp
-L Mechanical:MountingHole_Pad MH1308
-U 1 1 5BB508A3
-P 4490 3140
-F 0 "MH1308" H 4490 3390 50  0000 C CNN
-F 1 "MountingHole" H 4490 3315 50  0000 C CNN
-F 2 "Mounting_Holes:MountingHole_3mm_Pad_Via" H 4490 3140 50  0001 C CNN
-F 3 "~" H 4490 3140 50  0001 C CNN
-	1    4490 3140
-	1    0    0    -1
-$EndComp
-$Comp
-L power:Earth_Protective #PWR01308
-U 1 1 5BB508AA
-P 4490 3240
-F 0 "#PWR01308" H 4740 2990 50  0001 C CNN
-F 1 "Earth_Protective" H 4940 3090 50  0001 C CNN
-F 2 "" H 4490 3140 50  0001 C CNN
-F 3 "~" H 4490 3140 50  0001 C CNN
-	1    4490 3240
-	1    0    0    -1
-$EndComp
 Text Notes 540  690  0    100  ~ 20
 Mounting Holes and Mechanical Components
@@
 	1    0    0    -1
 $EndComp
+$Comp
+L Mechanical:MountingHole MH1301
+U 1 1 5BB9BDFA
+P 1320 1940
+F 0 "MH1301" H 1320 2140 50  0000 C CNN
+F 1 "MountingHole" H 1320 2065 50  0000 C CNN
+F 2 "Mounting_Holes:MountingHole_3mm" H 1320 1940 50  0001 C CNN
+F 3 "~" H 1320 1940 50  0001 C CNN
+	1    1320 1940
+	1    0    0    -1
+$EndComp
+$Comp
+L Mechanical:MountingHole MH1303
+U 1 1 5BB9BE84
+P 2070 1940
+F 0 "MH1303" H 2070 2140 50  0000 C CNN
+F 1 "MountingHole" H 2070 2065 50  0000 C CNN
+F 2 "Mounting_Holes:MountingHole_3mm" H 2070 1940 50  0001 C CNN
+F 3 "~" H 2070 1940 50  0001 C CNN
+	1    2070 1940
+	1    0    0    -1
+$EndComp
+$Comp
+L Mechanical:MountingHole MH1305
+U 1 1 5BB9BEE2
+P 2820 1940
+F 0 "MH1305" H 2820 2140 50  0000 C CNN
+F 1 "MountingHole" H 2820 2065 50  0000 C CNN
+F 2 "Mounting_Holes:MountingHole_3mm" H 2820 1940 50  0001 C CNN
+F 3 "~" H 2820 1940 50  0001 C CNN
+	1    2820 1940
+	1    0    0    -1
+$EndComp
+$Comp
+L Mechanical:MountingHole MH1307
+U 1 1 5BB9BF36
+P 3570 1940
+F 0 "MH1307" H 3570 2140 50  0000 C CNN
+F 1 "MountingHole" H 3570 2065 50  0000 C CNN
+F 2 "Mounting_Holes:MountingHole_3mm" H 3570 1940 50  0001 C CNN
+F 3 "~" H 3570 1940 50  0001 C CNN
+	1    3570 1940
+	1    0    0    -1
+$EndComp
+$Comp
+L Mechanical:MountingHole MH1302
+U 1 1 5BB9C02C
+P 1320 2450
+F 0 "MH1302" H 1320 2650 50  0000 C CNN
+F 1 "MountingHole" H 1320 2575 50  0000 C CNN
+F 2 "Mounting_Holes:MountingHole_3mm" H 1320 2450 50  0001 C CNN
+F 3 "~" H 1320 2450 50  0001 C CNN
+	1    1320 2450
+	1    0    0    -1
+$EndComp
+$Comp
+L Mechanical:MountingHole MH1306
+U 1 1 5BB9C03A
+P 2820 2450
+F 0 "MH1306" H 2820 2650 50  0000 C CNN
+F 1 "MountingHole" H 2820 2575 50  0000 C CNN
+F 2 "Mounting_Holes:MountingHole_3mm" H 2820 2450 50  0001 C CNN
+F 3 "~" H 2820 2450 50  0001 C CNN
+	1    2820 2450
+	1    0    0    -1
+$EndComp
+$Comp
+L Mechanical:MountingHole MH1308
+U 1 1 5BB9C041
+P 3570 2450
+F 0 "MH1308" H 3570 2650 50  0000 C CNN
+F 1 "MountingHole" H 3570 2575 50  0000 C CNN
+F 2 "Mounting_Holes:MountingHole_3mm" H 3570 2450 50  0001 C CNN
+F 3 "~" H 3570 2450 50  0001 C CNN
+	1    3570 2450
+	1    0    0    -1
+$EndComp

Commit message: Made a fw minor adjustments to PCB
Parts:
- removed MK1308: 4-40 Screw, symbol Custom_Library:Screw
- removed MK1310: 4-40 Standoff, symbol Custom_Library:Standoff
Changed lines of the file:
@@
-$EndComp
-$Comp
-L Custom_Library:Screw MK1308
-U 1 1 5BC113F5
-P 7220 2960
-F 0 "MK1308" H 7220 3060 50  0000 C CNN
-F 1 "4-40 Screw" H 7220 3160 50  0000 C CNN
-F 2 "" H 7220 3210 50  0001 C CNN
-F 3 "" H 7220 3210 50  0001 C CNN
-F 4 "36-9900-ND" H 0   0   50  0001 C CNN "Digi-Key PN"
-	1    7220 2960
-	1    0    0    -1
 $EndComp
 $Comp
@@
 	1    0    0    -1
 $EndComp
-$Comp
-L Custom_Library:Standoff MK1310
-U 1 1 5BC1253B
-P 7220 4470
-F 0 "MK1310" H 7220 4620 50  0000 C CNN
-F 1 "4-40 Standoff" H 7220 4720 50  0000 C CNN
-F 2 "" H 7220 4820 50  0001 C CNN
-F 3 "" H 7220 4820 50  0001 C CNN
-F 4 "36-8400-ND" H 0   0   50  0001 C CNN "Digi-Key PN"
-	1    7220 4470
-	1    0    0    -1
-$EndComp
