File: hdw/AC_Power_Meter/Microcontroller.sch (KiCad schematic (older format))
At the start: 7 parts

Commit message: Added +3.3V power supply, +12V window comparator, a few design files
Connections:
- net labels added: USB_UART_RX, USB_UART_TX
Changed lines of the file:
@@
 $Descr A 11000 8500
 encoding utf-8
-Sheet 7 15
+Sheet 7 16
 Title ""
 Date "2018-10-01"
@@
 Wire Wire Line
 	3530 7090 3530 7050
+Text GLabel 6580 4390 2    60   Output ~ 0
+USB_UART_TX
+Text GLabel 6580 4290 2    60   Input ~ 0
+USB_UART_RX
 $EndSCHEMATC

Commit message: Added MU logo and titles to all sheets
Other:
- note added: "8 bit High Performance Enhanced Flash PIC Microcontroller"
Changed lines of the file:
@@
 Text GLabel 6580 4290 2    60   Input ~ 0
 USB_UART_RX
+Text Notes 540  690  0    100  ~ 20
+8 bit High Performance Enhanced Flash PIC Microcontroller
+$Comp
+L Mu_Logo:LOGO #G?
+U 1 1 5BBF3BA6
+P 9900 1000
+F 0 "#G?" H 9900 670 60  0001 C CNN
+F 1 "LOGO" H 9900 1330 60  0001 C CNN
+F 2 "" H 9900 1000 50  0001 C CNN
+F 3 "" H 9900 1000 50  0001 C CNN
+	1    9900 1000
+	1    0    0    -1
+$EndComp
 $EndSCHEMATC

Commit message: Updated MU logo to crisper image
Changed lines of the file:
@@
 8 bit High Performance Enhanced Flash PIC Microcontroller
 $Comp
-L Mu_Logo:LOGO #G?
-U 1 1 5BBF3BA6
-P 9900 1000
-F 0 "#G?" H 9900 670 60  0001 C CNN
-F 1 "LOGO" H 9900 1330 60  0001 C CNN
-F 2 "" H 9900 1000 50  0001 C CNN
-F 3 "" H 9900 1000 50  0001 C CNN
-	1    9900 1000
+L Custom_Library:MU_Logo #G?
+U 1 1 5BB68D1E
+P 9900 1100
+F 0 "#G?" H 9900 614 60  0001 C CNN
+F 1 "MU_Logo" H 9900 1586 60  0001 C CNN
+F 2 "" H 9900 1100 50  0001 C CNN
+F 3 "" H 9900 1100 50  0001 C CNN
+	1    9900 1100
 	1    0    0    -1
 $EndComp

Commit message: Revised signal conditioning, cleaned up a lot of pages
Parts:
- added C?: 47uF, symbol Custom_Library:CP_Tant_Custom
- added C?: 0.1uF, symbol Custom_Library:C_Custom
- added C?: 10nF, symbol Custom_Library:C_Custom
- added C?: 1nF, symbol Custom_Library:C_Custom
- added R? (x3): 10k, symbol Custom_Library:R_Custom
- added R? (x2): 0, Resistors_SMD:R_0603, symbol Device:R
- added X?: ASV-16.000MHz, Oscillator:Oscillator_SMD_Abracon_ASV-4Pin_7.0x5.1mm, symbol Oscillator:ASV-xxxMHz
Connections:
- net labels added: ADC_Error, CLKIN, Comm_Error, Heartbeat, I2C_SCL, I2C_SDA, ISNS_ADC, POS12_PGOOD, POS3P3_PGOOD, SSR_Dim, SSR_Force, Zero_Cross_Detect, ~Reset
- wire segments 34 -> 54

Commit message: Added pushbuttons sheet, prelim wiring on micro
Parts:
- U?: value PIC18LF67K40-I_PT -> PIC18LF67K40-I/PT
Connections:
- net labels added: Active, POS12_ADC, POS3P3_ADC, Sleep
- net labels removed: ~Reset
Changed lines of the file:
@@
 $Descr A 11000 8500
 encoding utf-8
-Sheet 7 16
+Sheet 7 17
 Title ""
 Date "2018-10-01"
@@
 P 5330 3640
 F 0 "U?" H 6380 1840 50  0000 R CNN
-F 1 "PIC18LF67K40-I_PT" H 5330 3690 50  0000 C CNN
+F 1 "PIC18LF67K40-I/PT" H 5330 3690 50  0000 C CNN
 F 2 "Housings_QFP:TQFP-64_10x10mm_Pitch0.5mm" H 5330 5740 50  0001 C CNN
 F 3 "" H 4680 4290 50  0001 C CNN
@@
 	1    0    0    -1
 $EndComp
-Text GLabel 1090 2160 2    50   Output ~ 0
+Text GLabel 4080 4190 0    50   Input ~ 0
 POS12_PGOOD
-Text GLabel 1590 2390 0    50   Output ~ 0
+Text GLabel 4080 4390 0    50   Input ~ 0
 POS3P3_PGOOD
-Text GLabel 1090 2890 2    50   Output ~ 0
+Text GLabel 4080 1890 0    50   Input ~ 0
 ISNS_ADC
 $Comp
@@
 Text GLabel 4080 2790 0    50   Input ~ 0
 Zero_Cross_Detect
-Text GLabel 2960 1990 0    50   Input ~ 0
+Text GLabel 6580 3690 2    50   Output ~ 0
 SSR_Force
-Text GLabel 2960 2090 0    50   Input ~ 0
+Text GLabel 6580 3790 2    50   Output ~ 0
 SSR_Dim
-Text GLabel 8630 1880 0    50   Input ~ 0
-~Reset
-Text GLabel 8630 4520 0    50   Input ~ 0
+Text GLabel 6580 2790 2    50   Output ~ 0
+Active
+Text GLabel 6580 2890 2    50   Output ~ 0
 Comm_Error
-Text GLabel 8640 2590 0    50   Input ~ 0
+Text GLabel 6580 2990 2    50   Output ~ 0
 Heartbeat
-Text GLabel 8450 3110 0    50   Input ~ 0
+Text GLabel 6580 3090 2    50   Output ~ 0
 ADC_Error
 Wire Wire Line
@@
 U 1 1 5BBF0F15
 P 4950 6890
+AR Path="/5BB27B51/5BBF0F15" Ref="C?"  Part="1"
+AR Path="/5BB27B84/5BBF0F15" Ref="C?"  Part="1"
 F 0 "C?" H 4975 6990 50  0000 L CNN
 F 1 "47uF" H 4975 6790 50  0000 L CNN
@@
 Text GLabel 4080 2590 0    50   Input ~ 0
 CLKIN
+Text GLabel 4080 4290 0    50   Input ~ 0
+POS3P3_ADC
+Text GLabel 4080 4090 0    50   Input ~ 0
+POS12_ADC
+Text GLabel 4080 2890 0    50   Input ~ 0
+Sleep
 $EndSCHEMATC

Commit message: Rewired a few micro symbols, add FMW notes
Parts:
- gave numbers to parts that had none: 17
Connections:
- net labels added: +3.3VADC, GNDA, SW_Toggle, ~Active
- net labels removed: Active, Sleep
- no-connect marks 0 -> 37

Commit message: Updated most footprints
Parts:
- C701, C704, C708: footprint (none) -> Capacitors_SMD:C_0603; Digi-Key PN PN -> 490-8020-1-ND
- C702, C705, C709: footprint (none) -> Capacitors_SMD:C_0603; Digi-Key PN PN -> 1276-1921-1-ND
- C703, C706, C710: footprint (none) -> Capacitors_SMD:C_0603; Digi-Key PN PN -> 478-1215-1-ND
- C707: footprint (none) -> Capacitors_Tantalum_SMD:CP_Tantalum_Case-X_EIA-7343-43_Reflow
- R701, R702: Digi-Key PN (none) -> P0.0GCT-ND
- R703, R704, R705: footprint (none) -> Resistors_SMD:R_0603; Digi-Key PN PN -> RHM10KADCT-ND
- U701: Digi-Key PN (none) -> PIC18LF67K40-I/PT-ND
- X701: Digi-Key PN (none) -> 535-10072-1-ND
