File: hdw/AC_Power_Meter/Microcontroller.sch (KiCad schematic (older format))
At the start: 17 parts, among them U701 PIC18LF67K40-I/PT, X701 ASV-16.000MHz

Commit message: Arranged a few pages of components
Parts:
- X701: footprint Oscillator:Oscillator_SMD_Abracon_ASV-4Pin_7.0x5.1mm -> Oscillators:Oscillator_SMD_Abracon_ASV-4pin_7.0x5.1mm
Changed lines of the file:
@@
 F 0 "X701" H 9250 6220 50  0000 L CNN
 F 1 "ASV-16.000MHz" H 9500 5720 50  0000 L CNN
-F 2 "Oscillator:Oscillator_SMD_Abracon_ASV-4Pin_7.0x5.1mm" H 10150 5620 50  0001 C CNN
+F 2 "Oscillators:Oscillator_SMD_Abracon_ASV-4pin_7.0x5.1mm" H 10150 5620 50  0001 C CNN
 F 3 "http://www.abracon.com/Oscillators/ASV.pdf" H 9350 5970 50  0001 C CNN
 F 4 "535-10072-1-ND" H 9450 5970 50  0001 C CNN "Digi-Key PN"

Commit message: Finished placing parts
Changed lines of the file:
@@
 L Custom_Library:R_Custom R?
 U 1 1 5BBE6824
-P 2780 4820
+P 2790 3920
 AR Path="/5BB27BA3/5BBE6824" Ref="R?"  Part="1"
 AR Path="/5BB27BF7/5BBE6824" Ref="R?"  Part="1"
 AR Path="/5BB27B84/5BBE6824" Ref="R704"  Part="1"
-F 0 "R704" H 2700 4820 50  0000 R CNN
-F 1 "10k" V 2780 4820 50  0000 C CNN
-F 2 "Resistors_SMD:R_0603" H 2780 4820 50  0001 C CNN
-F 3 "" H 2780 4820 50  0001 C CNN
-F 4 "0603" H 2880 4900 50  0000 L CNN "display_footprint"
-F 5 "1%" H 2880 4820 50  0000 L CNN "Tolerance"
-F 6 "1/10W" H 2890 4740 50  0000 L CNN "Wattage"
-F 7 "RHM10KADCT-ND" H 3080 5220 60  0001 C CNN "Digi-Key PN"
-	1    2780 4820
+F 0 "R704" H 2710 3920 50  0000 R CNN
+F 1 "10k" V 2790 3920 50  0000 C CNN
+F 2 "Resistors_SMD:R_0603" H 2790 3920 50  0001 C CNN
+F 3 "" H 2790 3920 50  0001 C CNN
+F 4 "0603" H 2890 4000 50  0000 L CNN "display_footprint"
+F 5 "1%" H 2890 3920 50  0000 L CNN "Tolerance"
+F 6 "1/10W" H 2900 3840 50  0000 L CNN "Wattage"
+F 7 "RHM10KADCT-ND" H 3090 4320 60  0001 C CNN "Digi-Key PN"
+	1    2790 3920
 	1    0    0    -1
 $EndComp
@@
 L Custom_Library:R_Custom R?
 U 1 1 5BBE682F
-P 2030 4820
+P 2040 3920
 AR Path="/5BB27BA3/5BBE682F" Ref="R?"  Part="1"
 AR Path="/5BB27BF7/5BBE682F" Ref="R?"  Part="1"
 AR Path="/5BB27B84/5BBE682F" Ref="R703"  Part="1"
-F 0 "R703" H 1950 4820 50  0000 R CNN
-F 1 "10k" V 2030 4820 50  0000 C CNN
-F 2 "Resistors_SMD:R_0603" H 2030 4820 50  0001 C CNN
-F 3 "" H 2030 4820 50  0001 C CNN
-F 4 "0603" H 2130 4900 50  0000 L CNN "display_footprint"
-F 5 "1%" H 2130 4820 50  0000 L CNN "Tolerance"
-F 6 "1/10W" H 2140 4740 50  0000 L CNN "Wattage"
-F 7 "RHM10KADCT-ND" H 2330 5220 60  0001 C CNN "Digi-Key PN"
-	1    2030 4820
+F 0 "R703" H 1960 3920 50  0000 R CNN
+F 1 "10k" V 2040 3920 50  0000 C CNN
+F 2 "Resistors_SMD:R_0603" H 2040 3920 50  0001 C CNN
+F 3 "" H 2040 3920 50  0001 C CNN
+F 4 "0603" H 2140 4000 50  0000 L CNN "display_footprint"
+F 5 "1%" H 2140 3920 50  0000 L CNN "Tolerance"
+F 6 "1/10W" H 2150 3840 50  0000 L CNN "Wattage"
+F 7 "RHM10KADCT-ND" H 2340 4320 60  0001 C CNN "Digi-Key PN"
+	1    2040 3920
 	1    0    0    -1
 $EndComp
@@
 L Custom_Library:+3.3V #PWR?
 U 1 1 5BBE6836
-P 2780 4670
+P 2790 3770
 AR Path="/5BB27BF7/5BBE6836" Ref="#PWR?"  Part="1"
 AR Path="/5BB27B84/5BBE6836" Ref="#PWR0704"  Part="1"
-F 0 "#PWR0704" H 2780 4520 50  0001 C CNN
-F 1 "+3.3V" H 2780 4810 50  0000 C CNN
-F 2 "" H 2780 4670 50  0000 C CNN
-F 3 "" H 2780 4670 50  0000 C CNN
-	1    2780 4670
+F 0 "#PWR0704" H 2790 3620 50  0001 C CNN
+F 1 "+3.3V" H 2790 3910 50  0000 C CNN
+F 2 "" H 2790 3770 50  0000 C CNN
+F 3 "" H 2790 3770 50  0000 C CNN
+	1    2790 3770
 	1    0    0    -1
 $EndComp
@@
 L Custom_Library:+3.3V #PWR?
 U 1 1 5BBE683C
-P 2030 4670
+P 2040 3770
 AR Path="/5BB27BF7/5BBE683C" Ref="#PWR?"  Part="1"
 AR Path="/5BB27B84/5BBE683C" Ref="#PWR0703"  Part="1"
-F 0 "#PWR0703" H 2030 4520 50  0001 C CNN
-F 1 "+3.3V" H 2030 4810 50  0000 C CNN
-F 2 "" H 2030 4670 50  0000 C CNN
-F 3 "" H 2030 4670 50  0000 C CNN
-	1    2030 4670
+F 0 "#PWR0703" H 2040 3620 50  0001 C CNN
+F 1 "+3.3V" H 2040 3910 50  0000 C CNN
+F 2 "" H 2040 3770 50  0000 C CNN
+F 3 "" H 2040 3770 50  0000 C CNN
+	1    2040 3770
 	1    0    0    -1
 $EndComp
@@
 L Device:R R?
 U 1 1 5BBE6845
-P 1580 5190
+P 1590 4290
 AR Path="/5A2D2FD2/5BBE6845" Ref="R?"  Part="1"
 AR Path="/5A0A8BD0/5BBE6845" Ref="R?"  Part="1"
@@
 AR Path="/5BB27BF7/5BBE6845" Ref="R?"  Part="1"
 AR Path="/5BB27B84/5BBE6845" Ref="R701"  Part="1"
-F 0 "R701" V 1660 5190 50  0000 C CNN
-F 1 "0" V 1580 5190 50  0000 C CNN
-F 2 "Resistors_SMD:R_0603" V 1510 5190 50  0001 C CNN
-F 3 "" V 1660 5190 50  0001 C CNN
-F 4 "1%" V 1320 5190 50  0001 C CNN "Tolerance"
-F 5 "1/10W" V 1480 5190 50  0001 C CNN "Wattage"
-F 6 "0603" V 1400 5190 50  0001 C CNN "display_footprint"
-F 7 "P0.0GCT-ND" H 0   0   50  0001 C CNN "Digi-Key PN"
-	1    1580 5190
+F 0 "R701" V 1670 4290 50  0000 C CNN
+F 1 "0" V 1590 4290 50  0000 C CNN
+F 2 "Resistors_SMD:R_0603" V 1520 4290 50  0001 C CNN
+F 3 "" V 1670 4290 50  0001 C CNN
+F 4 "1%" V 1330 4290 50  0001 C CNN "Tolerance"
+F 5 "1/10W" V 1490 4290 50  0001 C CNN "Wattage"
+F 6 "0603" V 1410 4290 50  0001 C CNN "display_footprint"
+F 7 "P0.0GCT-ND" H 10  -900 50  0001 C CNN "Digi-Key PN"
+	1    1590 4290
 	0    -1   -1   0
 $EndComp
@@
 L Device:R R?
 U 1 1 5BBE684F
-P 1580 5290
+P 1590 4390
 AR Path="/5A2D2FD2/5BBE684F" Ref="R?"  Part="1"
 AR Path="/5A0A8BD0/5BBE684F" Ref="R?"  Part="1"
@@
 AR Path="/5BB27BF7/5BBE684F" Ref="R?"  Part="1"
 AR Path="/5BB27B84/5BBE684F" Ref="R702"  Part="1"
-F 0 "R702" V 1660 5290 50  0000 C CNN
-F 1 "0" V 1580 5290 50  0000 C CNN
-F 2 "Resistors_SMD:R_0603" V 1510 5290 50  0001 C CNN
-F 3 "" V 1660 5290 50  0001 C CNN
-F 4 "1%" V 1320 5290 50  0001 C CNN "Tolerance"
-F 5 "1/10W" V 1480 5290 50  0001 C CNN "Wattage"
-F 6 "0603" V 1400 5290 50  0001 C CNN "display_footprint"
-F 7 "P0.0GCT-ND" H 0   0   50  0001 C CNN "Digi-Key PN"
-	1    1580 5290
+F 0 "R702" V 1670 4390 50  0000 C CNN
+F 1 "0" V 1590 4390 50  0000 C CNN
+F 2 "Resistors_SMD:R_0603" V 1520 4390 50  0001 C CNN
+F 3 "" V 1670 4390 50  0001 C CNN
+F 4 "1%" V 1330 4390 50  0001 C CNN "Tolerance"
+F 5 "1/10W" V 1490 4390 50  0001 C CNN "Wattage"
+F 6 "0603" V 1410 4390 50  0001 C CNN "display_footprint"
+F 7 "P0.0GCT-ND" H 10  -900 50  0001 C CNN "Digi-Key PN"
+	1    1590 4390
 	0    1    1    0
 $EndComp
 Wire Wire Line
-	2030 4970 2030 5290
-Wire Wire Line
-	2780 4970 2780 5190
-Text GLabel 1430 5190 0    50   BiDi ~ 0
+	2040 4070 2040 4390
+Wire Wire Line
+	2790 4070 2790 4290
+Text GLabel 1440 4290 0    50   BiDi ~ 0
 I2C_SDA
-Text GLabel 1430 5290 0    50   Output ~ 0
+Text GLabel 1440 4390 0    50   Output ~ 0
 I2C_SCL
 Text GLabel 4080 2790 0    50   Input ~ 0
@@
 ADC_Error
 Wire Wire Line
-	2780 5190 4080 5190
-Wire Wire Line
-	2030 5290 4080 5290
-Wire Wire Line
-	2780 5190 1730 5190
-Connection ~ 2780 5190
-Wire Wire Line
-	1730 5290 2030 5290
-Connection ~ 2030 5290
+	2790 4290 1740 4290
+Wire Wire Line
+	1740 4390 2040 4390
 $Comp
 L Custom_Library:CP_Tant_Custom C?
@@
 NoConn ~ 4080 4090
 NoConn ~ 4080 4190
-NoConn ~ 4080 4290
-NoConn ~ 4080 4390
 NoConn ~ 4080 4590
 NoConn ~ 4080 4690
@@
 NoConn ~ 6580 4790
 NoConn ~ 6580 4890
+Wire Wire Line
+	4080 4390 2040 4390
+Connection ~ 2040 4390
+Wire Wire Line
+	2790 4290 4080 4290
+Connection ~ 2790 4290
+NoConn ~ 4080 5190
+NoConn ~ 4080 5290
 $EndSCHEMATC

Commit message: Finished routing, adding bells and whistles
Changed lines of the file:
@@
 	1    0    0    -1
 $EndComp
-Text GLabel 6580 1990 2    50   Input ~ 0
+Text GLabel 4080 3990 0    50   Input ~ 0
 POS12_PGOOD
-Text GLabel 6580 2190 2    50   Input ~ 0
+Text GLabel 4080 3890 0    50   Input ~ 0
 POS3P3_PGOOD
 Text GLabel 4080 1890 0    50   Input ~ 0
@@
 Text GLabel 1440 4390 0    50   Output ~ 0
 I2C_SCL
-Text GLabel 4080 2790 0    50   Input ~ 0
+Text GLabel 4080 2390 0    50   Input ~ 0
 Zero_Cross_Detect
 Text GLabel 6580 3690 2    50   Output ~ 0
@@
 Text GLabel 6580 2090 2    50   Input ~ 0
 POS3P3_ADC
-Text GLabel 6580 1890 2    50   Input ~ 0
+Text GLabel 4080 2290 0    50   Input ~ 0
 POS12_ADC
-Text GLabel 4080 2890 0    50   Input ~ 0
+Text GLabel 4080 2790 0    50   Input ~ 0
 SW_Toggle
 $Comp
@@
 $EndComp
 NoConn ~ 4080 1990
-NoConn ~ 4080 2290
-NoConn ~ 4080 2390
 NoConn ~ 4080 2490
 NoConn ~ 4080 2990
@@
 NoConn ~ 4080 3690
 NoConn ~ 4080 3790
-NoConn ~ 4080 3890
-NoConn ~ 4080 3990
 NoConn ~ 4080 4090
 NoConn ~ 4080 4190
@@
 NoConn ~ 4080 5190
 NoConn ~ 4080 5290
+NoConn ~ 4080 2890
+NoConn ~ 6580 1990
+NoConn ~ 6580 2190
+NoConn ~ 6580 1890
 $EndSCHEMATC

Commit message: Serious BOM scrubbing to drive price down
Parts:
- removed C707: 47uF, Capacitors_Tantalum_SMD:CP_Tantalum_Case-X_EIA-7343-43_Reflow, symbol Custom_Library:CP_Tant_Custom
Connections:
- net labels removed: POS12_PGOOD, POS3P3_PGOOD, SW_Toggle
- no-connect marks 37 -> 40
Changed lines of the file:
@@
 $Descr A 11000 8500
 encoding utf-8
-Sheet 7 18
+Sheet 7 17
 Title ""
 Date "2018-10-01"
@@
 	1    0    0    -1
 $EndComp
-Text GLabel 4080 3990 0    50   Input ~ 0
-POS12_PGOOD
-Text GLabel 4080 3890 0    50   Input ~ 0
-POS3P3_PGOOD
 Text GLabel 4080 1890 0    50   Input ~ 0
 ISNS_ADC
@@
 	1740 4390 2040 4390
 $Comp
-L Custom_Library:CP_Tant_Custom C?
-U 1 1 5BBF0F15
-P 4590 7010
-AR Path="/5BB27B51/5BBF0F15" Ref="C?"  Part="1"
-AR Path="/5BB27B84/5BBF0F15" Ref="C707"  Part="1"
-F 0 "C707" H 4615 7110 50  0000 L CNN
-F 1 "47uF" H 4615 6910 50  0000 L CNN
-F 2 "Capacitors_Tantalum_SMD:CP_Tantalum_Case-X_EIA-7343-43_Reflow" H 4628 6860 50  0001 C CNN
-F 3 "" H 4615 7110 50  0001 C CNN
-F 4 "478-3938-1-ND" H 4590 7010 50  0001 C CNN "Digi-Key PN"
-F 5 "7343" H 4440 7110 50  0000 R CNN "display_footprint"
-F 6 "16V" H 4440 7010 50  0000 R CNN "Voltage"
-F 7 "10%" H 4440 6910 50  0000 R CNN "Tolerance"
-	1    4590 7010
-	1    0    0    -1
-$EndComp
-$Comp
-L power:GND #PWR0708
-U 1 1 5BBF1696
-P 4590 7160
-F 0 "#PWR0708" H 4590 6910 50  0001 C CNN
-F 1 "GND" H 4590 7010 50  0000 C CNN
-F 2 "" H 4590 7160 50  0001 C CNN
-F 3 "" H 4590 7160 50  0001 C CNN
-	1    4590 7160
-	1    0    0    -1
-$EndComp
-$Comp
-L Custom_Library:+3.3V #PWR0707
-U 1 1 5BBF16B9
-P 4590 6860
-F 0 "#PWR0707" H 4590 6710 50  0001 C CNN
-F 1 "+3.3V" H 4590 7000 50  0000 C CNN
-F 2 "" H 4590 6860 50  0000 C CNN
-F 3 "" H 4590 6860 50  0000 C CNN
-	1    4590 6860
-	1    0    0    -1
-$EndComp
-$Comp
 L Oscillator:ASV-xxxMHz X701
 U 1 1 5BBF1E7B
@@
 Text GLabel 4080 2290 0    50   Input ~ 0
 POS12_ADC
-Text GLabel 4080 2790 0    50   Input ~ 0
-SW_Toggle
 $Comp
 L power:+3.3VADC #PWR0710
@@
 NoConn ~ 6580 2190
 NoConn ~ 6580 1890
+NoConn ~ 4080 2790
+NoConn ~ 4080 3890
+NoConn ~ 4080 3990
 $EndSCHEMATC
