File: hdw/AC_Power_Meter/Microcontroller.sch (KiCad schematic (older format))
At the start: 16 parts, among them U701 PIC18LF67K40-I/PT, X701 ASV-16.000MHz

Commit message: Schematic cleanup, live updates working in code
Changed lines of the file:
@@
 	5380 5580 5380 5540
 Connection ~ 5330 5580
-$Comp
-L Custom_Library:+3.3V #PWR0711
-U 1 1 5BB27F33
-P 5330 1560
-F 0 "#PWR0711" H 5330 1410 50  0001 C CNN
-F 1 "+3.3V" H 5330 1700 50  0000 C CNN
-F 2 "" H 5330 1560 50  0000 C CNN
-F 3 "" H 5330 1560 50  0000 C CNN
-	1    5330 1560
-	1    0    0    -1
-$EndComp
 Wire Wire Line
 	5330 1560 5330 1600
@@
 	1    0    0    -1
 $EndComp
-$Comp
-L Custom_Library:+3.3V #PWR0701
-U 1 1 5BB28F98
-P 1950 6790
-F 0 "#PWR0701" H 1950 6640 50  0001 C CNN
-F 1 "+3.3V" H 1950 6930 50  0000 C CNN
-F 2 "" H 1950 6790 50  0000 C CNN
-F 3 "" H 1950 6790 50  0000 C CNN
-	1    1950 6790
-	1    0    0    -1
-$EndComp
 Wire Wire Line
 	1950 6790 1950 6830
@@
 F 3 "" H 3520 7250 50  0001 C CNN
 	1    3520 7250
-	1    0    0    -1
-$EndComp
-$Comp
-L Custom_Library:+3.3V #PWR0705
-U 1 1 5BB29969
-P 3520 6790
-F 0 "#PWR0705" H 3520 6640 50  0001 C CNN
-F 1 "+3.3V" H 3520 6930 50  0000 C CNN
-F 2 "" H 3520 6790 50  0000 C CNN
-F 3 "" H 3520 6790 50  0000 C CNN
-	1    3520 6790
 	1    0    0    -1
 $EndComp
@@
 F 7 "RHM10KADCT-ND" H 2340 4320 60  0001 C CNN "Digi-Key PN"
 	1    2040 3920
-	1    0    0    -1
-$EndComp
-$Comp
-L Custom_Library:+3.3V #PWR?
-U 1 1 5BBE6836
-P 2790 3770
-AR Path="/5BB27BF7/5BBE6836" Ref="#PWR?"  Part="1"
-AR Path="/5BB27B84/5BBE6836" Ref="#PWR0704"  Part="1"
-F 0 "#PWR0704" H 2790 3620 50  0001 C CNN
-F 1 "+3.3V" H 2790 3910 50  0000 C CNN
-F 2 "" H 2790 3770 50  0000 C CNN
-F 3 "" H 2790 3770 50  0000 C CNN
-	1    2790 3770
-	1    0    0    -1
-$EndComp
-$Comp
-L Custom_Library:+3.3V #PWR?
-U 1 1 5BBE683C
-P 2040 3770
-AR Path="/5BB27BF7/5BBE683C" Ref="#PWR?"  Part="1"
-AR Path="/5BB27B84/5BBE683C" Ref="#PWR0703"  Part="1"
-F 0 "#PWR0703" H 2040 3620 50  0001 C CNN
-F 1 "+3.3V" H 2040 3910 50  0000 C CNN
-F 2 "" H 2040 3770 50  0000 C CNN
-F 3 "" H 2040 3770 50  0000 C CNN
-	1    2040 3770
 	1    0    0    -1
 $EndComp
@@
 U 1 1 5BBF1E7B
 P 9450 5970
-F 0 "X701" H 9250 6220 50  0000 L CNN
+F 0 "X701" H 9500 6220 50  0000 L CNN
 F 1 "ASV-16.000MHz" H 9500 5720 50  0000 L CNN
 F 2 "Oscillators:Oscillator_SMD_Abracon_ASV-4pin_7.0x5.1mm" H 10150 5620 50  0001 C CNN
@@
 F 3 "" H 9450 6270 50  0001 C CNN
 	1    9450 6270
-	1    0    0    -1
-$EndComp
-$Comp
-L Custom_Library:+3.3V #PWR0716
-U 1 1 5BBF289D
-P 9450 5670
-F 0 "#PWR0716" H 9450 5520 50  0001 C CNN
-F 1 "+3.3V" H 9450 5810 50  0000 C CNN
-F 2 "" H 9450 5670 50  0000 C CNN
-F 3 "" H 9450 5670 50  0000 C CNN
-	1    9450 5670
 	1    0    0    -1
 $EndComp
@@
 	1    0    0    -1
 $EndComp
-$Comp
-L Custom_Library:+3.3V #PWR?
-U 1 1 5BBF2F02
-P 8680 5510
-AR Path="/5BB27BF7/5BBF2F02" Ref="#PWR?"  Part="1"
-AR Path="/5BB27B84/5BBF2F02" Ref="#PWR0715"  Part="1"
-F 0 "#PWR0715" H 8680 5360 50  0001 C CNN
-F 1 "+3.3V" H 8680 5650 50  0000 C CNN
-F 2 "" H 8680 5510 50  0000 C CNN
-F 3 "" H 8680 5510 50  0000 C CNN
-	1    8680 5510
-	1    0    0    -1
-$EndComp
 Wire Wire Line
 	9150 5970 8680 5970
@@
 F 3 "" H 7980 6240 50  0001 C CNN
 	1    7980 6240
-	1    0    0    -1
-$EndComp
-$Comp
-L Custom_Library:+3.3V #PWR0713
-U 1 1 5BBF43A3
-P 7980 5780
-F 0 "#PWR0713" H 7980 5630 50  0001 C CNN
-F 1 "+3.3V" H 7980 5920 50  0000 C CNN
-F 2 "" H 7980 5780 50  0000 C CNN
-F 3 "" H 7980 5780 50  0000 C CNN
-	1    7980 5780
 	1    0    0    -1
 $EndComp
@@
 NoConn ~ 4080 3890
 NoConn ~ 4080 3990
+$Comp
+L power:+3.3V #PWR?
+U 1 1 5BF35500
+P 1950 6790
+F 0 "#PWR?" H 1950 6640 50  0001 C CNN
+F 1 "+3.3V" H 1950 6930 50  0000 C CNN
+F 2 "" H 1950 6790 50  0001 C CNN
+F 3 "" H 1950 6790 50  0001 C CNN
+	1    1950 6790
+	1    0    0    -1
+$EndComp
+$Comp
+L power:+3.3V #PWR?
+U 1 1 5BF355A2
+P 3520 6790
+F 0 "#PWR?" H 3520 6640 50  0001 C CNN
+F 1 "+3.3V" H 3520 6930 50  0000 C CNN
+F 2 "" H 3520 6790 50  0001 C CNN
+F 3 "" H 3520 6790 50  0001 C CNN
+	1    3520 6790
+	1    0    0    -1
+$EndComp
+$Comp
+L power:+3.3V #PWR?
+U 1 1 5BF3565D
+P 2040 3770
+F 0 "#PWR?" H 2040 3620 50  0001 C CNN
+F 1 "+3.3V" H 2040 3910 50  0000 C CNN
+F 2 "" H 2040 3770 50  0001 C CNN
+F 3 "" H 2040 3770 50  0001 C CNN
+	1    2040 3770
+	1    0    0    -1
+$EndComp
+$Comp
+L power:+3.3V #PWR?
+U 1 1 5BF35768
+P 2790 3770
+F 0 "#PWR?" H 2790 3620 50  0001 C CNN
+F 1 "+3.3V" H 2790 3910 50  0000 C CNN
+F 2 "" H 2790 3770 50  0001 C CNN
+F 3 "" H 2790 3770 50  0001 C CNN
+	1    2790 3770
+	1    0    0    -1
+$EndComp
+$Comp
+L power:+3.3V #PWR?
+U 1 1 5BF35793
+P 5330 1560
+F 0 "#PWR?" H 5330 1410 50  0001 C CNN
+F 1 "+3.3V" H 5330 1700 50  0000 C CNN
+F 2 "" H 5330 1560 50  0001 C CNN
+F 3 "" H 5330 1560 50  0001 C CNN
+	1    5330 1560
+	1    0    0    -1
+$EndComp
+$Comp
+L power:+3.3V #PWR?
+U 1 1 5BF3588E
+P 7980 5780
+F 0 "#PWR?" H 7980 5630 50  0001 C CNN
+F 1 "+3.3V" H 7980 5920 50  0000 C CNN
+F 2 "" H 7980 5780 50  0001 C CNN
+F 3 "" H 7980 5780 50  0001 C CNN
+	1    7980 5780
+	1    0    0    -1
+$EndComp
+$Comp
+L power:+3.3V #PWR?
+U 1 1 5BF35999
+P 8680 5510
+F 0 "#PWR?" H 8680 5360 50  0001 C CNN
+F 1 "+3.3V" H 8680 5650 50  0000 C CNN
+F 2 "" H 8680 5510 50  0001 C CNN
+F 3 "" H 8680 5510 50  0001 C CNN
+	1    8680 5510
+	1    0    0    -1
+$EndComp
+$Comp
+L power:+3.3V #PWR?
+U 1 1 5BF35A94
+P 9450 5670
+F 0 "#PWR?" H 9450 5520 50  0001 C CNN
+F 1 "+3.3V" H 9450 5810 50  0000 C CNN
+F 2 "" H 9450 5670 50  0001 C CNN
+F 3 "" H 9450 5670 50  0001 C CNN
+	1    9450 5670
+	1    0    0    -1
+$EndComp
 $EndSCHEMATC
