File: hdw/AC_Power_Meter/Microcontroller_Programming.sch (KiCad schematic (older format))
At the start: 17 parts

Commit message: Added +3.3V power supply, +12V window comparator, a few design files
Parts:
- removed R?: 10k, symbol Custom_Library:R_Custom
Connections:
- wire segments 21 -> 18

Commit message: Added MU logo and titles to all sheets
Other:
- note added: "Programming Header, ~MCLR~ Reset Filter, ICSP Detection"
- note removed: "Programming Header/ICSP Detection"
Changed lines of the file:
@@
 	1    0    0    -1
 $EndComp
-Text Notes 3890 1070 0    100  ~ 20
-Programming Header/ICSP Detection
+Text Notes 540  690  0    100  ~ 20
+Programming Header, ~MCLR~ Reset Filter, ICSP Detection
 $Comp
 L Custom_Library:+3.3V #PWR?
@@
 	1    0    0    -1
 $EndComp
+$Comp
+L Mu_Logo:LOGO #G?
+U 1 1 5BBF40D0
+P 9900 1000
+F 0 "#G?" H 9900 670 60  0001 C CNN
+F 1 "LOGO" H 9900 1330 60  0001 C CNN
+F 2 "" H 9900 1000 50  0001 C CNN
+F 3 "" H 9900 1000 50  0001 C CNN
+	1    9900 1000
+	1    0    0    -1
+$EndComp

Commit message: Updated MU logo to crisper image
Changed lines of the file:
@@
 $EndComp
 $Comp
-L Mu_Logo:LOGO #G?
-U 1 1 5BBF40D0
-P 9900 1000
-F 0 "#G?" H 9900 670 60  0001 C CNN
-F 1 "LOGO" H 9900 1330 60  0001 C CNN
-F 2 "" H 9900 1000 50  0001 C CNN
-F 3 "" H 9900 1000 50  0001 C CNN
-	1    9900 1000
+L Custom_Library:MU_Logo #G?
+U 1 1 5BB69125
+P 9900 1100
+F 0 "#G?" H 9900 614 60  0001 C CNN
+F 1 "MU_Logo" H 9900 1586 60  0001 C CNN
+F 2 "" H 9900 1100 50  0001 C CNN
+F 3 "" H 9900 1100 50  0001 C CNN
+	1    9900 1100
 	1    0    0    -1
 $EndComp

Commit message: Revised signal conditioning, cleaned up a lot of pages
Parts:
- Z?: value ZENER_Custom -> UDZSTE-175.1B; Digi-Key PN (none) -> UDZSTE-175.1BCT-ND
Changed lines of the file:
@@
 P 2000 4440
 F 0 "Z?" V 2000 4640 50  0000 C CNN
-F 1 "ZENER_Custom" V 1900 4340 50  0000 R CNN
+F 1 "UDZSTE-175.1B" V 1900 4340 50  0000 R CNN
 F 2 "" H 2000 4440 60  0000 C CNN
 F 3 "" H 2000 4440 60  0000 C CNN
-F 4 "SOD323" V 2000 4340 50  0000 R CNN "display_footprint"
-F 5 "5.1V" V 2100 4340 50  0000 R CNN "Voltage"
+F 4 "UDZSTE-175.1BCT-ND" H 2000 4440 50  0001 C CNN "Digi-Key PN"
+F 5 "SOD323" V 2000 4340 50  0000 R CNN "display_footprint"
+F 6 "5.1V" V 2100 4340 50  0000 R CNN "Voltage"
 	1    2000 4440
 	0    1    1    0

Commit message: Rewired a few micro symbols, add FMW notes
Parts:
- added C803: 0.1uF, symbol Custom_Library:C_Custom
- added C804: 10nF, symbol Custom_Library:C_Custom
- added C805: 1nF, symbol Custom_Library:C_Custom
- added L801, L802: 600R 0.5A, Inductors_SMD:L_0603, symbol Device:Ferrite_Bead
- gave numbers to parts that had none: 16
Connections:
- net labels added: +3.3VADC, GNDA
- wire segments 18 -> 38

Commit message: Updated most footprints
Parts:
- C801, C802, C803, C806, C807, C808: footprint (none) -> Capacitors_SMD:C_0603; Digi-Key PN PN -> 490-8020-1-ND
- C804: footprint (none) -> Capacitors_SMD:C_0603; Digi-Key PN PN -> 1276-1921-1-ND
- C805: footprint (none) -> Capacitors_SMD:C_0603; Digi-Key PN PN -> 478-1215-1-ND
- R801, R802, R803, R805: footprint (none) -> Resistors_SMD:R_0603; Digi-Key PN PN -> RHM10KADCT-ND
- R804: footprint (none) -> Resistors_SMD:R_0603; Digi-Key PN PN -> P0.0GCT-ND
- R806: footprint (none) -> Resistors_SMD:R_0603; Digi-Key PN PN -> (none)
- R807: footprint (none) -> Resistors_SMD:R_0603; Digi-Key PN PN -> MCT0603-1.00K-CFCT-ND
- U801: Digi-Key PN (none) -> 296-10168-1-ND
- Z801: footprint (none) -> Diodes_SMD:D_SOD-523
Changed lines of the file:
@@
 F 2 "TO_SOT_Packages_SMD:SOT-23-5" H 3310 2760 50  0001 C CNN
 F 3 "http://www.ti.com/lit/ds/symlink/tl331.pdf" H 3310 2860 50  0001 C CNN
+F 4 "296-10168-1-ND" H 3310 2660 50  0001 C CNN "Digi-Key PN"
 	1    3310 2660
 	1    0    0    -1
@@
 F 0 "R801" H 1750 2520 50  0000 R CNN
 F 1 "10k" V 1830 2520 50  0000 C CNN
-F 2 "" H 1830 2520 50  0001 C CNN
+F 2 "Resistors_SMD:R_0603" H 1830 2520 50  0001 C CNN
 F 3 "" H 1830 2520 50  0001 C CNN
 F 4 "0603" H 1930 2600 50  0000 L CNN "display_footprint"
 F 5 "1%" H 1930 2520 50  0000 L CNN "Tolerance"
 F 6 "1/10W" H 1940 2440 50  0000 L CNN "Wattage"
-F 7 "PN" H 2130 2920 60  0001 C CNN "Digi-Key PN"
+F 7 "RHM10KADCT-ND" H 2130 2920 60  0001 C CNN "Digi-Key PN"
 	1    1830 2520
 	1    0    0    -1
@@
 F 0 "R803" H 4420 2360 50  0000 R CNN
 F 1 "10k" V 4500 2360 50  0000 C CNN
-F 2 "" H 4500 2360 50  0001 C CNN
+F 2 "Resistors_SMD:R_0603" H 4500 2360 50  0001 C CNN
 F 3 "" H 4500 2360 50  0001 C CNN
 F 4 "0603" H 4600 2440 50  0000 L CNN "display_footprint"
 F 5 "1%" H 4600 2360 50  0000 L CNN "Tolerance"
 F 6 "1/10W" H 4610 2280 50  0000 L CNN "Wattage"
-F 7 "PN" H 4800 2760 60  0001 C CNN "Digi-Key PN"
+F 7 "RHM10KADCT-ND" H 4800 2760 60  0001 C CNN "Digi-Key PN"
 	1    4500 2360
 	1    0    0    -1
@@
 F 0 "R804" H 4420 3050 50  0000 R CNN
 F 1 "0" V 4500 3050 50  0000 C CNN
-F 2 "" H 4500 3050 50  0001 C CNN
+F 2 "Resistors_SMD:R_0603" H 4500 3050 50  0001 C CNN
 F 3 "" H 4500 3050 50  0001 C CNN
 F 4 "0603" H 4600 3130 50  0000 L CNN "display_footprint"
 F 5 "1%" H 4600 3050 50  0000 L CNN "Tolerance"
 F 6 "1/10W" H 4610 2970 50  0000 L CNN "Wattage"
-F 7 "PN" H 4800 3450 60  0001 C CNN "Digi-Key PN"
+F 7 "P0.0GCT-ND" H 4800 3450 60  0001 C CNN "Digi-Key PN"
 	1    4500 3050
 	1    0    0    -1
@@
 F 0 "R802" H 3780 2430 50  0000 R CNN
 F 1 "10k" V 3860 2430 50  0000 C CNN
-F 2 "" H 3860 2430 50  0001 C CNN
+F 2 "Resistors_SMD:R_0603" H 3860 2430 50  0001 C CNN
 F 3 "" H 3860 2430 50  0001 C CNN
 F 4 "0603" H 3960 2510 50  0000 L CNN "display_footprint"
 F 5 "1%" H 3960 2430 50  0000 L CNN "Tolerance"
 F 6 "1/10W" H 3970 2350 50  0000 L CNN "Wattage"
-F 7 "PN" H 4160 2830 60  0001 C CNN "Digi-Key PN"
+F 7 "RHM10KADCT-ND" H 4160 2830 60  0001 C CNN "Digi-Key PN"
 	1    3860 2430
 	1    0    0    -1
@@
 F 0 "C802" H 3565 3470 50  0000 L CNN
 F 1 "0.1uF" H 3565 3270 50  0000 L CNN
-F 2 "" H 3578 3220 50  0001 C CNN
+F 2 "Capacitors_SMD:C_0603" H 3578 3220 50  0001 C CNN
 F 3 "" H 3565 3470 50  0001 C CNN
 F 4 "0603" H 3390 3470 50  0000 R CNN "display_footprint"
 F 5 "50V" H 3390 3370 50  0000 R CNN "Voltage"
 F 6 "X7R" H 3390 3270 50  0000 R CNN "Dielectric"
-F 7 "PN" H 3965 3870 60  0001 C CNN "Digi-Key PN"
+F 7 "490-8020-1-ND" H 3965 3870 60  0001 C CNN "Digi-Key PN"
 	1    3540 3370
 	-1   0    0    -1
@@
 F 0 "C801" H 2485 3160 50  0000 L CNN
 F 1 "0.1uF" H 2485 2960 50  0000 L CNN
-F 2 "" H 2498 2910 50  0001 C CNN
+F 2 "Capacitors_SMD:C_0603" H 2498 2910 50  0001 C CNN
 F 3 "" H 2485 3160 50  0001 C CNN
 F 4 "0603" H 2310 3160 50  0000 R CNN "display_footprint"
 F 5 "50V" H 2310 3060 50  0000 R CNN "Voltage"
 F 6 "X7R" H 2310 2960 50  0000 R CNN "Dielectric"
-F 7 "PN" H 2885 3560 60  0001 C CNN "Digi-Key PN"
+F 7 "490-8020-1-ND" H 2885 3560 60  0001 C CNN "Digi-Key PN"
 	1    2460 3060
 	-1   0    0    -1
@@
 F 0 "C806" H 5175 3490 50  0000 L CNN
 F 1 "0.1uF" H 5175 3290 50  0000 L CNN
-F 2 "" H 5188 3240 50  0001 C CNN
+F 2 "Capacitors_SMD:C_0603" H 5188 3240 50  0001 C CNN
 F 3 "" H 5175 3490 50  0001 C CNN
 F 4 "0603" H 5000 3490 50  0000 R CNN "display_footprint"
 F 5 "50V" H 5000 3390 50  0000 R CNN "Voltage"
 F 6 "X7R" H 5000 3290 50  0000 R CNN "Dielectric"
-F 7 "PN" H 5575 3890 60  0001 C CNN "Digi-Key PN"
+F 7 "490-8020-1-ND" H 5575 3890 60  0001 C CNN "Digi-Key PN"
 	1    5150 3390
 	-1   0    0    -1
@@
 F 0 "C807" H 7185 2210 50  0000 L CNN
 F 1 "0.1uF" H 7185 2010 50  0000 L CNN
-F 2 "" H 7198 1960 50  0001 C CNN
+F 2 "Capacitors_SMD:C_0603" H 7198 1960 50  0001 C CNN
 F 3 "" H 7185 2210 50  0001 C CNN
 F 4 "0603" H 7010 2210 50  0000 R CNN "display_footprint"
 F 5 "50V" H 7010 2110 50  0000 R CNN "Voltage"
 F 6 "X7R" H 7010 2010 50  0000 R CNN "Dielectric"
-F 7 "PN" H 7585 2610 60  0001 C CNN "Digi-Key PN"
+F 7 "490-8020-1-ND" H 7585 2610 60  0001 C CNN "Digi-Key PN"
 	1    7160 2110
 	-1   0    0    -1
@@
 F 0 "Z801" V 1830 3240 50  0000 C CNN
 F 1 "UDZSTE-175.1B" V 1730 2940 50  0000 R CNN
-F 2 "" H 1830 3040 60  0000 C CNN
+F 2 "Diodes_SMD:D_SOD-523" H 1830 3040 60  0001 C CNN
 F 3 "" H 1830 3040 60  0000 C CNN
 F 4 "UDZSTE-175.1BCT-ND" H 1830 3040 50  0001 C CNN "Digi-Key PN"
@@
 F 0 "R805" H 8140 3830 50  0000 R CNN
 F 1 "10k" V 8220 3830 50  0000 C CNN
-F 2 "" H 8220 3830 50  0001 C CNN
+F 2 "Resistors_SMD:R_0603" H 8220 3830 50  0001 C CNN
 F 3 "" H 8220 3830 50  0001 C CNN
 F 4 "0603" H 8320 3910 50  0000 L CNN "display_footprint"
 F 5 "1%" H 8320 3830 50  0000 L CNN "Tolerance"
 F 6 "1/10W" H 8330 3750 50  0000 L CNN "Wattage"
-F 7 "PN" H 8520 4230 60  0001 C CNN "Digi-Key PN"
+F 7 "RHM10KADCT-ND" H 8520 4230 60  0001 C CNN "Digi-Key PN"
 	1    8220 3830
 	-1   0    0    -1
@@
 F 0 "R807" V 8800 4090 50  0000 C CNN
 F 1 "1k" V 8900 4090 50  0000 C CNN
-F 2 "" H 8900 4090 50  0001 C CNN
+F 2 "Resistors_SMD:R_0603" H 8900 4090 50  0001 C CNN
 F 3 "" H 8900 4090 50  0001 C CNN
 F 4 "0603" V 9000 4090 50  0000 C CNN "display_footprint"
 F 5 "1%" V 9100 4090 50  0000 C CNN "Tolerance"
 F 6 "1/10W" V 9200 4090 50  0000 C CNN "Wattage"
-F 7 "PN" H 9200 4490 60  0001 C CNN "Digi-Key PN"
+F 7 "MCT0603-1.00K-CFCT-ND" H 9200 4490 60  0001 C CNN "Digi-Key PN"
 	1    8900 4090
 	0    1    1    0
@@
 F 0 "R806" H 8140 4310 50  0000 R CNN
 F 1 "0" V 8220 4310 50  0000 C CNN
-F 2 "" H 8220 4310 50  0001 C CNN
+F 2 "Resistors_SMD:R_0603" H 8220 4310 50  0001 C CNN
 F 3 "" H 8220 4310 50  0001 C CNN
 F 4 "None" H 8140 4390 50  0000 R CNN "Config"
@@
 F 6 "1%" H 8320 4310 50  0000 L CNN "Tolerance"
 F 7 "1/10W" H 8330 4230 50  0000 L CNN "Wattage"
-F 8 "PN" H 8520 4710 60  0001 C CNN "Digi-Key PN"
+F 8 "" H 8520 4710 60  0001 C CNN "Digi-Key PN"
 	1    8220 4310
 	-1   0    0    1
@@
 F 0 "C808" H 8245 4710 50  0000 L CNN
 F 1 "0.1uF" H 8245 4510 50  0000 L CNN
-F 2 "" H 8258 4460 50  0001 C CNN
+F 2 "Capacitors_SMD:C_0603" H 8258 4460 50  0001 C CNN
 F 3 "" H 8245 4710 50  0001 C CNN
 F 4 "0603" H 8070 4710 50  0000 R CNN "display_footprint"
 F 5 "50V" H 8070 4610 50  0000 R CNN "Voltage"
 F 6 "X7R" H 8070 4510 50  0000 R CNN "Dielectric"
-F 7 "PN" H 8645 5110 60  0001 C CNN "Digi-Key PN"
+F 7 "490-8020-1-ND" H 8645 5110 60  0001 C CNN "Digi-Key PN"
 	1    8220 4610
 	1    0    0    -1
@@
 F 0 "C803" H 3655 5110 50  0000 L CNN
 F 1 "0.1uF" H 3655 4910 50  0000 L CNN
-F 2 "" H 3668 4860 50  0001 C CNN
+F 2 "Capacitors_SMD:C_0603" H 3668 4860 50  0001 C CNN
 F 3 "" H 3655 5110 50  0001 C CNN
 F 4 "0603" H 3480 5110 50  0000 R CNN "display_footprint"
 F 5 "50V" H 3480 5010 50  0000 R CNN "Voltage"
 F 6 "X7R" H 3480 4910 50  0000 R CNN "Dielectric"
-F 7 "PN" H 4055 5510 60  0001 C CNN "Digi-Key PN"
+F 7 "490-8020-1-ND" H 4055 5510 60  0001 C CNN "Digi-Key PN"
 	1    3630 5010
 	1    0    0    -1
@@
 F 0 "C804" H 4005 5110 50  0000 L CNN
 F 1 "10nF" H 4005 4910 50  0000 L CNN
-F 2 "" H 4018 4860 50  0001 C CNN
+F 2 "Capacitors_SMD:C_0603" H 4018 4860 50  0001 C CNN
 F 3 "" H 4005 5110 50  0001 C CNN
 F 4 "0603" H 3830 5110 50  0001 R CNN "display_footprint"
 F 5 "50V" H 3830 5010 50  0001 R CNN "Voltage"
 F 6 "X7R" H 3830 4910 50  0001 R CNN "Dielectric"
-F 7 "PN" H 4405 5510 60  0001 C CNN "Digi-Key PN"
+F 7 "1276-1921-1-ND" H 4405 5510 60  0001 C CNN "Digi-Key PN"
 	1    3980 5010
 	1    0    0    -1
@@
 F 0 "C805" H 4355 5110 50  0000 L CNN
 F 1 "1nF" H 4355 4910 50  0000 L CNN
-F 2 "" H 4368 4860 50  0001 C CNN
+F 2 "Capacitors_SMD:C_0603" H 4368 4860 50  0001 C CNN
 F 3 "" H 4355 5110 50  0001 C CNN
 F 4 "0603" H 4180 5110 50  0001 R CNN "display_footprint"
 F 5 "50V" H 4180 5010 50  0001 R CNN "Voltage"
 F 6 "X7R" H 4180 4910 50  0001 R CNN "Dielectric"
-F 7 "PN" H 4755 5510 60  0001 C CNN "Digi-Key PN"
+F 7 "478-1215-1-ND" H 4755 5510 60  0001 C CNN "Digi-Key PN"
 	1    4330 5010
 	1    0    0    -1
