File: hdw/AC_Power_Meter/Microcontroller_Programming.sch (KiCad schematic (older format))
At the start: 21 parts, among them J801 Prog, U801 TL331, U802 74LVC1G86

Commit message: A few routing adjustments and more graphics added to PCB
Connections:
- net labels added: ~MRST
- wire segments 38 -> 39
Changed lines of the file:
@@
 Wire Wire Line
 	3630 5280 3630 5200
+Text GLabel 7550 4090 0    50   Input ~ 0
+~MRST
+Wire Wire Line
+	7550 4090 8220 4090
 $EndSCHEMATC

Commit message: Serious BOM scrubbing to drive price down
Parts:
- removed C801, C802, C806: 0.1uF, Capacitors_SMD:C_0603, symbol Custom_Library:C_Custom
- removed R801, R802, R803: 10k, Resistors_SMD:R_0603, symbol Custom_Library:R_Custom
- removed R804: 0, Resistors_SMD:R_0603, symbol Custom_Library:R_Custom
- removed U801: TL331, TO_SOT_Packages_SMD:SOT-23-5, symbol Custom_Library:TL331
- removed U802: 74LVC1G86, TO_SOT_Packages_SMD:SOT-353_SC-70-5, symbol Custom_Library:74LVC1G86_Power
- removed Z801: UDZSTE-175.1B, Diodes_SMD:D_SOD-523, symbol Custom_Library:ZENER_Custom
- added SW801: MRESET, Buttons_Switches_THT:SW_PUSH_6mm, symbol Switch:SW_Push
Connections:
- net labels removed: +12V, ICSP_DETECT
- wire segments 39 -> 30
