File: hdw/AC_Power_Meter/OLED_Display.sch (KiCad schematic (older format))
At the start: 0 parts

Commit message: Added zero cross detect circuit
Parts:
- added U?: SSD1306, symbol Custom_Library:SSD1306
Connections:
- net labels added: +3.3V, GND
Changed lines of the file:
@@
 $Descr A 11000 8500
 encoding utf-8
-Sheet 1 13
+Sheet 12 15
 Title ""
 Date "2018-10-01"
@@
 Comment4 ""
 $EndDescr
+$Comp
+L Custom_Library:SSD1306 U?
+U 1 1 5BB30C5D
+P 5590 3410
+F 0 "U?" H 6090 3010 60  0000 C CNN
+F 1 "SSD1306" H 5590 3410 60  0000 C CNN
+F 2 "" H 5590 4110 60  0000 C CNN
+F 3 "" H 5590 4110 60  0000 C CNN
+	1    5590 3410
+	1    0    0    -1
+$EndComp
+$Comp
+L Custom_Library:+3.3V #PWR?
+U 1 1 5BB30CC0
+P 5590 2860
+F 0 "#PWR?" H 5590 2710 50  0001 C CNN
+F 1 "+3.3V" H 5590 3000 50  0000 C CNN
+F 2 "" H 5590 2860 50  0000 C CNN
+F 3 "" H 5590 2860 50  0000 C CNN
+	1    5590 2860
+	1    0    0    -1
+$EndComp
+$Comp
+L power:GND #PWR?
+U 1 1 5BB30D0E
+P 5590 3960
+F 0 "#PWR?" H 5590 3710 50  0001 C CNN
+F 1 "GND" H 5590 3810 50  0000 C CNN
+F 2 "" H 5590 3960 50  0001 C CNN
+F 3 "" H 5590 3960 50  0001 C CNN
+	1    5590 3960
+	1    0    0    -1
+$EndComp
 $EndSCHEMATC

Commit message: Added supporting parts for OLED display
Parts:
- added C?: 0.1uF, symbol Custom_Library:C_Custom
- added C?: 10nF, symbol Custom_Library:C_Custom
- added C?: 1nF, symbol Custom_Library:C_Custom
- added C?: 1uF, symbol Custom_Library:C_Custom
- added R? (x2): 10k, symbol Custom_Library:R_Custom
- added R? (x2): 0, Resistors_SMD:R_0603, symbol Device:R
Connections:
- net labels added: I2C_SCL, I2C_SDA
- wire segments 0 -> 18

Commit message: Added MU logo and titles to all sheets
Other:
- note added: "OLED Display"
Changed lines of the file:
@@
+	1    0    0    -1
+$EndComp
+Text Notes 540  690  0    100  ~ 20
+OLED Display
+$Comp
+L Mu_Logo:LOGO #G?
+U 1 1 5BBF7298
+P 9900 1000
+F 0 "#G?" H 9900 670 60  0001 C CNN
+F 1 "LOGO" H 9900 1330 60  0001 C CNN
+F 2 "" H 9900 1000 50  0001 C CNN
+F 3 "" H 9900 1000 50  0001 C CNN
+	1    9900 1000
 	1    0    0    -1
 $EndComp

Commit message: Updated MU logo to crisper image
Changed lines of the file:
@@
 OLED Display
 $Comp
-L Mu_Logo:LOGO #G?
-U 1 1 5BBF7298
-P 9900 1000
-F 0 "#G?" H 9900 670 60  0001 C CNN
-F 1 "LOGO" H 9900 1330 60  0001 C CNN
-F 2 "" H 9900 1000 50  0001 C CNN
-F 3 "" H 9900 1000 50  0001 C CNN
-	1    9900 1000
+L Custom_Library:MU_Logo #G?
+U 1 1 5BB6A1B9
+P 9900 1100
+F 0 "#G?" H 9900 614 60  0001 C CNN
+F 1 "MU_Logo" H 9900 1586 60  0001 C CNN
+F 2 "" H 9900 1100 50  0001 C CNN
+F 3 "" H 9900 1100 50  0001 C CNN
+	1    9900 1100
 	1    0    0    -1
 $EndComp

Commit message: Rewired a few micro symbols, add FMW notes
Parts:
- gave numbers to parts that had none: 9
Changed lines of the file:
@@
 $Descr A 11000 8500
 encoding utf-8
-Sheet 12 17
+Sheet 12 18
 Title ""
 Date "2018-10-01"
@@
 $EndDescr
 $Comp
-L Custom_Library:SSD1306 U?
+L Custom_Library:SSD1306 U1201
 U 1 1 5BB30C5D
 P 6600 3580
-F 0 "U?" H 7100 3180 60  0000 C CNN
+F 0 "U1201" H 7100 3180 60  0000 C CNN
 F 1 "SSD1306" H 6600 3580 60  0000 C CNN
 F 2 "" H 6600 4280 60  0000 C CNN
@@
 $EndComp
 $Comp
-L Custom_Library:+3.3V #PWR?
+L Custom_Library:+3.3V #PWR01205
 U 1 1 5BB30CC0
 P 6600 3030
-F 0 "#PWR?" H 6600 2880 50  0001 C CNN
+F 0 "#PWR01205" H 6600 2880 50  0001 C CNN
 F 1 "+3.3V" H 6600 3170 50  0000 C CNN
 F 2 "" H 6600 3030 50  0000 C CNN
@@
 $EndComp
 $Comp
-L power:GND #PWR?
+L power:GND #PWR01206
 U 1 1 5BB30D0E
 P 6600 4130
-F 0 "#PWR?" H 6600 3880 50  0001 C CNN
+F 0 "#PWR01206" H 6600 3880 50  0001 C CNN
 F 1 "GND" H 6600 3980 50  0000 C CNN
 F 2 "" H 6600 4130 50  0001 C CNN
@@
 P 5540 3160
 AR Path="/5BB27BA3/5BB4077B" Ref="R?"  Part="1"
-AR Path="/5BB27BF7/5BB4077B" Ref="R?"  Part="1"
-F 0 "R?" H 5460 3160 50  0000 R CNN
+AR Path="/5BB27BF7/5BB4077B" Ref="R1204"  Part="1"
+F 0 "R1204" H 5460 3160 50  0000 R CNN
 F 1 "10k" V 5540 3160 50  0000 C CNN
 F 2 "" H 5540 3160 50  0001 C CNN
@@
 P 4790 3160
 AR Path="/5BB27BA3/5BB4078A" Ref="R?"  Part="1"
-AR Path="/5BB27BF7/5BB4078A" Ref="R?"  Part="1"
-F 0 "R?" H 4710 3160 50  0000 R CNN
+AR Path="/5BB27BF7/5BB4078A" Ref="R1203"  Part="1"
+F 0 "R1203" H 4710 3160 50  0000 R CNN
 F 1 "10k" V 4790 3160 50  0000 C CNN
 F 2 "" H 4790 3160 50  0001 C CNN
@@
 $EndComp
 $Comp
-L Custom_Library:+3.3V #PWR?
+L Custom_Library:+3.3V #PWR01202
 U 1 1 5BB407B8
 P 5540 3010
-F 0 "#PWR?" H 5540 2860 50  0001 C CNN
+F 0 "#PWR01202" H 5540 2860 50  0001 C CNN
 F 1 "+3.3V" H 5540 3150 50  0000 C CNN
 F 2 "" H 5540 3010 50  0000 C CNN
@@
 $EndComp
 $Comp
-L Custom_Library:+3.3V #PWR?
+L Custom_Library:+3.3V #PWR01201
 U 1 1 5BB407C9
 P 4790 3010
-F 0 "#PWR?" H 4790 2860 50  0001 C CNN
+F 0 "#PWR01201" H 4790 2860 50  0001 C CNN
 F 1 "+3.3V" H 4790 3150 50  0000 C CNN
 F 2 "" H 4790 3010 50  0000 C CNN
@@
 AR Path="/5A0A8BD0/5BB4162C" Ref="R?"  Part="1"
 AR Path="/5BB27BCC/5BB4162C" Ref="R?"  Part="1"
-AR Path="/5BB27BF7/5BB4162C" Ref="R?"  Part="1"
-F 0 "R?" V 4020 3530 50  0000 C CNN
+AR Path="/5BB27BF7/5BB4162C" Ref="R1201"  Part="1"
+F 0 "R1201" V 4020 3530 50  0000 C CNN
 F 1 "0" V 3940 3530 50  0000 C CNN
 F 2 "Resistors_SMD:R_0603" V 3870 3530 50  0001 C CNN
@@
 AR Path="/5A0A8BD0/5BB41637" Ref="R?"  Part="1"
 AR Path="/5BB27BCC/5BB41637" Ref="R?"  Part="1"
-AR Path="/5BB27BF7/5BB41637" Ref="R?"  Part="1"
-F 0 "R?" V 4020 3630 50  0000 C CNN
+AR Path="/5BB27BF7/5BB41637" Ref="R1202"  Part="1"
+F 0 "R1202" V 4020 3630 50  0000 C CNN
 F 1 "0" V 3940 3630 50  0000 C CNN
 F 2 "Resistors_SMD:R_0603" V 3870 3630 50  0001 C CNN
@@
 AR Path="/5BB27B24/5BB42E4B" Ref="C?"  Part="1"
 AR Path="/5BB27BB5/5BB42E4B" Ref="C?"  Part="1"
-AR Path="/5BB27BF7/5BB42E4B" Ref="C?"  Part="1"
-F 0 "C?" H 5605 5240 50  0000 L CNN
+AR Path="/5BB27BF7/5BB42E4B" Ref="C1201"  Part="1"
+F 0 "C1201" H 5605 5240 50  0000 L CNN
 F 1 "0.1uF" H 5605 5040 50  0000 L CNN
 F 2 "" H 5618 4990 50  0001 C CNN
@@
 AR Path="/5BB27B24/5BB42E56" Ref="C?"  Part="1"
 AR Path="/5BB27BB5/5BB42E56" Ref="C?"  Part="1"
-AR Path="/5BB27BF7/5BB42E56" Ref="C?"  Part="1"
-F 0 "C?" H 5955 5240 50  0000 L CNN
+AR Path="/5BB27BF7/5BB42E56" Ref="C1202"  Part="1"
+F 0 "C1202" H 5955 5240 50  0000 L CNN
 F 1 "10nF" H 5955 5040 50  0000 L CNN
 F 2 "" H 5968 4990 50  0001 C CNN
@@
 AR Path="/5BB27B24/5BB42E61" Ref="C?"  Part="1"
 AR Path="/5BB27BB5/5BB42E61" Ref="C?"  Part="1"
-AR Path="/5BB27BF7/5BB42E61" Ref="C?"  Part="1"
-F 0 "C?" H 6305 5240 50  0000 L CNN
+AR Path="/5BB27BF7/5BB42E61" Ref="C1203"  Part="1"
+F 0 "C1203" H 6305 5240 50  0000 L CNN
 F 1 "1nF" H 6305 5040 50  0000 L CNN
 F 2 "" H 6318 4990 50  0001 C CNN
@@
 AR Path="/5BB27B24/5BB42E68" Ref="#PWR?"  Part="1"
 AR Path="/5BB27BB5/5BB42E68" Ref="#PWR?"  Part="1"
-AR Path="/5BB27BF7/5BB42E68" Ref="#PWR?"  Part="1"
-F 0 "#PWR?" H 5930 5120 50  0001 C CNN
+AR Path="/5BB27BF7/5BB42E68" Ref="#PWR01204"  Part="1"
+F 0 "#PWR01204" H 5930 5120 50  0001 C CNN
 F 1 "GND" H 5930 5220 50  0000 C CNN
 F 2 "" H 5930 5370 50  0001 C CNN
@@
 AR Path="/5BB27B24/5BB42E6E" Ref="#PWR?"  Part="1"
 AR Path="/5BB27BB5/5BB42E6E" Ref="#PWR?"  Part="1"
-AR Path="/5BB27BF7/5BB42E6E" Ref="#PWR?"  Part="1"
-F 0 "#PWR?" H 5930 4760 50  0001 C CNN
+AR Path="/5BB27BF7/5BB42E6E" Ref="#PWR01203"  Part="1"
+F 0 "#PWR01203" H 5930 4760 50  0001 C CNN
 F 1 "+3.3V" H 5930 5050 50  0000 C CNN
 F 2 "" H 5930 4910 50  0000 C CNN
@@
 AR Path="/5BB27B24/5BB42E9D" Ref="C?"  Part="1"
 AR Path="/5BB27BB5/5BB42E9D" Ref="C?"  Part="1"
-AR Path="/5BB27BF7/5BB42E9D" Ref="C?"  Part="1"
-F 0 "C?" H 6995 5240 50  0000 L CNN
+AR Path="/5BB27BF7/5BB42E9D" Ref="C1204"  Part="1"
+F 0 "C1204" H 6995 5240 50  0000 L CNN
 F 1 "1uF" H 6995 5040 50  0000 L CNN
 F 2 "" H 7008 4990 50  0001 C CNN
@@
 AR Path="/5BB27B24/5BB42EA4" Ref="#PWR?"  Part="1"
 AR Path="/5BB27BB5/5BB42EA4" Ref="#PWR?"  Part="1"
-AR Path="/5BB27BF7/5BB42EA4" Ref="#PWR?"  Part="1"
-F 0 "#PWR?" H 6970 5040 50  0001 C CNN
+AR Path="/5BB27BF7/5BB42EA4" Ref="#PWR01208"  Part="1"
+F 0 "#PWR01208" H 6970 5040 50  0001 C CNN
 F 1 "GND" H 6970 5140 50  0000 C CNN
 F 2 "" H 6970 5290 50  0001 C CNN
@@
 AR Path="/5BB27B24/5BB42EAA" Ref="#PWR?"  Part="1"
 AR Path="/5BB27BB5/5BB42EAA" Ref="#PWR?"  Part="1"
-AR Path="/5BB27BF7/5BB42EAA" Ref="#PWR?"  Part="1"
-F 0 "#PWR?" H 6970 4840 50  0001 C CNN
+AR Path="/5BB27BF7/5BB42EAA" Ref="#PWR01207"  Part="1"
+F 0 "#PWR01207" H 6970 4840 50  0001 C CNN
 F 1 "+3.3V" H 6970 5130 50  0000 C CNN
 F 2 "" H 6970 4990 50  0000 C CNN
@@
 OLED Display
 $Comp
-L Custom_Library:MU_Logo #G?
+L Custom_Library:MU_Logo #G1201
 U 1 1 5BB6A1B9
 P 9900 1100
-F 0 "#G?" H 9900 614 60  0001 C CNN
+F 0 "#G1201" H 9900 614 60  0001 C CNN
 F 1 "MU_Logo" H 9900 1586 60  0001 C CNN
 F 2 "" H 9900 1100 50  0001 C CNN

Commit message: Updated most footprints
Parts:
- C1201: footprint (none) -> Capacitors_SMD:C_0603; Digi-Key PN PN -> 490-8020-1-ND
- C1202: footprint (none) -> Capacitors_SMD:C_0603; Digi-Key PN PN -> 1276-1921-1-ND
- C1203: footprint (none) -> Capacitors_SMD:C_0603; Digi-Key PN PN -> 478-1215-1-ND
- C1204: footprint (none) -> Capacitors_SMD:C_0805; Digi-Key PN PN -> 490-1695-1-ND
- R1201, R1202: Digi-Key PN (none) -> P0.0GCT-ND
- R1203, R1204: footprint (none) -> Resistors_SMD:R_0603; Digi-Key PN PN -> RHM10KADCT-ND
- U1201: footprint (none) -> Pin_Headers:Pin_Header_Straight_1x04_Pitch2.54mm
Changed lines of the file:
@@
 F 0 "U1201" H 7100 3180 60  0000 C CNN
 F 1 "SSD1306" H 6600 3580 60  0000 C CNN
-F 2 "" H 6600 4280 60  0000 C CNN
+F 2 "Pin_Headers:Pin_Header_Straight_1x04_Pitch2.54mm" H 6600 4280 60  0001 C CNN
 F 3 "" H 6600 4280 60  0000 C CNN
 	1    6600 3580
@@
 F 0 "R1204" H 5460 3160 50  0000 R CNN
 F 1 "10k" V 5540 3160 50  0000 C CNN
-F 2 "" H 5540 3160 50  0001 C CNN
+F 2 "Resistors_SMD:R_0603" H 5540 3160 50  0001 C CNN
 F 3 "" H 5540 3160 50  0001 C CNN
 F 4 "0603" H 5640 3240 50  0000 L CNN "display_footprint"
 F 5 "1%" H 5640 3160 50  0000 L CNN "Tolerance"
 F 6 "1/10W" H 5650 3080 50  0000 L CNN "Wattage"
-F 7 "PN" H 5840 3560 60  0001 C CNN "Digi-Key PN"
+F 7 "RHM10KADCT-ND" H 5840 3560 60  0001 C CNN "Digi-Key PN"
 	1    5540 3160
 	1    0    0    -1
@@
 F 0 "R1203" H 4710 3160 50  0000 R CNN
 F 1 "10k" V 4790 3160 50  0000 C CNN
-F 2 "" H 4790 3160 50  0001 C CNN
+F 2 "Resistors_SMD:R_0603" H 4790 3160 50  0001 C CNN
 F 3 "" H 4790 3160 50  0001 C CNN
 F 4 "0603" H 4890 3240 50  0000 L CNN "display_footprint"
 F 5 "1%" H 4890 3160 50  0000 L CNN "Tolerance"
 F 6 "1/10W" H 4900 3080 50  0000 L CNN "Wattage"
-F 7 "PN" H 5090 3560 60  0001 C CNN "Digi-Key PN"
+F 7 "RHM10KADCT-ND" H 5090 3560 60  0001 C CNN "Digi-Key PN"
 	1    4790 3160
 	1    0    0    -1
@@
 F 5 "1/10W" V 3840 3530 50  0001 C CNN "Wattage"
 F 6 "0603" V 3760 3530 50  0001 C CNN "display_footprint"
+F 7 "P0.0GCT-ND" H 0   0   50  0001 C CNN "Digi-Key PN"
 	1    3940 3530
 	0    -1   -1   0
@@
 F 5 "1/10W" V 3840 3630 50  0001 C CNN "Wattage"
 F 6 "0603" V 3760 3630 50  0001 C CNN "display_footprint"
+F 7 "P0.0GCT-ND" H 0   0   50  0001 C CNN "Digi-Key PN"
 	1    3940 3630
 	0    1    1    0
@@
 F 0 "C1201" H 5605 5240 50  0000 L CNN
 F 1 "0.1uF" H 5605 5040 50  0000 L CNN
-F 2 "" H 5618 4990 50  0001 C CNN
+F 2 "Capacitors_SMD:C_0603" H 5618 4990 50  0001 C CNN
 F 3 "" H 5605 5240 50  0001 C CNN
 F 4 "0603" H 5430 5240 50  0000 R CNN "display_footprint"
 F 5 "50V" H 5430 5140 50  0000 R CNN "Voltage"
 F 6 "X7R" H 5430 5040 50  0000 R CNN "Dielectric"
-F 7 "PN" H 6005 5640 60  0001 C CNN "Digi-Key PN"
+F 7 "490-8020-1-ND" H 6005 5640 60  0001 C CNN "Digi-Key PN"
 	1    5580 5140
 	1    0    0    -1
@@
 F 0 "C1202" H 5955 5240 50  0000 L CNN
 F 1 "10nF" H 5955 5040 50  0000 L CNN
-F 2 "" H 5968 4990 50  0001 C CNN
+F 2 "Capacitors_SMD:C_0603" H 5968 4990 50  0001 C CNN
 F 3 "" H 5955 5240 50  0001 C CNN
 F 4 "0603" H 5780 5240 50  0001 R CNN "display_footprint"
 F 5 "50V" H 5780 5140 50  0001 R CNN "Voltage"
 F 6 "X7R" H 5780 5040 50  0001 R CNN "Dielectric"
-F 7 "PN" H 6355 5640 60  0001 C CNN "Digi-Key PN"
+F 7 "1276-1921-1-ND" H 6355 5640 60  0001 C CNN "Digi-Key PN"
 	1    5930 5140
 	1    0    0    -1
@@
 F 0 "C1203" H 6305 5240 50  0000 L CNN
 F 1 "1nF" H 6305 5040 50  0000 L CNN
-F 2 "" H 6318 4990 50  0001 C CNN
+F 2 "Capacitors_SMD:C_0603" H 6318 4990 50  0001 C CNN
 F 3 "" H 6305 5240 50  0001 C CNN
 F 4 "0603" H 6130 5240 50  0001 R CNN "display_footprint"
 F 5 "50V" H 6130 5140 50  0001 R CNN "Voltage"
 F 6 "X7R" H 6130 5040 50  0001 R CNN "Dielectric"
-F 7 "PN" H 6705 5640 60  0001 C CNN "Digi-Key PN"
+F 7 "478-1215-1-ND" H 6705 5640 60  0001 C CNN "Digi-Key PN"
 	1    6280 5140
 	1    0    0    -1
@@
 F 0 "C1204" H 6995 5240 50  0000 L CNN
 F 1 "1uF" H 6995 5040 50  0000 L CNN
-F 2 "" H 7008 4990 50  0001 C CNN
+F 2 "Capacitors_SMD:C_0805" H 7008 4990 50  0001 C CNN
 F 3 "" H 6995 5240 50  0001 C CNN
 F 4 "0805" H 6820 5240 50  0000 R CNN "display_footprint"
 F 5 "10V" H 6820 5140 50  0000 R CNN "Voltage"
 F 6 "X7R" H 6820 5040 50  0000 R CNN "Dielectric"
-F 7 "PN" H 7395 5640 60  0001 C CNN "Digi-Key PN"
+F 7 "490-1695-1-ND" H 7395 5640 60  0001 C CNN "Digi-Key PN"
 	1    6970 5140
 	1    0    0    -1
