File: hdw/AC_Power_Meter/Sensor_Signal_Conditioning.sch (KiCad schematic (older format))
At the start: 19 parts

Commit message: Added MU logo and titles to all sheets
Other:
- note added: "Current Sensing Peak Detector, ADC Buffer"
Changed lines of the file:
@@
 Text Notes 8340 3400 0    50   ~ 0
 66mV/A, with a 1.65V offset\n(2.65V = 15A)
+Text Notes 540  690  0    100  ~ 20
+Current Sensing Peak Detector, ADC Buffer
+$Comp
+L Mu_Logo:LOGO #G?
+U 1 1 5BBF4E2D
+P 9900 1000
+F 0 "#G?" H 9900 670 60  0001 C CNN
+F 1 "LOGO" H 9900 1330 60  0001 C CNN
+F 2 "" H 9900 1000 50  0001 C CNN
+F 3 "" H 9900 1000 50  0001 C CNN
+	1    9900 1000
+	1    0    0    -1
+$EndComp
 $EndSCHEMATC

Commit message: Updated MU logo to crisper image
Changed lines of the file:
@@
 Current Sensing Peak Detector, ADC Buffer
 $Comp
-L Mu_Logo:LOGO #G?
-U 1 1 5BBF4E2D
-P 9900 1000
-F 0 "#G?" H 9900 670 60  0001 C CNN
-F 1 "LOGO" H 9900 1330 60  0001 C CNN
-F 2 "" H 9900 1000 50  0001 C CNN
-F 3 "" H 9900 1000 50  0001 C CNN
-	1    9900 1000
+L Custom_Library:MU_Logo #G?
+U 1 1 5BB69544
+P 9900 1100
+F 0 "#G?" H 9900 614 60  0001 C CNN
+F 1 "MU_Logo" H 9900 1586 60  0001 C CNN
+F 2 "" H 9900 1100 50  0001 C CNN
+F 3 "" H 9900 1100 50  0001 C CNN
+	1    9900 1100
 	1    0    0    -1
 $EndComp

Commit message: Revised signal conditioning, cleaned up a lot of pages
Parts:
- removed C? (x2): 0.1uF, symbol Custom_Library:C_Custom
- removed C? (x2): 10nF, symbol Custom_Library:C_Custom
- removed C? (x2): 1nF, symbol Custom_Library:C_Custom
- removed C? (x2): 10uF, symbol Custom_Library:C_Custom
- removed C? (x2): 1uF, symbol Custom_Library:C_Custom
- added C? (x4): 0.1uF, symbol Custom_Library:C_Custom
- added C? (x4): 10nF, symbol Custom_Library:C_Custom
- added C? (x4): 1nF, symbol Custom_Library:C_Custom
- added C? (x4): 10uF, symbol Custom_Library:C_Custom
- added C? (x4): 1uF, symbol Custom_Library:C_Custom
- added R? (x4): 10k, symbol Custom_Library:R_Custom
- added R?: 3.3k, symbol Custom_Library:R_Custom
- added U? (x2): LTC6240IS5, Package_TO_SOT_SMD:SOT-23-5, symbol Custom_Library:LTC6240IS5
- R?: value 1k -> 10k
- R?: value 100k -> 1M
Connections:
- net labels added: +0.825V_REF
- wire segments 44 -> 88
Other:
- note added: "ISNS_ADC Scaling: 5.35ARMS/V"
- note added: "Offset Removal, Active Peak Detector, 2V/V Gain Stage"
- note removed: "66mV/A, with a 1.65V offset\n(2.65V = 15A)"
- note removed: "Current Sensing Peak Detector, ADC Buffer"

Commit message: Rewired a few micro symbols, add FMW notes
Parts:
- gave numbers to parts that had none: 36

Commit message: Updated most footprints
Parts:
- C901, C902, C911, C917: footprint (none) -> Capacitors_SMD:C_0603; Digi-Key PN PN -> 490-8020-1-ND
- C903, C904, C912, C918: footprint (none) -> Capacitors_SMD:C_0603; Digi-Key PN PN -> 1276-1921-1-ND
- C905, C906, C913, C919: footprint (none) -> Capacitors_SMD:C_0603; Digi-Key PN PN -> 478-1215-1-ND
- C907, C908, C914, C916, C920: footprint (none) -> Capacitors_SMD:C_0805; Digi-Key PN PN -> 490-10517-1-ND
- C909, C910, C915, C921: footprint (none) -> Capacitors_SMD:C_0805; Digi-Key PN PN -> 490-1695-1-ND
- D901: Digi-Key PN (none) -> 1N4148WSFSCT-ND
- R901, R902, R904, R905, R906, R909, R910: footprint (none) -> Resistors_SMD:R_0603; Digi-Key PN PN -> RHM10KADCT-ND
- R903: footprint (none) -> Resistors_SMD:R_0603; Digi-Key PN PN -> 311-3.30KHRCT-ND
- R907: footprint (none) -> Resistors_SMD:R_0603; Digi-Key PN PN -> A130109CT-ND
- R908: footprint (none) -> Resistors_SMD:R_0603; Digi-Key PN PN -> MCT0603-1.00K-CFCT-ND
- U903, U904: Digi-Key PN (none) -> LTC6240IS5#TRMPBFCT-ND
