File: hdw/AC_Power_Meter/Sensor_Signal_Conditioning.sch (KiCad schematic (older format))
At the start: 36 parts, among them U901 LTC6240IS5, U902 LTC6240IS5, U903 LTC6240IS5, U904 LTC6240IS5

Commit message: Arranged a few pages of components
Parts:
- U901, U902, U903, U904: footprint Package_TO_SOT_SMD:SOT-23-5 -> TO_SOT_Packages_SMD:SOT-23-5
Changed lines of the file:
@@
 F 0 "U904" H 9140 3530 50  0000 L CNN
 F 1 "LTC6240IS5" H 9140 3130 50  0000 L CNN
-F 2 "Package_TO_SOT_SMD:SOT-23-5" H 9140 3330 50  0001 C CNN
+F 2 "TO_SOT_Packages_SMD:SOT-23-5" H 9140 3330 50  0001 C CNN
 F 3 "http://www.analog.com/media/en/technical-documentation/data-sheets/624012fe.pdf" H 9140 3330 50  0001 C CNN
 F 4 "LTC6240IS5#TRMPBFCT-ND" H 0   0   50  0001 C CNN "Digi-Key PN"
@@
 F 0 "U903" H 4990 3430 50  0000 L CNN
 F 1 "LTC6240IS5" H 4990 3030 50  0000 L CNN
-F 2 "Package_TO_SOT_SMD:SOT-23-5" H 4990 3230 50  0001 C CNN
+F 2 "TO_SOT_Packages_SMD:SOT-23-5" H 4990 3230 50  0001 C CNN
 F 3 "http://www.analog.com/media/en/technical-documentation/data-sheets/624012fe.pdf" H 4990 3230 50  0001 C CNN
 F 4 "LTC6240IS5#TRMPBFCT-ND" H 0   0   50  0001 C CNN "Digi-Key PN"
@@
 F 0 "U901" H 2660 3330 50  0000 L CNN
 F 1 "LTC6240IS5" H 2660 2930 50  0000 L CNN
-F 2 "Package_TO_SOT_SMD:SOT-23-5" H 2660 3130 50  0001 C CNN
+F 2 "TO_SOT_Packages_SMD:SOT-23-5" H 2660 3130 50  0001 C CNN
 F 3 "http://www.analog.com/media/en/technical-documentation/data-sheets/624012fe.pdf" H 2660 3130 50  0001 C CNN
 F 4 "LTC6240IS5#TRMPBFCT-ND" H -4160 -380 50  0001 C CNN "Digi-Key PN"
@@
 F 0 "U902" H 2660 6380 50  0000 L CNN
 F 1 "LTC6240IS5" H 2660 5980 50  0000 L CNN
-F 2 "Package_TO_SOT_SMD:SOT-23-5" H 2660 6180 50  0001 C CNN
+F 2 "TO_SOT_Packages_SMD:SOT-23-5" H 2660 6180 50  0001 C CNN
 F 3 "http://www.analog.com/media/en/technical-documentation/data-sheets/624012fe.pdf" H 2660 6180 50  0001 C CNN
 F 4 "LTC6240IS5#TRMPBFCT-ND" H -4160 2670 50  0001 C CNN "Digi-Key PN"

Commit message: Nailed down board outline, placed a few sections
Parts:
- D901: footprint Diode_SMD:D_SOD-323 -> Diodes_SMD:D_SOD-323
Changed lines of the file:
@@
 F 0 "D901" H 5740 3330 50  0000 C CNN
 F 1 "1N4148WS" H 5740 3130 50  0000 C CNN
-F 2 "Diode_SMD:D_SOD-323" H 5740 3055 50  0001 C CNN
+F 2 "Diodes_SMD:D_SOD-323" H 5740 3055 50  0001 C CNN
 F 3 "https://www.vishay.com/docs/85751/1n4148ws.pdf" H 5740 3230 50  0001 C CNN
 F 4 "1N4148WSFSCT-ND" H 5740 3230 50  0001 C CNN "Digi-Key PN"

Commit message: Added a lot of functionality in formware
Other:
- note added: "ISNS_ADC Scaling: 3.787Apk/2V"
- note removed: "ISNS_ADC Scaling: 5.35ARMS/V"
Changed lines of the file:
@@
 	9200 2680 9560 2680
 Text Notes 8500 5340 0    50   ~ 0
-ISNS_ADC Scaling: 5.35ARMS/V
+ISNS_ADC Scaling: 3.787Apk/2V
 $Comp
 L Custom_Library:LTC6240IS5 U?
