File: hdw/AC_Power_Meter/Zero_Cross_Detect.sch (KiCad schematic (older format))
At the start: 12 parts

Commit message: Added TRIAC circuit and POS12 AC/DC converter
Parts:
- added C?: 0.1uF, symbol Custom_Library:C_Custom
- added R?: 10k, symbol Custom_Library:R_Custom
- added U?: 74LVC1G17, symbol Custom_Library:74LVC1G17_Power
Connections:
- net labels added: Zero_Cross_Detect
- net labels removed: ZCD_OUT
- wire segments 39 -> 42
Changed lines of the file:
@@
 Wire Wire Line
 	3460 4010 3460 4130
-Text GLabel 6540 3870 2    50   Output ~ 0
-ZCD_OUT
-Wire Wire Line
-	6540 3870 6460 3870
 Connection ~ 6460 3870
 $Comp
 L Custom_Library:C_Custom C?
 U 1 1 5BB38E0F
-P 7210 3140
+P 6710 2700
 AR Path="/5BB27BA3/5BB38E0F" Ref="C?"  Part="1"
 AR Path="/5BB27B84/5BB38E0F" Ref="C?"  Part="1"
-F 0 "C?" H 7235 3240 50  0000 L CNN
-F 1 "0.1uF" H 7235 3040 50  0000 L CNN
-F 2 "" H 7248 2990 50  0001 C CNN
-F 3 "" H 7235 3240 50  0001 C CNN
-F 4 "0603" H 7060 3240 50  0000 R CNN "display_footprint"
-F 5 "50V" H 7060 3140 50  0000 R CNN "Voltage"
-F 6 "X7R" H 7060 3040 50  0000 R CNN "Dielectric"
-F 7 "PN" H 7635 3640 60  0001 C CNN "Digi-Key PN"
-	1    7210 3140
+AR Path="/5BB31311/5BB38E0F" Ref="C?"  Part="1"
+F 0 "C?" H 6735 2800 50  0000 L CNN
+F 1 "0.1uF" H 6735 2600 50  0000 L CNN
+F 2 "" H 6748 2550 50  0001 C CNN
+F 3 "" H 6735 2800 50  0001 C CNN
+F 4 "0603" H 6560 2800 50  0000 R CNN "display_footprint"
+F 5 "50V" H 6560 2700 50  0000 R CNN "Voltage"
+F 6 "X7R" H 6560 2600 50  0000 R CNN "Dielectric"
+F 7 "PN" H 7135 3200 60  0001 C CNN "Digi-Key PN"
+	1    6710 2700
 	1    0    0    -1
 $EndComp
@@
 L Custom_Library:C_Custom C?
 U 1 1 5BB38E1A
-P 7560 3140
+P 7060 2700
 AR Path="/5BB27BA3/5BB38E1A" Ref="C?"  Part="1"
 AR Path="/5BB27B84/5BB38E1A" Ref="C?"  Part="1"
-F 0 "C?" H 7585 3240 50  0000 L CNN
-F 1 "10nF" H 7585 3040 50  0000 L CNN
-F 2 "" H 7598 2990 50  0001 C CNN
-F 3 "" H 7585 3240 50  0001 C CNN
-F 4 "0603" H 7410 3240 50  0001 R CNN "display_footprint"
-F 5 "50V" H 7410 3140 50  0001 R CNN "Voltage"
-F 6 "X7R" H 7410 3040 50  0001 R CNN "Dielectric"
-F 7 "PN" H 7985 3640 60  0001 C CNN "Digi-Key PN"
-	1    7560 3140
+AR Path="/5BB31311/5BB38E1A" Ref="C?"  Part="1"
+F 0 "C?" H 7085 2800 50  0000 L CNN
+F 1 "10nF" H 7085 2600 50  0000 L CNN
+F 2 "" H 7098 2550 50  0001 C CNN
+F 3 "" H 7085 2800 50  0001 C CNN
+F 4 "0603" H 6910 2800 50  0001 R CNN "display_footprint"
+F 5 "50V" H 6910 2700 50  0001 R CNN "Voltage"
+F 6 "X7R" H 6910 2600 50  0001 R CNN "Dielectric"
+F 7 "PN" H 7485 3200 60  0001 C CNN "Digi-Key PN"
+	1    7060 2700
 	1    0    0    -1
 $EndComp
@@
 L Custom_Library:C_Custom C?
 U 1 1 5BB38E25
-P 7910 3140
+P 7410 2700
 AR Path="/5BB27BA3/5BB38E25" Ref="C?"  Part="1"
 AR Path="/5BB27B84/5BB38E25" Ref="C?"  Part="1"
-F 0 "C?" H 7935 3240 50  0000 L CNN
-F 1 "1nF" H 7935 3040 50  0000 L CNN
-F 2 "" H 7948 2990 50  0001 C CNN
-F 3 "" H 7935 3240 50  0001 C CNN
-F 4 "0603" H 7760 3240 50  0001 R CNN "display_footprint"
-F 5 "50V" H 7760 3140 50  0001 R CNN "Voltage"
-F 6 "X7R" H 7760 3040 50  0001 R CNN "Dielectric"
-F 7 "PN" H 8335 3640 60  0001 C CNN "Digi-Key PN"
-	1    7910 3140
+AR Path="/5BB31311/5BB38E25" Ref="C?"  Part="1"
+F 0 "C?" H 7435 2800 50  0000 L CNN
+F 1 "1nF" H 7435 2600 50  0000 L CNN
+F 2 "" H 7448 2550 50  0001 C CNN
+F 3 "" H 7435 2800 50  0001 C CNN
+F 4 "0603" H 7260 2800 50  0001 R CNN "display_footprint"
+F 5 "50V" H 7260 2700 50  0001 R CNN "Voltage"
+F 6 "X7R" H 7260 2600 50  0001 R CNN "Dielectric"
+F 7 "PN" H 7835 3200 60  0001 C CNN "Digi-Key PN"
+	1    7410 2700
 	1    0    0    -1
 $EndComp
@@
 L power:GND #PWR?
 U 1 1 5BB38E2C
-P 7560 3370
-F 0 "#PWR?" H 7560 3120 50  0001 C CNN
-F 1 "GND" H 7560 3220 50  0000 C CNN
-F 2 "" H 7560 3370 50  0001 C CNN
-F 3 "" H 7560 3370 50  0001 C CNN
-	1    7560 3370
+P 7060 2930
+F 0 "#PWR?" H 7060 2680 50  0001 C CNN
+F 1 "GND" H 7060 2780 50  0000 C CNN
+F 2 "" H 7060 2930 50  0001 C CNN
+F 3 "" H 7060 2930 50  0001 C CNN
+	1    7060 2930
 	1    0    0    -1
 $EndComp
@@
 L Custom_Library:+3.3V #PWR?
 U 1 1 5BB38E32
-P 7560 2910
-F 0 "#PWR?" H 7560 2760 50  0001 C CNN
-F 1 "+3.3V" H 7560 3050 50  0000 C CNN
-F 2 "" H 7560 2910 50  0000 C CNN
-F 3 "" H 7560 2910 50  0000 C CNN
-	1    7560 2910
-	1    0    0    -1
-$EndComp
-Wire Wire Line
-	7560 2910 7560 2950
-Wire Wire Line
-	7560 2950 7910 2950
-Wire Wire Line
-	7910 2950 7910 2990
-Connection ~ 7560 2950
-Wire Wire Line
-	7560 2950 7560 2990
-Wire Wire Line
-	7560 2950 7210 2950
-Wire Wire Line
-	7210 2950 7210 2990
-Wire Wire Line
-	7560 3290 7560 3330
-Wire Wire Line
-	7560 3330 7910 3330
-Wire Wire Line
-	7910 3330 7910 3290
-Connection ~ 7560 3330
-Wire Wire Line
-	7560 3330 7560 3370
-Wire Wire Line
-	7560 3330 7210 3330
-Wire Wire Line
-	7210 3330 7210 3290
+P 7060 2470
+F 0 "#PWR?" H 7060 2320 50  0001 C CNN
+F 1 "+3.3V" H 7060 2610 50  0000 C CNN
+F 2 "" H 7060 2470 50  0000 C CNN
+F 3 "" H 7060 2470 50  0000 C CNN
+	1    7060 2470
+	1    0    0    -1
+$EndComp
+Wire Wire Line
+	7060 2470 7060 2510
+Wire Wire Line
+	7060 2510 7410 2510
+Wire Wire Line
+	7410 2510 7410 2550
+Connection ~ 7060 2510
+Wire Wire Line
+	7060 2510 7060 2550
+Wire Wire Line
+	7060 2510 6710 2510
+Wire Wire Line
+	6710 2510 6710 2550
+Wire Wire Line
+	7060 2850 7060 2890
+Wire Wire Line
+	7060 2890 7410 2890
+Wire Wire Line
+	7410 2890 7410 2850
+Connection ~ 7060 2890
+Wire Wire Line
+	7060 2890 7060 2930
+Wire Wire Line
+	7060 2890 6710 2890
+Wire Wire Line
+	6710 2890 6710 2850
+$Comp
+L Custom_Library:74LVC1G17_Power U?
+U 1 1 5BB3F2C2
+P 7010 3870
+F 0 "U?" H 6910 4020 50  0000 R CNN
+F 1 "74LVC1G17" H 7330 3760 50  0000 C CNN
+F 2 "" H 7010 3870 50  0001 C CNN
+F 3 "http://www.ti.com/lit/sg/scyt129e/scyt129e.pdf" H 7010 3870 50  0001 C CNN
+	1    7010 3870
+	1    0    0    -1
+$EndComp
+Wire Wire Line
+	6460 3870 6710 3870
+$Comp
+L power:GND #PWR?
+U 1 1 5BB3FE9C
+P 7010 3970
+F 0 "#PWR?" H 7010 3720 50  0001 C CNN
+F 1 "GND" H 7010 3820 50  0000 C CNN
+F 2 "" H 7010 3970 50  0001 C CNN
+F 3 "" H 7010 3970 50  0001 C CNN
+	1    7010 3970
+	1    0    0    -1
+$EndComp
+$Comp
+L Custom_Library:+3.3V #PWR?
+U 1 1 5BB401D8
+P 7010 3770
+F 0 "#PWR?" H 7010 3620 50  0001 C CNN
+F 1 "+3.3V" H 7010 3910 50  0000 C CNN
+F 2 "" H 7010 3770 50  0000 C CNN
+F 3 "" H 7010 3770 50  0000 C CNN
+	1    7010 3770
+	1    0    0    -1
+$EndComp
+$Comp
+L Custom_Library:C_Custom C?
+U 1 1 5BB40215
+P 7390 4530
+AR Path="/5BB27BA3/5BB40215" Ref="C?"  Part="1"
+AR Path="/5BB27B84/5BB40215" Ref="C?"  Part="1"
+AR Path="/5BB31311/5BB40215" Ref="C?"  Part="1"
+F 0 "C?" H 7415 4630 50  0000 L CNN
+F 1 "0.1uF" H 7415 4430 50  0000 L CNN
+F 2 "" H 7428 4380 50  0001 C CNN
+F 3 "" H 7415 4630 50  0001 C CNN
+F 4 "0603" H 7240 4630 50  0000 R CNN "display_footprint"
+F 5 "50V" H 7240 4530 50  0000 R CNN "Voltage"
+F 6 "X7R" H 7240 4430 50  0000 R CNN "Dielectric"
+F 7 "PN" H 7815 5030 60  0001 C CNN "Digi-Key PN"
+	1    7390 4530
+	1    0    0    -1
+$EndComp
+$Comp
+L power:GND #PWR?
+U 1 1 5BB40261
+P 7390 4680
+F 0 "#PWR?" H 7390 4430 50  0001 C CNN
+F 1 "GND" H 7390 4530 50  0000 C CNN
+F 2 "" H 7390 4680 50  0001 C CNN
+F 3 "" H 7390 4680 50  0001 C CNN
+	1    7390 4680
+	1    0    0    -1
+$EndComp
+$Comp
+L Custom_Library:+3.3V #PWR?
+U 1 1 5BB402A4
+P 7390 4380
+F 0 "#PWR?" H 7390 4230 50  0001 C CNN
+F 1 "+3.3V" H 7390 4520 50  0000 C CNN
+F 2 "" H 7390 4380 50  0000 C CNN
+F 3 "" H 7390 4380 50  0000 C CNN
+	1    7390 4380
+	1    0    0    -1
+$EndComp
+$Comp
+L Custom_Library:R_Custom R?
+U 1 1 5BB405B2
+P 8110 4120
+AR Path="/5BB27BA3/5BB405B2" Ref="R?"  Part="1"
+AR Path="/5BB27BE1/5BB405B2" Ref="R?"  Part="1"
+AR Path="/5BB31311/5BB405B2" Ref="R?"  Part="1"
+F 0 "R?" H 8030 4120 50  0000 R CNN
+F 1 "10k" V 8110 4120 50  0000 C CNN
+F 2 "" H 8110 4120 50  0001 C CNN
+F 3 "" H 8110 4120 50  0001 C CNN
+F 4 "0603" H 8210 4200 50  0000 L CNN "display_footprint"
+F 5 "1%" H 8210 4120 50  0000 L CNN "Tolerance"
+F 6 "1/10W" H 8220 4040 50  0000 L CNN "Wattage"
+F 7 "PN" H 8410 4520 60  0001 C CNN "Digi-Key PN"
+	1    8110 4120
+	-1   0    0    -1
+$EndComp
+Wire Wire Line
+	8110 3970 8110 3870
+Wire Wire Line
+	8110 3870 7260 3870
+$Comp
+L power:GND #PWR?
+U 1 1 5BB40EF6
+P 8110 4270
+F 0 "#PWR?" H 8110 4020 50  0001 C CNN
+F 1 "GND" H 8110 4120 50  0000 C CNN
+F 2 "" H 8110 4270 50  0001 C CNN
+F 3 "" H 8110 4270 50  0001 C CNN
+	1    8110 4270
+	1    0    0    -1
+$EndComp
+Text GLabel 8190 3870 2    50   Output ~ 0
+Zero_Cross_Detect
+Wire Wire Line
+	8190 3870 8110 3870
+Connection ~ 8110 3870
 $EndSCHEMATC

Commit message: Added MU logo and titles to all sheets
Parts:
- removed U?: 74LVC1G17, symbol Custom_Library:74LVC1G17_Power
- added U?: 74LVC1G17, TO_SOT_Packages_SMD:SOT-353_SC-70-5, symbol Custom_Library:74LVC1G17_Power
Other:
- note added: "Input AC Zero-Cross Detection"
Changed lines of the file:
@@
 Wire Wire Line
 	6710 2890 6710 2850
-$Comp
-L Custom_Library:74LVC1G17_Power U?
-U 1 1 5BB3F2C2
-P 7010 3870
-F 0 "U?" H 6910 4020 50  0000 R CNN
-F 1 "74LVC1G17" H 7330 3760 50  0000 C CNN
-F 2 "" H 7010 3870 50  0001 C CNN
-F 3 "http://www.ti.com/lit/sg/scyt129e/scyt129e.pdf" H 7010 3870 50  0001 C CNN
-	1    7010 3870
-	1    0    0    -1
-$EndComp
 Wire Wire Line
 	6460 3870 6710 3870
@@
 	8190 3870 8110 3870
 Connection ~ 8110 3870
+$Comp
+L Custom_Library:74LVC1G17_Power U?
+U 1 1 5BBD8008
+P 7010 3870
+F 0 "U?" H 7110 4020 50  0000 L CNN
+F 1 "74LVC1G17" H 7110 3720 50  0000 L CNN
+F 2 "TO_SOT_Packages_SMD:SOT-353_SC-70-5" H 7010 3870 50  0001 C CNN
+F 3 "http://www.ti.com/lit/sg/scyt129e/scyt129e.pdf" H 7110 4020 50  0001 C CNN
+F 4 "296-11934-1-ND" H 7010 3870 50  0001 C CNN "Digi-Key PN"
+	1    7010 3870
+	1    0    0    -1
+$EndComp
+Text Notes 540  690  0    100  ~ 20
+Input AC Zero-Cross Detection
+$Comp
+L power:GNDPWR #PWR?
+U 1 1 5BBD88A3
+P 3870 4430
+F 0 "#PWR?" H 3870 4230 50  0001 C CNN
+F 1 "GNDPWR" H 3870 4300 50  0000 C CNN
+F 2 "" H 3870 4380 50  0001 C CNN
+F 3 "" H 3870 4380 50  0001 C CNN
+	1    3870 4430
+	1    0    0    -1
+$EndComp
+$Comp
+L power:PWR_FLAG #FLG?
+U 1 1 5BBD88DC
+P 3870 4430
+F 0 "#FLG?" H 3870 4505 50  0001 C CNN
+F 1 "PWR_FLAG" H 3870 4580 50  0000 C CNN
+F 2 "" H 3870 4430 50  0001 C CNN
+F 3 "~" H 3870 4430 50  0001 C CNN
+	1    3870 4430
+	1    0    0    -1
+$EndComp
+$Comp
+L Mu_Logo:LOGO #G?
+U 1 1 5BBF815F
+P 9900 1000
+F 0 "#G?" H 9900 670 60  0001 C CNN
+F 1 "LOGO" H 9900 1330 60  0001 C CNN
+F 2 "" H 9900 1000 50  0001 C CNN
+F 3 "" H 9900 1000 50  0001 C CNN
+	1    9900 1000
+	1    0    0    -1
+$EndComp
 $EndSCHEMATC

Commit message: Updated MU logo to crisper image
Changed lines of the file:
@@
 $EndComp
 $Comp
-L Mu_Logo:LOGO #G?
-U 1 1 5BBF815F
-P 9900 1000
-F 0 "#G?" H 9900 670 60  0001 C CNN
-F 1 "LOGO" H 9900 1330 60  0001 C CNN
-F 2 "" H 9900 1000 50  0001 C CNN
-F 3 "" H 9900 1000 50  0001 C CNN
-	1    9900 1000
+L Custom_Library:MU_Logo #G?
+U 1 1 5BB6AA49
+P 9900 1100
+F 0 "#G?" H 9900 614 60  0001 C CNN
+F 1 "MU_Logo" H 9900 1586 60  0001 C CNN
+F 2 "" H 9900 1100 50  0001 C CNN
+F 3 "" H 9900 1100 50  0001 C CNN
+	1    9900 1100
 	1    0    0    -1
 $EndComp

Commit message: Added series resistor in ZCD circuit
Parts:
- added C?: 0.056uF, symbol Custom_Library:C_Custom
- added R?: 1k, symbol Custom_Library:R_Custom
- R?: Tolerance 1% -> 5%; Wattage 1/10W -> 1/2W; display_footprint 0603 -> 1206
Connections:
- wire segments 42 -> 47
Other:
- moved on the sheet: D?

Commit message: Rewired a few micro symbols, add FMW notes
Parts:
- gave numbers to parts that had none: 17

Commit message: Updated most footprints
Parts:
- removed D1401, D1402, D1403, D1404, D1405: LL4448, Diode_SMD:D_MiniMELF, symbol Diode:LL4448
- added D1401, D1402, D1403, D1404, D1405: BAV21, Diodes_SMD:D_SOD-123, symbol Diode:BAV21
- C1401: footprint (none) -> Capacitors_SMD:C_0805; Digi-Key PN PN -> 399-9245-1-ND
- C1402: footprint (none) -> Capacitors_SMD:C_2220; Digi-Key PN PN -> 490-7747-1-ND
- C1403, C1405: footprint (none) -> Capacitors_SMD:C_0603; Digi-Key PN PN -> 490-8020-1-ND
- C1404: footprint (none) -> Capacitors_SMD:C_0603; Digi-Key PN PN -> 1276-1921-1-ND
- C1406: footprint (none) -> Capacitors_SMD:C_0603; Digi-Key PN PN -> 478-1215-1-ND
- R1401: footprint (none) -> Resistors_SMD:R_1206; Digi-Key PN PN -> RHM100KICT-ND
- R1402: footprint (none) -> Resistors_SMD:R_0603; Digi-Key PN PN -> MCT0603-1.00K-CFCT-ND
- R1403: footprint (none) -> Resistors_SMD:R_0603; Digi-Key PN PN -> P100KHCT-ND
- R1404: footprint (none) -> Resistors_SMD:R_0603; Digi-Key PN PN -> RHM10KADCT-ND
- U1401: Digi-Key PN (none) -> 160-1337-1-ND
Changed lines of the file:
@@
 F 0 "R1403" H 6380 4130 50  0000 R CNN
 F 1 "100k" V 6460 4130 40  0000 C CNN
-F 2 "" H 6460 4130 50  0001 C CNN
+F 2 "Resistors_SMD:R_0603" H 6460 4130 50  0001 C CNN
 F 3 "" H 6460 4130 50  0001 C CNN
 F 4 "0603" H 6560 4210 50  0000 L CNN "display_footprint"
 F 5 "1%" H 6560 4130 50  0000 L CNN "Tolerance"
 F 6 "1/10W" H 6570 4050 50  0000 L CNN "Wattage"
-F 7 "PN" H 6760 4530 60  0001 C CNN "Digi-Key PN"
+F 7 "P100KHCT-ND" H 6760 4530 60  0001 C CNN "Digi-Key PN"
 	1    6460 4130
 	-1   0    0    -1
@@
 AR Path="/5BB31311/5BB33935" Ref="U1401"  Part="1"
 F 0 "U1401" H 5760 3960 50  0000 L CNN
-F 1 "LTV-356T" H 5970 3970 50  0000 L CNN
+F 1 "LTV-356T" H 5970 3570 50  0000 C CNN
 F 2 "Package_SO:SO-4_4.4x3.6mm_P2.54mm" H 5770 3570 50  0001 L CIN
 F 3 "http://optoelectronics.liteon.com/upload/download/DS70-2001-010/S_110_LTV-356T%2020140520.pdf" H 5970 3770 50  0001 L CNN
+F 4 "160-1337-1-ND" H 5970 3770 50  0001 C CNN "Digi-Key PN"
 	1    5970 3770
 	1    0    0    -1
@@
 	1    0    0    -1
 $EndComp
-$Comp
-L Diode:LL4448 D1405
-U 1 1 5BB3428A
-P 5280 3760
-F 0 "D1405" H 5280 3860 50  0000 C CNN
-F 1 "LL4448" H 5280 3660 50  0000 C CNN
-F 2 "Diode_SMD:D_MiniMELF" H 5280 3585 50  0001 C CNN
-F 3 "http://www.vishay.com/docs/85557/ll4148.pdf" H 5280 3760 50  0001 C CNN
-	1    5280 3760
-	0    1    1    0
-$EndComp
 Wire Wire Line
 	5670 3870 5520 3870
@@
 F 0 "C1401" V 4260 3410 50  0000 R CNN
 F 1 "4.7nF" V 4260 3590 50  0000 L CNN
-F 2 "" H 4228 3360 50  0001 C CNN
+F 2 "Capacitors_SMD:C_0805" H 4228 3360 50  0001 C CNN
 F 3 "" H 4215 3610 50  0001 C CNN
 F 4 "0805" V 3848 3510 50  0000 C CNN "display_footprint"
 F 5 "200V" V 3939 3510 50  0000 C CNN "Voltage"
 F 6 "X7R" V 4030 3510 50  0000 C CNN "Dielectric"
-F 7 "PN" H 4615 4010 60  0001 C CNN "Digi-Key PN"
+F 7 "399-9245-1-ND" H 4615 4010 60  0001 C CNN "Digi-Key PN"
 	1    4190 3510
 	0    1    1    0
@@
 F 0 "R1401" H 3750 3890 50  0000 R CNN
 F 1 "100k" V 3830 3890 40  0000 C CNN
-F 2 "" H 3830 3890 50  0001 C CNN
+F 2 "Resistors_SMD:R_1206" H 3830 3890 50  0001 C CNN
 F 3 "" H 3830 3890 50  0001 C CNN
 F 4 "1206" H 3930 3970 50  0000 L CNN "display_footprint"
 F 5 "5%" H 3930 3890 50  0000 L CNN "Tolerance"
 F 6 "1/2W" H 3940 3810 50  0000 L CNN "Wattage"
-F 7 "PN" H 4130 4290 60  0001 C CNN "Digi-Key PN"
+F 7 "RHM100KICT-ND" H 4130 4290 60  0001 C CNN "Digi-Key PN"
 	1    3830 3890
 	-1   0    0    -1
@@
 Wire Wire Line
 	3830 3510 4040 3510
-$Comp
-L Diode:LL4448 D1403
-U 1 1 5BB36337
-P 2980 3740
-F 0 "D1403" H 2980 3840 50  0000 C CNN
-F 1 "LL4448" H 2980 3640 50  0000 C CNN
-F 2 "Diode_SMD:D_MiniMELF" H 2980 3565 50  0001 C CNN
-F 3 "http://www.vishay.com/docs/85557/ll4148.pdf" H 2980 3740 50  0001 C CNN
-	1    2980 3740
-	0    1    1    0
-$EndComp
-$Comp
-L Diode:LL4448 D1401
-U 1 1 5BB363D1
-P 2340 3740
-F 0 "D1401" H 2340 3840 50  0000 C CNN
-F 1 "LL4448" H 2340 3640 50  0000 C CNN
-F 2 "Diode_SMD:D_MiniMELF" H 2340 3565 50  0001 C CNN
-F 3 "http://www.vishay.com/docs/85557/ll4148.pdf" H 2340 3740 50  0001 C CNN
-	1    2340 3740
-	0    1    1    0
-$EndComp
-$Comp
-L Diode:LL4448 D1404
-U 1 1 5BB36464
-P 2980 4280
-F 0 "D1404" H 2980 4380 50  0000 C CNN
-F 1 "LL4448" H 2980 4180 50  0000 C CNN
-F 2 "Diode_SMD:D_MiniMELF" H 2980 4105 50  0001 C CNN
-F 3 "http://www.vishay.com/docs/85557/ll4148.pdf" H 2980 4280 50  0001 C CNN
-	1    2980 4280
-	0    1    1    0
-$EndComp
-$Comp
-L Diode:LL4448 D1402
-U 1 1 5BB3646B
-P 2340 4280
-F 0 "D1402" H 2340 4380 50  0000 C CNN
-F 1 "LL4448" H 2340 4180 50  0000 C CNN
-F 2 "Diode_SMD:D_MiniMELF" H 2340 4105 50  0001 C CNN
-F 3 "http://www.vishay.com/docs/85557/ll4148.pdf" H 2340 4280 50  0001 C CNN
-	1    2340 4280
-	0    1    1    0
-$EndComp
 $Comp
 L power:GNDPWR #PWR01404
@@
 F 0 "C1403" H 6735 2800 50  0000 L CNN
 F 1 "0.1uF" H 6735 2600 50  0000 L CNN
-F 2 "" H 6748 2550 50  0001 C CNN
+F 2 "Capacitors_SMD:C_0603" H 6748 2550 50  0001 C CNN
 F 3 "" H 6735 2800 50  0001 C CNN
 F 4 "0603" H 6560 2800 50  0000 R CNN "display_footprint"
 F 5 "50V" H 6560 2700 50  0000 R CNN "Voltage"
 F 6 "X7R" H 6560 2600 50  0000 R CNN "Dielectric"
-F 7 "PN" H 7135 3200 60  0001 C CNN "Digi-Key PN"
+F 7 "490-8020-1-ND" H 7135 3200 60  0001 C CNN "Digi-Key PN"
 	1    6710 2700
 	1    0    0    -1
@@
 F 0 "C1404" H 7085 2800 50  0000 L CNN
 F 1 "10nF" H 7085 2600 50  0000 L CNN
-F 2 "" H 7098 2550 50  0001 C CNN
+F 2 "Capacitors_SMD:C_0603" H 7098 2550 50  0001 C CNN
 F 3 "" H 7085 2800 50  0001 C CNN
 F 4 "0603" H 6910 2800 50  0001 R CNN "display_footprint"
 F 5 "50V" H 6910 2700 50  0001 R CNN "Voltage"
 F 6 "X7R" H 6910 2600 50  0001 R CNN "Dielectric"
-F 7 "PN" H 7485 3200 60  0001 C CNN "Digi-Key PN"
+F 7 "1276-1921-1-ND" H 7485 3200 60  0001 C CNN "Digi-Key PN"
 	1    7060 2700
 	1    0    0    -1
@@
 F 0 "C1406" H 7435 2800 50  0000 L CNN
 F 1 "1nF" H 7435 2600 50  0000 L CNN
-F 2 "" H 7448 2550 50  0001 C CNN
+F 2 "Capacitors_SMD:C_0603" H 7448 2550 50  0001 C CNN
 F 3 "" H 7435 2800 50  0001 C CNN
 F 4 "0603" H 7260 2800 50  0001 R CNN "display_footprint"
 F 5 "50V" H 7260 2700 50  0001 R CNN "Voltage"
 F 6 "X7R" H 7260 2600 50  0001 R CNN "Dielectric"
-F 7 "PN" H 7835 3200 60  0001 C CNN "Digi-Key PN"
+F 7 "478-1215-1-ND" H 7835 3200 60  0001 C CNN "Digi-Key PN"
 	1    7410 2700
 	1    0    0    -1
@@
 F 0 "C1405" H 7415 4630 50  0000 L CNN
 F 1 "0.1uF" H 7415 4430 50  0000 L CNN
-F 2 "" H 7428 4380 50  0001 C CNN
+F 2 "Capacitors_SMD:C_0603" H 7428 4380 50  0001 C CNN
 F 3 "" H 7415 4630 50  0001 C CNN
 F 4 "0603" H 7240 4630 50  0000 R CNN "display_footprint"
 F 5 "50V" H 7240 4530 50  0000 R CNN "Voltage"
 F 6 "X7R" H 7240 4430 50  0000 R CNN "Dielectric"
-F 7 "PN" H 7815 5030 60  0001 C CNN "Digi-Key PN"
+F 7 "490-8020-1-ND" H 7815 5030 60  0001 C CNN "Digi-Key PN"
 	1    7390 4530
 	1    0    0    -1
@@
 F 0 "R1404" H 8030 4120 50  0000 R CNN
 F 1 "10k" V 8110 4120 50  0000 C CNN
-F 2 "" H 8110 4120 50  0001 C CNN
+F 2 "Resistors_SMD:R_0603" H 8110 4120 50  0001 C CNN
 F 3 "" H 8110 4120 50  0001 C CNN
 F 4 "0603" H 8210 4200 50  0000 L CNN "display_footprint"
 F 5 "1%" H 8210 4120 50  0000 L CNN "Tolerance"
 F 6 "1/10W" H 8220 4040 50  0000 L CNN "Wattage"
-F 7 "PN" H 8410 4520 60  0001 C CNN "Digi-Key PN"
+F 7 "RHM10KADCT-ND" H 8410 4520 60  0001 C CNN "Digi-Key PN"
 	1    8110 4120
 	-1   0    0    -1
@@
 F 0 "C1402" V 6020 4840 50  0000 L CNN
 F 1 "0.056uF" V 6020 4660 50  0000 R CNN
-F 2 "" H 6008 4600 50  0001 C CNN
+F 2 "Capacitors_SMD:C_2220" H 6008 4600 50  0001 C CNN
 F 3 "" H 5995 4850 50  0001 C CNN
 F 4 "2220" V 5830 4750 50  0000 C CNN "display_footprint"
 F 5 "250VAC" V 5750 4750 50  0000 C CNN "Voltage"
 F 6 "X7R" V 5660 4750 50  0000 C CNN "Dielectric"
-F 7 "PN" H 6395 5250 60  0001 C CNN "Digi-Key PN"
+F 7 "490-7747-1-ND" H 6395 5250 60  0001 C CNN "Digi-Key PN"
 	1    5970 4750
 	0    1    1    0
@@
 F 0 "R1402" V 4680 3510 50  0000 C CNN
 F 1 "1k" V 4780 3510 50  0000 C CNN
-F 2 "" H 4780 3510 50  0001 C CNN
+F 2 "Resistors_SMD:R_0603" H 4780 3510 50  0001 C CNN
 F 3 "" H 4780 3510 50  0001 C CNN
 F 4 "0603" V 4880 3510 50  0000 C CNN "display_footprint"
 F 5 "1%" V 4980 3510 50  0000 C CNN "Tolerance"
 F 6 "1/10W" V 5080 3510 50  0000 C CNN "Wattage"
-F 7 "PN" H 5080 3910 60  0001 C CNN "Digi-Key PN"
+F 7 "MCT0603-1.00K-CFCT-ND" H 5080 3910 60  0001 C CNN "Digi-Key PN"
 	1    4780 3510
 	0    -1   -1   0
@@
 Wire Wire Line
 	4630 3510 4340 3510
+$Comp
+L Diode:BAV21 D1401
+U 1 1 5BB8619D
+P 2340 3740
+F 0 "D1401" H 2340 3840 50  0000 C CNN
+F 1 "BAV21" H 2340 3640 50  0000 C CNN
+F 2 "Diodes_SMD:D_SOD-123" H 2340 3565 50  0001 C CNN
+F 3 "http://www.vishay.com/docs/85543/bav17.pdf" H 2340 3740 50  0001 C CNN
+F 4 "BAV21W-FDICT-ND" H 2340 3740 50  0001 C CNN "Digi-Key PN"
+	1    2340 3740
+	0    1    1    0
+$EndComp
+$Comp
+L Diode:BAV21 D1402
+U 1 1 5BB867DD
+P 2340 4280
+F 0 "D1402" H 2340 4380 50  0000 C CNN
+F 1 "BAV21" H 2340 4180 50  0000 C CNN
+F 2 "Diodes_SMD:D_SOD-123" H 2340 4105 50  0001 C CNN
+F 3 "http://www.vishay.com/docs/85543/bav17.pdf" H 2340 4280 50  0001 C CNN
+F 4 "BAV21W-FDICT-ND" H 2340 4280 50  0001 C CNN "Digi-Key PN"
+	1    2340 4280
+	0    1    1    0
+$EndComp
+$Comp
+L Diode:BAV21 D1403
+U 1 1 5BB86831
+P 2980 3740
+F 0 "D1403" H 2980 3840 50  0000 C CNN
+F 1 "BAV21" H 2980 3640 50  0000 C CNN
+F 2 "Diodes_SMD:D_SOD-123" H 2980 3565 50  0001 C CNN
+F 3 "http://www.vishay.com/docs/85543/bav17.pdf" H 2980 3740 50  0001 C CNN
+F 4 "BAV21W-FDICT-ND" H 2980 3740 50  0001 C CNN "Digi-Key PN"
+	1    2980 3740
+	0    1    1    0
+$EndComp
+$Comp
+L Diode:BAV21 D1404
+U 1 1 5BB86887
+P 2980 4280
+F 0 "D1404" H 2980 4380 50  0000 C CNN
+F 1 "BAV21" H 2980 4180 50  0000 C CNN
+F 2 "Diodes_SMD:D_SOD-123" H 2980 4105 50  0001 C CNN
+F 3 "http://www.vishay.com/docs/85543/bav17.pdf" H 2980 4280 50  0001 C CNN
+F 4 "BAV21W-FDICT-ND" H 2980 4280 50  0001 C CNN "Digi-Key PN"
+	1    2980 4280
+	0    1    1    0
+$EndComp
+$Comp
+L Diode:BAV21 D1405
+U 1 1 5BB8692E
+P 5280 3760
+F 0 "D1405" H 5280 3860 50  0000 C CNN
+F 1 "BAV21" H 5280 3660 50  0000 C CNN
+F 2 "Diodes_SMD:D_SOD-123" H 5280 3585 50  0001 C CNN
+F 3 "http://www.vishay.com/docs/85543/bav17.pdf" H 5280 3760 50  0001 C CNN
+F 4 "BAV21W-FDICT-ND" H 5280 3760 50  0001 C CNN "Digi-Key PN"
+	1    5280 3760
+	0    1    1    0
+$EndComp
 $EndSCHEMATC
