File: hdw/AC_Power_Meter/Zero_Cross_Detect.sch (KiCad schematic (older format))
At the start: 17 parts, among them U1401 LTV-356T, U1402 74LVC1G17

Commit message: Arranged a few pages of components
Parts:
- U1401: footprint Package_SO:SO-4_4.4x3.6mm_P2.54mm -> Housings_SOIC:SO-4_4.4x3.6mm_Pitch2.54mm
Changed lines of the file:
@@
 F 0 "U1401" H 5760 3960 50  0000 L CNN
 F 1 "LTV-356T" H 5970 3570 50  0000 C CNN
-F 2 "Package_SO:SO-4_4.4x3.6mm_P2.54mm" H 5770 3570 50  0001 L CIN
+F 2 "Housings_SOIC:SO-4_4.4x3.6mm_Pitch2.54mm" H 5770 3570 50  0001 L CIN
 F 3 "http://optoelectronics.liteon.com/upload/download/DS70-2001-010/S_110_LTV-356T%2020140520.pdf" H 5970 3770 50  0001 L CNN
 F 4 "160-1337-1-ND" H 5970 3770 50  0001 C CNN "Digi-Key PN"

Commit message: Serious BOM scrubbing to drive price down
Parts:
- removed C1402: 0.056uF, Capacitors_SMD:C_2220, symbol Custom_Library:C_Custom
Connections:
- wire segments 47 -> 43
Changed lines of the file:
@@
 $Descr A 11000 8500
 encoding utf-8
-Sheet 14 18
+Sheet 16 17
 Title ""
 Date ""
@@
 AR Path="/5BB27BE1/5BB338DA" Ref="R?"  Part="1"
 AR Path="/5BB31311/5BB338DA" Ref="R1403"  Part="1"
+AR Path="/5BBE5EA4/5BB338DA" Ref="R1403"  Part="1"
 F 0 "R1403" H 6380 4130 50  0000 R CNN
 F 1 "100k" V 6460 4130 40  0000 C CNN
@@
 AR Path="/5BB31314/5BB3392D" Ref="#PWR?"  Part="1"
 AR Path="/5BB31311/5BB3392D" Ref="#PWR01409"  Part="1"
+AR Path="/5BBE5EA4/5BB3392D" Ref="#PWR01409"  Part="1"
 F 0 "#PWR01409" H 6460 3440 50  0001 C CNN
 F 1 "+3.3V" H 6460 3730 50  0000 C CNN
@@
 AR Path="/5BB31314/5BB33935" Ref="U?"  Part="1"
 AR Path="/5BB31311/5BB33935" Ref="U1401"  Part="1"
+AR Path="/5BBE5EA4/5BB33935" Ref="U1401"  Part="1"
 F 0 "U1401" H 5760 3960 50  0000 L CNN
 F 1 "LTV-356T" H 5970 3570 50  0000 C CNN
@@
 AR Path="/5BB27BE1/5BB3583A" Ref="R?"  Part="1"
 AR Path="/5BB31311/5BB3583A" Ref="R1401"  Part="1"
+AR Path="/5BBE5EA4/5BB3583A" Ref="R1401"  Part="1"
 F 0 "R1401" H 3750 3890 50  0000 R CNN
 F 1 "100k" V 3830 3890 40  0000 C CNN
@@
 AR Path="/5BB27B84/5BB38E0F" Ref="C?"  Part="1"
 AR Path="/5BB31311/5BB38E0F" Ref="C1403"  Part="1"
+AR Path="/5BBE5EA4/5BB38E0F" Ref="C1403"  Part="1"
 F 0 "C1403" H 6735 2800 50  0000 L CNN
 F 1 "0.1uF" H 6735 2600 50  0000 L CNN
@@
 AR Path="/5BB27B84/5BB38E1A" Ref="C?"  Part="1"
 AR Path="/5BB31311/5BB38E1A" Ref="C1404"  Part="1"
+AR Path="/5BBE5EA4/5BB38E1A" Ref="C1404"  Part="1"
 F 0 "C1404" H 7085 2800 50  0000 L CNN
 F 1 "10nF" H 7085 2600 50  0000 L CNN
@@
 AR Path="/5BB27B84/5BB38E25" Ref="C?"  Part="1"
 AR Path="/5BB31311/5BB38E25" Ref="C1406"  Part="1"
+AR Path="/5BBE5EA4/5BB38E25" Ref="C1406"  Part="1"
 F 0 "C1406" H 7435 2800 50  0000 L CNN
 F 1 "1nF" H 7435 2600 50  0000 L CNN
@@
 AR Path="/5BB27B84/5BB40215" Ref="C?"  Part="1"
 AR Path="/5BB31311/5BB40215" Ref="C1405"  Part="1"
+AR Path="/5BBE5EA4/5BB40215" Ref="C1405"  Part="1"
 F 0 "C1405" H 7415 4630 50  0000 L CNN
 F 1 "0.1uF" H 7415 4430 50  0000 L CNN
@@
 AR Path="/5BB27BE1/5BB405B2" Ref="R?"  Part="1"
 AR Path="/5BB31311/5BB405B2" Ref="R1404"  Part="1"
+AR Path="/5BBE5EA4/5BB405B2" Ref="R1404"  Part="1"
 F 0 "R1404" H 8030 4120 50  0000 R CNN
 F 1 "10k" V 8110 4120 50  0000 C CNN
@@
 	1    0    0    -1
 $EndComp
-$Comp
-L Custom_Library:C_Custom C1402
-U 1 1 5BB6C4C6
-P 5970 4750
-F 0 "C1402" V 6020 4840 50  0000 L CNN
-F 1 "0.056uF" V 6020 4660 50  0000 R CNN
-F 2 "Capacitors_SMD:C_2220" H 6008 4600 50  0001 C CNN
-F 3 "" H 5995 4850 50  0001 C CNN
-F 4 "2220" V 5830 4750 50  0000 C CNN "display_footprint"
-F 5 "250VAC" V 5750 4750 50  0000 C CNN "Voltage"
-F 6 "X7R" V 5660 4750 50  0000 C CNN "Dielectric"
-F 7 "490-7747-1-ND" H 6395 5250 60  0001 C CNN "Digi-Key PN"
-	1    5970 4750
-	0    1    1    0
-$EndComp
-Wire Wire Line
-	6490 4830 6490 4750
-Wire Wire Line
-	6490 4750 6120 4750
-Wire Wire Line
-	5450 4830 5450 4750
-Wire Wire Line
-	5450 4750 5820 4750
-$Comp
-L power:GND #PWR01411
-U 1 1 5BB6D592
-P 6490 4830
-F 0 "#PWR01411" H 6490 4580 50  0001 C CNN
-F 1 "GND" H 6490 4680 50  0000 C CNN
-F 2 "" H 6490 4830 50  0001 C CNN
-F 3 "" H 6490 4830 50  0001 C CNN
-	1    6490 4830
-	1    0    0    -1
-$EndComp
-$Comp
-L power:GNDPWR #PWR01408
-U 1 1 5BB6D5FD
-P 5450 4830
-F 0 "#PWR01408" H 5450 4630 50  0001 C CNN
-F 1 "GNDPWR" H 5450 4700 50  0000 C CNN
-F 2 "" H 5450 4780 50  0001 C CNN
-F 3 "" H 5450 4780 50  0001 C CNN
-	1    5450 4830
-	1    0    0    -1
-$EndComp
