File: hdw/AC_Power_Meter/POS3P3_Power_Supply.sch (KiCad schematic (older format))
At the start: 0 parts

Commit message: Added +3.3V power supply, +12V window comparator, a few design files
Parts:
- added C?: 0.47uF, symbol Custom_Library:C_Custom
- added C? (x3): 0.1uF, symbol Custom_Library:C_Custom
- added C? (x2): 4.7uF, symbol Custom_Library:C_Custom
- added C?: 15pF, symbol Custom_Library:C_Custom
- added C? (x2): 10uF, symbol Custom_Library:C_Custom
- added L?: 3.3u, symbol Custom_Library:L_Custom
- added R?: 80.6k, symbol Custom_Library:R_Custom
- added R? (x3): 10k, symbol Custom_Library:R_Custom
- added R?: 43.2k, symbol Custom_Library:R_Custom
- added R?: 1M, symbol Custom_Library:R_Custom
- added R?: 576k, symbol Custom_Library:R_Custom
- added TP?: TP, symbol Custom_Library:TP
- added U?: LT3973-DD, Housings_DFN_QFN:DFN-10-1EP_3x3mm_Pitch0.5mm, symbol Custom_Library:LT3973-DD
- added U?: 74LVC1G17, TO_SOT_Packages_SMD:SOT-353_SC-70-5, symbol Custom_Library:74LVC1G17_Power
Connections:
- net labels added: +12V, +3.3V, GND, POS3P3_PGOOD
- wire segments 0 -> 53
Other:
- note added: "+3.3V, 750mA, 2MHz Buck Converter"

Commit message: Added MU logo and titles to all sheets
Changed lines of the file:
@@
 	1410 4450 1490 4450
 Connection ~ 1490 4450
-Text Notes 3860 900  0    100  ~ 20
+Text Notes 540  690  0    100  ~ 20
 +3.3V, 750mA, 2MHz Buck Converter
+$Comp
+L Mu_Logo:LOGO #G?
+U 1 1 5BBF3205
+P 9900 1000
+F 0 "#G?" H 9900 670 60  0001 C CNN
+F 1 "LOGO" H 9900 1330 60  0001 C CNN
+F 2 "" H 9900 1000 50  0001 C CNN
+F 3 "" H 9900 1000 50  0001 C CNN
+	1    9900 1000
+	1    0    0    -1
+$EndComp
 $EndSCHEMATC

Commit message: Updated MU logo to crisper image
Changed lines of the file:
@@
 +3.3V, 750mA, 2MHz Buck Converter
 $Comp
-L Mu_Logo:LOGO #G?
-U 1 1 5BBF3205
-P 9900 1000
-F 0 "#G?" H 9900 670 60  0001 C CNN
-F 1 "LOGO" H 9900 1330 60  0001 C CNN
-F 2 "" H 9900 1000 50  0001 C CNN
-F 3 "" H 9900 1000 50  0001 C CNN
-	1    9900 1000
+L Custom_Library:MU_Logo #G?
+U 1 1 5BB6890F
+P 9900 1100
+F 0 "#G?" H 9900 614 60  0001 C CNN
+F 1 "MU_Logo" H 9900 1586 60  0001 C CNN
+F 2 "" H 9900 1100 50  0001 C CNN
+F 3 "" H 9900 1100 50  0001 C CNN
+	1    9900 1100
 	1    0    0    -1
 $EndComp

Commit message: Added pushbuttons sheet, prelim wiring on micro
Parts:
- added R? (x2): 10k, symbol Custom_Library:R_Custom
Connections:
- net labels added: POS3P3_ADC
- wire segments 53 -> 56
Changed lines of the file:
@@
 $Descr A 11000 8500
 encoding utf-8
-Sheet 6 16
+Sheet 6 17
 Title ""
 Date "2018-10-01"
@@
 	1    0    0    -1
 $EndComp
+$Comp
+L Custom_Library:R_Custom R?
+U 1 1 5BC21861
+P 2740 6910
+AR Path="/5BB27BA3/5BC21861" Ref="R?"  Part="1"
+AR Path="/5BB27B51/5BC21861" Ref="R?"  Part="1"
+AR Path="/5BB7FA89/5BC21861" Ref="R?"  Part="1"
+AR Path="/5BB27B73/5BC21861" Ref="R?"  Part="1"
+F 0 "R?" H 2660 6910 50  0000 R CNN
+F 1 "10k" V 2740 6910 50  0000 C CNN
+F 2 "" H 2740 6910 50  0001 C CNN
+F 3 "" H 2740 6910 50  0001 C CNN
+F 4 "0603" H 2840 6990 50  0000 L CNN "display_footprint"
+F 5 "1%" H 2840 6910 50  0000 L CNN "Tolerance"
+F 6 "1/10W" H 2850 6830 50  0000 L CNN "Wattage"
+F 7 "PN" H 3040 7310 60  0001 C CNN "Digi-Key PN"
+	1    2740 6910
+	1    0    0    -1
+$EndComp
+$Comp
+L Custom_Library:R_Custom R?
+U 1 1 5BC21957
+P 2740 6390
+AR Path="/5BB27BA3/5BC21957" Ref="R?"  Part="1"
+AR Path="/5BB27B51/5BC21957" Ref="R?"  Part="1"
+AR Path="/5BB7FA89/5BC21957" Ref="R?"  Part="1"
+AR Path="/5BB27B73/5BC21957" Ref="R?"  Part="1"
+F 0 "R?" H 2660 6390 50  0000 R CNN
+F 1 "10k" V 2740 6390 50  0000 C CNN
+F 2 "" H 2740 6390 50  0001 C CNN
+F 3 "" H 2740 6390 50  0001 C CNN
+F 4 "0603" H 2840 6470 50  0000 L CNN "display_footprint"
+F 5 "1%" H 2840 6390 50  0000 L CNN "Tolerance"
+F 6 "1/10W" H 2850 6310 50  0000 L CNN "Wattage"
+F 7 "PN" H 3040 6790 60  0001 C CNN "Digi-Key PN"
+	1    2740 6390
+	1    0    0    -1
+$EndComp
+$Comp
+L Custom_Library:+3.3V #PWR?
+U 1 1 5BC219D1
+P 2740 6240
+F 0 "#PWR?" H 2740 6090 50  0001 C CNN
+F 1 "+3.3V" H 2740 6380 50  0000 C CNN
+F 2 "" H 2740 6240 50  0000 C CNN
+F 3 "" H 2740 6240 50  0000 C CNN
+	1    2740 6240
+	1    0    0    -1
+$EndComp
+$Comp
+L power:GND #PWR?
+U 1 1 5BC21AA2
+P 2740 7060
+F 0 "#PWR?" H 2740 6810 50  0001 C CNN
+F 1 "GND" H 2740 6910 50  0000 C CNN
+F 2 "" H 2740 7060 50  0001 C CNN
+F 3 "" H 2740 7060 50  0001 C CNN
+	1    2740 7060
+	1    0    0    -1
+$EndComp
+Wire Wire Line
+	2740 6540 2740 6650
+Text GLabel 2890 6650 2    50   Output ~ 0
+POS3P3_ADC
+Wire Wire Line
+	2890 6650 2740 6650
+Connection ~ 2740 6650
+Wire Wire Line
+	2740 6650 2740 6760
 $EndSCHEMATC

Commit message: Rewired a few micro symbols, add FMW notes
Parts:
- gave numbers to parts that had none: 22

Commit message: Updated most footprints
Parts:
- C601, C603: footprint (none) -> Capacitors_SMD:C_0805; Digi-Key PN PN -> 587-2990-1-ND
- C602, C604, C607: footprint (none) -> Capacitors_SMD:C_0603; Digi-Key PN PN -> 490-8020-1-ND
- C605: footprint (none) -> Capacitors_SMD:C_0603; Digi-Key PN PN -> 490-3291-1-ND
- C606: footprint (none) -> Capacitors_SMD:C_0603; Digi-Key PN PN -> 478-10290-1-ND
- C608, C609: footprint (none) -> Capacitors_SMD:C_0805; Digi-Key PN PN -> 490-10517-1-ND
- L601: footprint (none) -> Inductors_SMD:L_Vishay_IHLP-1212
- R601, R602, R603, R604, R606: footprint (none) -> Resistors_SMD:R_0603; Digi-Key PN PN -> RHM10KADCT-ND
- R605: footprint (none) -> Resistors_SMD:R_0603; Digi-Key PN PN -> P80.6KHCT-ND
- R607: footprint (none) -> Resistors_SMD:R_0603; Digi-Key PN PN -> P43.2KHCT-ND
- R608: footprint (none) -> Resistors_SMD:R_0603; Digi-Key PN PN -> A130109CT-ND
- R609: footprint (none) -> Resistors_SMD:R_0603; Digi-Key PN PN -> 311-576KHRCT-ND
- TP601: footprint (none) -> Measurement_Points:Measurement_Point_Round-SMD-Pad_Small
Changed lines of the file:
@@
 F 0 "R605" H 3540 3280 50  0000 R CNN
 F 1 "80.6k" V 3620 3280 40  0000 C CNN
-F 2 "" H 3620 3280 50  0001 C CNN
+F 2 "Resistors_SMD:R_0603" H 3620 3280 50  0001 C CNN
 F 3 "" H 3620 3280 50  0001 C CNN
 F 4 "0603" H 3720 3360 50  0000 L CNN "display_footprint"
 F 5 "1%" H 3720 3280 50  0000 L CNN "Tolerance"
 F 6 "1/10W" H 3730 3200 50  0000 L CNN "Wattage"
-F 7 "PN" H 3920 3680 60  0001 C CNN "Digi-Key PN"
+F 7 "P80.6KHCT-ND" H 3920 3680 60  0001 C CNN "Digi-Key PN"
 	1    3620 3280
 	1    0    0    -1
@@
 F 0 "R606" H 3540 3820 50  0000 R CNN
 F 1 "10k" V 3620 3820 50  0000 C CNN
-F 2 "" H 3620 3820 50  0001 C CNN
+F 2 "Resistors_SMD:R_0603" H 3620 3820 50  0001 C CNN
 F 3 "" H 3620 3820 50  0001 C CNN
 F 4 "0603" H 3720 3900 50  0000 L CNN "display_footprint"
 F 5 "1%" H 3720 3820 50  0000 L CNN "Tolerance"
 F 6 "1/10W" H 3730 3740 50  0000 L CNN "Wattage"
-F 7 "PN" H 3920 4220 60  0001 C CNN "Digi-Key PN"
+F 7 "RHM10KADCT-ND" H 3920 4220 60  0001 C CNN "Digi-Key PN"
 	1    3620 3820
 	1    0    0    -1
@@
 F 0 "C605" H 5795 3380 50  0000 L CNN
 F 1 "0.47uF" H 5795 3180 50  0000 L CNN
-F 2 "" H 5808 3130 50  0001 C CNN
+F 2 "Capacitors_SMD:C_0603" H 5808 3130 50  0001 C CNN
 F 3 "" H 5795 3380 50  0001 C CNN
 F 4 "0603" H 5620 3380 50  0000 R CNN "display_footprint"
 F 5 "25V" H 5620 3280 50  0000 R CNN "Voltage"
 F 6 "X7R" H 5620 3180 50  0000 R CNN "Dielectric"
-F 7 "PN" H 6195 3780 60  0001 C CNN "Digi-Key PN"
+F 7 "490-3291-1-ND" H 6195 3780 60  0001 C CNN "Digi-Key PN"
 	1    5770 3280
 	1    0    0    -1
@@
 F 0 "L601" V 6430 3550 50  0000 C CNN
 F 1 "3.3u" V 6555 3550 50  0000 C CNN
-F 2 "" H 6480 3550 50  0001 C CNN
+F 2 "Inductors_SMD:L_Vishay_IHLP-1212" H 6480 3550 50  0001 C CNN
 F 3 "" H 6480 3550 50  0001 C CNN
 F 4 "541-2567-1-ND" H 6480 3550 50  0001 C CNN "Digi-Key PN"
@@
 F 0 "C604" H 2995 3380 50  0000 L CNN
 F 1 "0.1uF" H 2995 3180 50  0000 L CNN
-F 2 "" H 3008 3130 50  0001 C CNN
+F 2 "Capacitors_SMD:C_0603" H 3008 3130 50  0001 C CNN
 F 3 "" H 2995 3380 50  0001 C CNN
 F 4 "0603" H 2820 3380 50  0000 R CNN "display_footprint"
 F 5 "50V" H 2820 3280 50  0000 R CNN "Voltage"
 F 6 "X7R" H 2820 3180 50  0000 R CNN "Dielectric"
-F 7 "PN" H 3395 3780 60  0001 C CNN "Digi-Key PN"
+F 7 "490-8020-1-ND" H 3395 3780 60  0001 C CNN "Digi-Key PN"
 	1    2970 3280
 	1    0    0    -1
@@
 F 0 "C603" H 2295 3380 50  0000 L CNN
 F 1 "4.7uF" H 2295 3180 50  0000 L CNN
-F 2 "" H 2308 3130 50  0001 C CNN
+F 2 "Capacitors_SMD:C_0805" H 2308 3130 50  0001 C CNN
 F 3 "" H 2295 3380 50  0001 C CNN
 F 4 "0805" H 2120 3380 50  0000 R CNN "display_footprint"
 F 5 "25V" H 2120 3280 50  0000 R CNN "Voltage"
 F 6 "X7R" H 2120 3180 50  0000 R CNN "Dielectric"
-F 7 "PN" H 2695 3780 60  0001 C CNN "Digi-Key PN"
+F 7 "587-2990-1-ND" H 2695 3780 60  0001 C CNN "Digi-Key PN"
 	1    2270 3280
 	1    0    0    -1
@@
 F 0 "R604" H 2870 4220 50  0000 R CNN
 F 1 "10k" V 2950 4220 50  0000 C CNN
-F 2 "" H 2950 4220 50  0001 C CNN
+F 2 "Resistors_SMD:R_0603" H 2950 4220 50  0001 C CNN
 F 3 "" H 2950 4220 50  0001 C CNN
 F 4 "0603" H 3050 4300 50  0000 L CNN "display_footprint"
 F 5 "1%" H 3050 4220 50  0000 L CNN "Tolerance"
 F 6 "1/10W" H 3060 4140 50  0000 L CNN "Wattage"
-F 7 "PN" H 3250 4620 60  0001 C CNN "Digi-Key PN"
+F 7 "RHM10KADCT-ND" H 3250 4620 60  0001 C CNN "Digi-Key PN"
 	1    2950 4220
 	1    0    0    -1
@@
 F 0 "R607" H 3540 5080 50  0000 R CNN
 F 1 "43.2k" V 3620 5080 40  0000 C CNN
-F 2 "" H 3620 5080 50  0001 C CNN
+F 2 "Resistors_SMD:R_0603" H 3620 5080 50  0001 C CNN
 F 3 "" H 3620 5080 50  0001 C CNN
 F 4 "0603" H 3720 5160 50  0000 L CNN "display_footprint"
 F 5 "1%" H 3720 5080 50  0000 L CNN "Tolerance"
 F 6 "1/10W" H 3730 5000 50  0000 L CNN "Wattage"
-F 7 "PN" H 3920 5480 60  0001 C CNN "Digi-Key PN"
+F 7 "P43.2KHCT-ND" H 3920 5480 60  0001 C CNN "Digi-Key PN"
 	1    3620 5080
 	1    0    0    -1
@@
 F 0 "C606" H 6885 4390 50  0000 L CNN
 F 1 "15pF" H 6885 4190 50  0000 L CNN
-F 2 "" H 6898 4140 50  0001 C CNN
+F 2 "Capacitors_SMD:C_0603" H 6898 4140 50  0001 C CNN
 F 3 "" H 6885 4390 50  0001 C CNN
 F 4 "0603" H 6710 4390 50  0000 R CNN "display_footprint"
 F 5 "50V" H 6710 4290 50  0000 R CNN "Voltage"
 F 6 "C0G/NP0" H 6710 4190 50  0000 R CNN "Dielectric"
-F 7 "PN" H 7285 4790 60  0001 C CNN "Digi-Key PN"
+F 7 "478-10290-1-ND" H 7285 4790 60  0001 C CNN "Digi-Key PN"
 	1    6860 4290
 	1    0    0    -1
@@
 F 0 "R608" H 7420 4290 50  0000 R CNN
 F 1 "1M" V 7500 4290 50  0000 C CNN
-F 2 "" H 7500 4290 50  0001 C CNN
+F 2 "Resistors_SMD:R_0603" H 7500 4290 50  0001 C CNN
 F 3 "" H 7500 4290 50  0001 C CNN
 F 4 "0603" H 7600 4370 50  0000 L CNN "display_footprint"
 F 5 "1%" H 7600 4290 50  0000 L CNN "Tolerance"
 F 6 "1/10W" H 7610 4210 50  0000 L CNN "Wattage"
-F 7 "PN" H 7800 4690 60  0001 C CNN "Digi-Key PN"
+F 7 "A130109CT-ND" H 7800 4690 60  0001 C CNN "Digi-Key PN"
 	1    7500 4290
 	1    0    0    -1
@@
 F 0 "R609" H 7420 4910 50  0000 R CNN
 F 1 "576k" V 7500 4910 40  0000 C CNN
-F 2 "" H 7500 4910 50  0001 C CNN
+F 2 "Resistors_SMD:R_0603" H 7500 4910 50  0001 C CNN
 F 3 "" H 7500 4910 50  0001 C CNN
 F 4 "0603" H 7600 4990 50  0000 L CNN "display_footprint"
 F 5 "1%" H 7600 4910 50  0000 L CNN "Tolerance"
 F 6 "1/10W" H 7610 4830 50  0000 L CNN "Wattage"
-F 7 "PN" H 7800 5310 60  0001 C CNN "Digi-Key PN"
+F 7 "311-576KHRCT-ND" H 7800 5310 60  0001 C CNN "Digi-Key PN"
 	1    7500 4910
 	1    0    0    -1
@@
 F 0 "C607" H 8135 3880 50  0000 L CNN
 F 1 "0.1uF" H 8135 3680 50  0000 L CNN
-F 2 "" H 8148 3630 50  0001 C CNN
+F 2 "Capacitors_SMD:C_0603" H 8148 3630 50  0001 C CNN
 F 3 "" H 8135 3880 50  0001 C CNN
 F 4 "0603" H 7960 3880 50  0000 R CNN "display_footprint"
 F 5 "50V" H 7960 3780 50  0000 R CNN "Voltage"
 F 6 "X7R" H 7960 3680 50  0000 R CNN "Dielectric"
-F 7 "PN" H 8535 4280 60  0001 C CNN "Digi-Key PN"
+F 7 "490-8020-1-ND" H 8535 4280 60  0001 C CNN "Digi-Key PN"
 	1    8110 3780
 	1    0    0    -1
@@
 F 0 "TP601" H 8110 3620 50  0000 C CNN
 F 1 "TP" H 8110 3620 50  0001 C CNN
-F 2 "" H 8110 3470 60  0000 C CNN
+F 2 "Measurement_Points:Measurement_Point_Round-SMD-Pad_Small" H 8110 3470 60  0001 C CNN
 F 3 "" H 8110 3470 60  0000 C CNN
 	1    8110 3470
@@
 F 0 "C608" H 8835 3880 50  0000 L CNN
 F 1 "10uF" H 8835 3680 50  0000 L CNN
-F 2 "" H 8848 3630 50  0001 C CNN
+F 2 "Capacitors_SMD:C_0805" H 8848 3630 50  0001 C CNN
 F 3 "" H 8835 3880 50  0001 C CNN
 F 4 "0805" H 8660 3880 50  0000 R CNN "display_footprint"
 F 5 "6.3V" H 8660 3780 50  0000 R CNN "Voltage"
 F 6 "X7R" H 8660 3680 50  0000 R CNN "Dielectric"
-F 7 "PN" H 9235 4280 60  0001 C CNN "Digi-Key PN"
+F 7 "490-10517-1-ND" H 9235 4280 60  0001 C CNN "Digi-Key PN"
 	1    8810 3780
 	1    0    0    -1
@@
 F 0 "C609" H 9535 3880 50  0000 L CNN
 F 1 "10uF" H 9535 3680 50  0000 L CNN
-F 2 "" H 9548 3630 50  0001 C CNN
+F 2 "Capacitors_SMD:C_0805" H 9548 3630 50  0001 C CNN
 F 3 "" H 9535 3880 50  0001 C CNN
 F 4 "0805" H 9360 3880 50  0000 R CNN "display_footprint"
 F 5 "6.3V" H 9360 3780 50  0000 R CNN "Voltage"
 F 6 "X7R" H 9360 3680 50  0000 R CNN "Dielectric"
-F 7 "PN" H 9935 4280 60  0001 C CNN "Digi-Key PN"
+F 7 "490-10517-1-ND" H 9935 4280 60  0001 C CNN "Digi-Key PN"
 	1    9510 3780
 	1    0    0    -1
@@
 F 0 "C601" H 1595 3380 50  0000 L CNN
 F 1 "4.7uF" H 1595 3180 50  0000 L CNN
-F 2 "" H 1608 3130 50  0001 C CNN
+F 2 "Capacitors_SMD:C_0805" H 1608 3130 50  0001 C CNN
 F 3 "" H 1595 3380 50  0001 C CNN
 F 4 "0805" H 1420 3380 50  0000 R CNN "display_footprint"
 F 5 "25V" H 1420 3280 50  0000 R CNN "Voltage"
 F 6 "X7R" H 1420 3180 50  0000 R CNN "Dielectric"
-F 7 "PN" H 1995 3780 60  0001 C CNN "Digi-Key PN"
+F 7 "587-2990-1-ND" H 1995 3780 60  0001 C CNN "Digi-Key PN"
 	1    1570 3280
 	1    0    0    -1
@@
 F 0 "C602" H 2215 5250 50  0000 L CNN
 F 1 "0.1uF" H 2215 5050 50  0000 L CNN
-F 2 "" H 2228 5000 50  0001 C CNN
+F 2 "Capacitors_SMD:C_0603" H 2228 5000 50  0001 C CNN
 F 3 "" H 2215 5250 50  0001 C CNN
 F 4 "0603" H 2040 5250 50  0000 R CNN "display_footprint"
 F 5 "50V" H 2040 5150 50  0000 R CNN "Voltage"
 F 6 "X7R" H 2040 5050 50  0000 R CNN "Dielectric"
-F 7 "PN" H 2615 5650 60  0001 C CNN "Digi-Key PN"
+F 7 "490-8020-1-ND" H 2615 5650 60  0001 C CNN "Digi-Key PN"
 	1    2190 5150
 	1    0    0    -1
@@
 F 0 "R601" H 1410 4830 50  0000 R CNN
 F 1 "10k" V 1490 4830 50  0000 C CNN
-F 2 "" H 1490 4830 50  0001 C CNN
+F 2 "Resistors_SMD:R_0603" H 1490 4830 50  0001 C CNN
 F 3 "" H 1490 4830 50  0001 C CNN
 F 4 "0603" H 1590 4910 50  0000 L CNN "display_footprint"
 F 5 "1%" H 1590 4830 50  0000 L CNN "Tolerance"
 F 6 "1/10W" H 1600 4750 50  0000 L CNN "Wattage"
-F 7 "PN" H 1790 5230 60  0001 C CNN "Digi-Key PN"
+F 7 "RHM10KADCT-ND" H 1790 5230 60  0001 C CNN "Digi-Key PN"
 	1    1490 4830
 	1    0    0    -1
@@
 F 0 "R603" H 2660 6910 50  0000 R CNN
 F 1 "10k" V 2740 6910 50  0000 C CNN
-F 2 "" H 2740 6910 50  0001 C CNN
+F 2 "Resistors_SMD:R_0603" H 2740 6910 50  0001 C CNN
 F 3 "" H 2740 6910 50  0001 C CNN
 F 4 "0603" H 2840 6990 50  0000 L CNN "display_footprint"
 F 5 "1%" H 2840 6910 50  0000 L CNN "Tolerance"
 F 6 "1/10W" H 2850 6830 50  0000 L CNN "Wattage"
-F 7 "PN" H 3040 7310 60  0001 C CNN "Digi-Key PN"
+F 7 "RHM10KADCT-ND" H 3040 7310 60  0001 C CNN "Digi-Key PN"
 	1    2740 6910
 	1    0    0    -1
@@
 F 0 "R602" H 2660 6390 50  0000 R CNN
 F 1 "10k" V 2740 6390 50  0000 C CNN
-F 2 "" H 2740 6390 50  0001 C CNN
+F 2 "Resistors_SMD:R_0603" H 2740 6390 50  0001 C CNN
 F 3 "" H 2740 6390 50  0001 C CNN
 F 4 "0603" H 2840 6470 50  0000 L CNN "display_footprint"
 F 5 "1%" H 2840 6390 50  0000 L CNN "Tolerance"
 F 6 "1/10W" H 2850 6310 50  0000 L CNN "Wattage"
-F 7 "PN" H 3040 6790 60  0001 C CNN "Digi-Key PN"
+F 7 "RHM10KADCT-ND" H 3040 6790 60  0001 C CNN "Digi-Key PN"
 	1    2740 6390
 	1    0    0    -1

Commit message: Serious BOM scrubbing to drive price down
Parts:
- removed C602: 0.1uF, Capacitors_SMD:C_0603, symbol Custom_Library:C_Custom
- removed R601, R604: 10k, Resistors_SMD:R_0603, symbol Custom_Library:R_Custom
- removed U601: 74LVC1G17, TO_SOT_Packages_SMD:SOT-353_SC-70-5, symbol Custom_Library:74LVC1G17_Power
- C601, C603: Digi-Key PN 587-2990-1-ND -> 478-10056-1-ND
Connections:
- net labels removed: POS3P3_PGOOD
- wire segments 56 -> 50
- no-connect marks 0 -> 1
Changed lines of the file:
@@
 $Descr A 11000 8500
 encoding utf-8
-Sheet 6 18
+Sheet 6 17
 Title ""
 Date "2018-10-01"
@@
 F 5 "25V" H 2120 3280 50  0000 R CNN "Voltage"
 F 6 "X7R" H 2120 3180 50  0000 R CNN "Dielectric"
-F 7 "587-2990-1-ND" H 2695 3780 60  0001 C CNN "Digi-Key PN"
+F 7 "478-10056-1-ND" H 2695 3780 60  0001 C CNN "Digi-Key PN"
 	1    2270 3280
 	1    0    0    -1
@@
 Wire Wire Line
 	2970 3050 3620 3050
-$Comp
-L Custom_Library:R_Custom R?
-U 1 1 5BBA41B9
-P 2950 4220
-AR Path="/5BB27BA3/5BBA41B9" Ref="R?"  Part="1"
-AR Path="/5BB27B51/5BBA41B9" Ref="R?"  Part="1"
-AR Path="/5BB7FA89/5BBA41B9" Ref="R?"  Part="1"
-AR Path="/5BB27B73/5BBA41B9" Ref="R604"  Part="1"
-F 0 "R604" H 2870 4220 50  0000 R CNN
-F 1 "10k" V 2950 4220 50  0000 C CNN
-F 2 "Resistors_SMD:R_0603" H 2950 4220 50  0001 C CNN
-F 3 "" H 2950 4220 50  0001 C CNN
-F 4 "0603" H 3050 4300 50  0000 L CNN "display_footprint"
-F 5 "1%" H 3050 4220 50  0000 L CNN "Tolerance"
-F 6 "1/10W" H 3060 4140 50  0000 L CNN "Wattage"
-F 7 "RHM10KADCT-ND" H 3250 4620 60  0001 C CNN "Digi-Key PN"
-	1    2950 4220
-	1    0    0    -1
-$EndComp
-$Comp
-L Custom_Library:+3.3V #PWR0611
-U 1 1 5BBA4231
-P 2950 4070
-F 0 "#PWR0611" H 2950 3920 50  0001 C CNN
-F 1 "+3.3V" H 2950 4210 50  0000 C CNN
-F 2 "" H 2950 4070 50  0000 C CNN
-F 3 "" H 2950 4070 50  0000 C CNN
-	1    2950 4070
-	1    0    0    -1
-$EndComp
-Wire Wire Line
-	3960 4450 2950 4450
-Wire Wire Line
-	2950 4450 2950 4370
-Connection ~ 2950 4450
 $Comp
 L Custom_Library:R_Custom R?
@@
 F 5 "25V" H 1420 3280 50  0000 R CNN "Voltage"
 F 6 "X7R" H 1420 3180 50  0000 R CNN "Dielectric"
-F 7 "587-2990-1-ND" H 1995 3780 60  0001 C CNN "Digi-Key PN"
+F 7 "478-10056-1-ND" H 1995 3780 60  0001 C CNN "Digi-Key PN"
 	1    1570 3280
 	1    0    0    -1
 $EndComp
-Text GLabel 1410 4450 0    50   Output ~ 0
-POS3P3_PGOOD
-$Comp
-L Custom_Library:74LVC1G17_Power U601
-U 1 1 5BBB8208
-P 2390 4450
-F 0 "U601" H 2490 4600 50  0000 L CNN
-F 1 "74LVC1G17" H 2490 4300 50  0000 L CNN
-F 2 "TO_SOT_Packages_SMD:SOT-353_SC-70-5" H 2390 4450 50  0001 C CNN
-F 3 "http://www.ti.com/lit/sg/scyt129e/scyt129e.pdf" H 2490 4600 50  0001 C CNN
-F 4 "296-11934-1-ND" H 2390 4450 50  0001 C CNN "Digi-Key PN"
-	1    2390 4450
-	-1   0    0    -1
-$EndComp
-$Comp
-L power:GND #PWR0608
-U 1 1 5BBB82D1
-P 2390 4550
-F 0 "#PWR0608" H 2390 4300 50  0001 C CNN
-F 1 "GND" H 2390 4400 50  0000 C CNN
-F 2 "" H 2390 4550 50  0001 C CNN
-F 3 "" H 2390 4550 50  0001 C CNN
-	1    2390 4550
-	1    0    0    -1
-$EndComp
-$Comp
-L Custom_Library:+3.3V #PWR0607
-U 1 1 5BBB8333
-P 2390 4350
-F 0 "#PWR0607" H 2390 4200 50  0001 C CNN
-F 1 "+3.3V" H 2390 4490 50  0000 C CNN
-F 2 "" H 2390 4350 50  0000 C CNN
-F 3 "" H 2390 4350 50  0000 C CNN
-	1    2390 4350
-	1    0    0    -1
-$EndComp
-$Comp
-L Custom_Library:C_Custom C602
-U 1 1 5BBB8788
-P 2190 5150
-F 0 "C602" H 2215 5250 50  0000 L CNN
-F 1 "0.1uF" H 2215 5050 50  0000 L CNN
-F 2 "Capacitors_SMD:C_0603" H 2228 5000 50  0001 C CNN
-F 3 "" H 2215 5250 50  0001 C CNN
-F 4 "0603" H 2040 5250 50  0000 R CNN "display_footprint"
-F 5 "50V" H 2040 5150 50  0000 R CNN "Voltage"
-F 6 "X7R" H 2040 5050 50  0000 R CNN "Dielectric"
-F 7 "490-8020-1-ND" H 2615 5650 60  0001 C CNN "Digi-Key PN"
-	1    2190 5150
-	1    0    0    -1
-$EndComp
-$Comp
-L power:GND #PWR0605
-U 1 1 5BBB8855
-P 2190 5300
-F 0 "#PWR0605" H 2190 5050 50  0001 C CNN
-F 1 "GND" H 2190 5150 50  0000 C CNN
-F 2 "" H 2190 5300 50  0001 C CNN
-F 3 "" H 2190 5300 50  0001 C CNN
-	1    2190 5300
-	1    0    0    -1
-$EndComp
-$Comp
-L Custom_Library:+3.3V #PWR0604
-U 1 1 5BBB88AC
-P 2190 5000
-F 0 "#PWR0604" H 2190 4850 50  0001 C CNN
-F 1 "+3.3V" H 2190 5140 50  0000 C CNN
-F 2 "" H 2190 5000 50  0000 C CNN
-F 3 "" H 2190 5000 50  0000 C CNN
-	1    2190 5000
-	1    0    0    -1
-$EndComp
-Wire Wire Line
-	2690 4450 2950 4450
-$Comp
-L Custom_Library:R_Custom R?
-U 1 1 5BBBB118
-P 1490 4830
-AR Path="/5BB27BA3/5BBBB118" Ref="R?"  Part="1"
-AR Path="/5BB27B51/5BBBB118" Ref="R?"  Part="1"
-AR Path="/5BB7FA89/5BBBB118" Ref="R?"  Part="1"
-AR Path="/5BB27B73/5BBBB118" Ref="R601"  Part="1"
-F 0 "R601" H 1410 4830 50  0000 R CNN
-F 1 "10k" V 1490 4830 50  0000 C CNN
-F 2 "Resistors_SMD:R_0603" H 1490 4830 50  0001 C CNN
-F 3 "" H 1490 4830 50  0001 C CNN
-F 4 "0603" H 1590 4910 50  0000 L CNN "display_footprint"
-F 5 "1%" H 1590 4830 50  0000 L CNN "Tolerance"
-F 6 "1/10W" H 1600 4750 50  0000 L CNN "Wattage"
-F 7 "RHM10KADCT-ND" H 1790 5230 60  0001 C CNN "Digi-Key PN"
-	1    1490 4830
-	1    0    0    -1
-$EndComp
-$Comp
-L power:GND #PWR0601
-U 1 1 5BBBB16E
-P 1490 4980
-F 0 "#PWR0601" H 1490 4730 50  0001 C CNN
-F 1 "GND" H 1490 4830 50  0000 C CNN
-F 2 "" H 1490 4980 50  0001 C CNN
-F 3 "" H 1490 4980 50  0001 C CNN
-	1    1490 4980
-	1    0    0    -1
-$EndComp
-Wire Wire Line
-	2140 4450 1490 4450
-Wire Wire Line
-	1490 4450 1490 4680
-Wire Wire Line
-	1410 4450 1490 4450
-Connection ~ 1490 4450
 Text Notes 540  690  0    100  ~ 20
 +3.3V, 750mA, 2MHz Buck Converter
@@
 Wire Wire Line
 	2740 6650 2740 6760
+NoConn ~ 3960 4450
 $EndSCHEMATC
