File: hdw/AC_Power_Meter/Pushbuttons.sch (KiCad schematic (older format))
At the start: 17 parts

Commit message: Rewired a few micro symbols, add FMW notes
Parts:
- added J1701: Ext_SW_Toggle, symbol Connector_Generic:Conn_02x01
- added SW1701: Ext_SW_Toggle, symbol Switch:SW_Push
- SW1703: renamed from SW?; value SLEEP -> SW_Toggle
- gave numbers to parts that had none: 16
Connections:
- net labels added: SW_Toggle
- net labels removed: Sleep
- wire segments 29 -> 31
- no-connect marks 0 -> 2

Commit message: Updated most footprints
Parts:
- C1701, C1702: footprint (none) -> Capacitors_SMD:C_0603; Digi-Key PN PN -> 1276-1921-1-ND
- C1703, C1704: footprint (none) -> Capacitors_SMD:C_0603; Digi-Key PN PN -> 490-8020-1-ND
- C1705, C1706: footprint (none) -> Capacitors_SMD:C_0805; Digi-Key PN PN -> 490-1695-1-ND
- Q1701: Digi-Key PN (none) -> 2N7002NCT-ND
- R1701, R1702, R1705: footprint (none) -> Resistors_SMD:R_0603; Digi-Key PN PN -> RHM10KADCT-ND
- R1703, R1704: footprint (none) -> Resistors_SMD:R_0603; Digi-Key PN PN -> P100KHCT-ND
- R1706: footprint (none) -> Resistors_SMD:R_0603; Digi-Key PN PN -> 311-220HRCT-ND
- SW1701: Digi-Key PN (none) -> EG2015-ND
- SW1702, SW1703: footprint (none) -> Buttons_Switches_THT:SW_PUSH_6mm
- U1701, U1702: footprint (none) -> Housings_SOIC:SO-8_5.3x6.2mm_Pitch1.27mm; Digi-Key PN (none) -> 296-34367-5-ND
Changed lines of the file:
@@
 F 0 "U1701" H 4150 3130 50  0000 L CNN
 F 1 "TLC555CPS" H 4650 3130 50  0000 L CNN
-F 2 "" H 4550 2780 50  0001 C CNN
+F 2 "Housings_SOIC:SO-8_5.3x6.2mm_Pitch1.27mm" H 4550 2780 50  0001 C CNN
 F 3 "http://www.ti.com/lit/ds/symlink/tlc555.pdf" H 4550 2780 50  0001 C CNN
+F 4 "296-34367-5-ND" H 0   0   50  0001 C CNN "Digi-Key PN"
 	1    4550 2780
 	1    0    0    -1
@@
 F 0 "SW1702" H 3180 3210 50  0000 L CNN
 F 1 "MRESET" H 3130 3050 50  0000 C CNN
-F 2 "" H 3130 3310 50  0001 C CNN
+F 2 "Buttons_Switches_THT:SW_PUSH_6mm" H 3130 3310 50  0001 C CNN
 F 3 "" H 3130 3310 50  0001 C CNN
 	1    3130 3110
@@
 F 0 "R1705" H 6060 2810 50  0000 R CNN
 F 1 "10k" V 6140 2810 50  0000 C CNN
-F 2 "" H 6140 2810 50  0001 C CNN
+F 2 "Resistors_SMD:R_0603" H 6140 2810 50  0001 C CNN
 F 3 "" H 6140 2810 50  0001 C CNN
 F 4 "0603" H 6240 2890 50  0000 L CNN "display_footprint"
 F 5 "1%" H 6240 2810 50  0000 L CNN "Tolerance"
 F 6 "1/10W" H 6250 2730 50  0000 L CNN "Wattage"
-F 7 "PN" H 6440 3210 60  0001 C CNN "Digi-Key PN"
+F 7 "RHM10KADCT-ND" H 6440 3210 60  0001 C CNN "Digi-Key PN"
 	1    6140 2810
 	1    0    0    -1
@@
 F 2 "Package_TO_SOT_SMD:SOT-23" H 7360 2505 50  0001 L CIN
 F 3 "https://www.fairchildsemi.com/datasheets/2N/2N7002.pdf" H 7160 2580 50  0001 L CNN
+F 4 "2N7002NCT-ND" H 0   0   50  0001 C CNN "Digi-Key PN"
 	1    7160 2580
 	1    0    0    -1
@@
 F 0 "R1706" V 6660 2580 50  0000 C CNN
 F 1 "220" V 6760 2580 50  0000 C CNN
-F 2 "" H 6760 2580 50  0001 C CNN
+F 2 "Resistors_SMD:R_0603" H 6760 2580 50  0001 C CNN
 F 3 "" H 6760 2580 50  0001 C CNN
 F 4 "0603" V 6860 2580 50  0000 C CNN "display_footprint"
 F 5 "1%" V 6960 2580 50  0000 C CNN "Tolerance"
 F 6 "1/10W" V 7060 2580 50  0000 C CNN "Wattage"
-F 7 "PN" H 7060 2980 60  0001 C CNN "Digi-Key PN"
+F 7 "311-220HRCT-ND" H 7060 2980 60  0001 C CNN "Digi-Key PN"
 	1    6760 2580
 	0    1    1    0
@@
 F 0 "R1703" H 5300 2170 50  0000 R CNN
 F 1 "100k" V 5380 2170 40  0000 C CNN
-F 2 "" H 5380 2170 50  0001 C CNN
+F 2 "Resistors_SMD:R_0603" H 5380 2170 50  0001 C CNN
 F 3 "" H 5380 2170 50  0001 C CNN
 F 4 "0603" H 5480 2250 50  0000 L CNN "display_footprint"
 F 5 "1%" H 5480 2170 50  0000 L CNN "Tolerance"
 F 6 "1/10W" H 5490 2090 50  0000 L CNN "Wattage"
-F 7 "PN" H 5680 2570 60  0001 C CNN "Digi-Key PN"
+F 7 "P100KHCT-ND" H 5680 2570 60  0001 C CNN "Digi-Key PN"
 	1    5380 2170
 	1    0    0    -1
@@
 F 0 "C1703" H 4235 3830 50  0000 L CNN
 F 1 "0.1uF" H 4235 3630 50  0000 L CNN
-F 2 "" H 4248 3580 50  0001 C CNN
+F 2 "Capacitors_SMD:C_0603" H 4248 3580 50  0001 C CNN
 F 3 "" H 4235 3830 50  0001 C CNN
 F 4 "0603" H 4060 3830 50  0000 R CNN "display_footprint"
 F 5 "50V" H 4060 3730 50  0000 R CNN "Voltage"
 F 6 "X7R" H 4060 3630 50  0000 R CNN "Dielectric"
-F 7 "PN" H 4635 4230 60  0001 C CNN "Digi-Key PN"
+F 7 "490-8020-1-ND" H 4635 4230 60  0001 C CNN "Digi-Key PN"
 	1    4210 3730
 	1    0    0    -1
@@
 F 0 "C1705" H 5405 3290 50  0000 L CNN
 F 1 "1uF" H 5405 3090 50  0000 L CNN
-F 2 "" H 5418 3040 50  0001 C CNN
+F 2 "Capacitors_SMD:C_0805" H 5418 3040 50  0001 C CNN
 F 3 "" H 5405 3290 50  0001 C CNN
 F 4 "0805" H 5230 3290 50  0000 R CNN "display_footprint"
 F 5 "10V" H 5230 3190 50  0000 R CNN "Voltage"
 F 6 "X7R" H 5230 3090 50  0000 R CNN "Dielectric"
-F 7 "PN" H 5805 3690 60  0001 C CNN "Digi-Key PN"
+F 7 "490-1695-1-ND" H 5805 3690 60  0001 C CNN "Digi-Key PN"
 	1    5380 3190
 	1    0    0    -1
@@
 F 0 "C1701" H 3775 3210 50  0000 L CNN
 F 1 "10nF" H 3775 3010 50  0000 L CNN
-F 2 "" H 3788 2960 50  0001 C CNN
+F 2 "Capacitors_SMD:C_0603" H 3788 2960 50  0001 C CNN
 F 3 "" H 3775 3210 50  0001 C CNN
 F 4 "0603" H 3600 3210 50  0000 R CNN "display_footprint"
 F 5 "50V" H 3600 3110 50  0000 R CNN "Voltage"
 F 6 "X7R" H 3600 3010 50  0000 R CNN "Dielectric"
-F 7 "PN" H 4175 3610 60  0001 C CNN "Digi-Key PN"
+F 7 "1276-1921-1-ND" H 4175 3610 60  0001 C CNN "Digi-Key PN"
 	1    3750 3110
 	1    0    0    -1
@@
 F 0 "R1701" H 3050 2330 50  0000 R CNN
 F 1 "10k" V 3130 2330 50  0000 C CNN
-F 2 "" H 3130 2330 50  0001 C CNN
+F 2 "Resistors_SMD:R_0603" H 3130 2330 50  0001 C CNN
 F 3 "" H 3130 2330 50  0001 C CNN
 F 4 "0603" H 3230 2410 50  0000 L CNN "display_footprint"
 F 5 "1%" H 3230 2330 50  0000 L CNN "Tolerance"
 F 6 "1/10W" H 3240 2250 50  0000 L CNN "Wattage"
-F 7 "PN" H 3430 2730 60  0001 C CNN "Digi-Key PN"
+F 7 "RHM10KADCT-ND" H 3430 2730 60  0001 C CNN "Digi-Key PN"
 	1    3130 2330
 	1    0    0    -1
@@
 F 0 "U1702" H 4150 5710 50  0000 L CNN
 F 1 "TLC555CPS" H 4650 5710 50  0000 L CNN
-F 2 "" H 4550 5360 50  0001 C CNN
+F 2 "Housings_SOIC:SO-8_5.3x6.2mm_Pitch1.27mm" H 4550 5360 50  0001 C CNN
 F 3 "http://www.ti.com/lit/ds/symlink/tlc555.pdf" H 4550 5360 50  0001 C CNN
+F 4 "296-34367-5-ND" H 0   0   50  0001 C CNN "Digi-Key PN"
 	1    4550 5360
 	1    0    0    -1
@@
 F 0 "SW1703" H 3180 5790 50  0000 L CNN
 F 1 "SW_Toggle" H 3130 5630 50  0000 C CNN
-F 2 "" H 3130 5890 50  0001 C CNN
+F 2 "Buttons_Switches_THT:SW_PUSH_6mm" H 3130 5890 50  0001 C CNN
 F 3 "" H 3130 5890 50  0001 C CNN
 	1    3130 5690
@@
 F 0 "R1704" H 5300 4750 50  0000 R CNN
 F 1 "100k" V 5380 4750 40  0000 C CNN
-F 2 "" H 5380 4750 50  0001 C CNN
+F 2 "Resistors_SMD:R_0603" H 5380 4750 50  0001 C CNN
 F 3 "" H 5380 4750 50  0001 C CNN
 F 4 "0603" H 5480 4830 50  0000 L CNN "display_footprint"
 F 5 "1%" H 5480 4750 50  0000 L CNN "Tolerance"
 F 6 "1/10W" H 5490 4670 50  0000 L CNN "Wattage"
-F 7 "PN" H 5680 5150 60  0001 C CNN "Digi-Key PN"
+F 7 "P100KHCT-ND" H 5680 5150 60  0001 C CNN "Digi-Key PN"
 	1    5380 4750
 	1    0    0    -1
@@
 F 0 "C1704" H 4235 6410 50  0000 L CNN
 F 1 "0.1uF" H 4235 6210 50  0000 L CNN
-F 2 "" H 4248 6160 50  0001 C CNN
+F 2 "Capacitors_SMD:C_0603" H 4248 6160 50  0001 C CNN
 F 3 "" H 4235 6410 50  0001 C CNN
 F 4 "0603" H 4060 6410 50  0000 R CNN "display_footprint"
 F 5 "50V" H 4060 6310 50  0000 R CNN "Voltage"
 F 6 "X7R" H 4060 6210 50  0000 R CNN "Dielectric"
-F 7 "PN" H 4635 6810 60  0001 C CNN "Digi-Key PN"
+F 7 "490-8020-1-ND" H 4635 6810 60  0001 C CNN "Digi-Key PN"
 	1    4210 6310
 	1    0    0    -1
@@
 F 0 "C1706" H 5405 5870 50  0000 L CNN
 F 1 "1uF" H 5405 5670 50  0000 L CNN
-F 2 "" H 5418 5620 50  0001 C CNN
+F 2 "Capacitors_SMD:C_0805" H 5418 5620 50  0001 C CNN
 F 3 "" H 5405 5870 50  0001 C CNN
 F 4 "0805" H 5230 5870 50  0000 R CNN "display_footprint"
 F 5 "10V" H 5230 5770 50  0000 R CNN "Voltage"
 F 6 "X7R" H 5230 5670 50  0000 R CNN "Dielectric"
-F 7 "PN" H 5805 6270 60  0001 C CNN "Digi-Key PN"
+F 7 "490-1695-1-ND" H 5805 6270 60  0001 C CNN "Digi-Key PN"
 	1    5380 5770
 	1    0    0    -1
@@
 F 0 "C1702" H 3775 5790 50  0000 L CNN
 F 1 "10nF" H 3775 5590 50  0000 L CNN
-F 2 "" H 3788 5540 50  0001 C CNN
+F 2 "Capacitors_SMD:C_0603" H 3788 5540 50  0001 C CNN
 F 3 "" H 3775 5790 50  0001 C CNN
 F 4 "0603" H 3600 5790 50  0000 R CNN "display_footprint"
 F 5 "50V" H 3600 5690 50  0000 R CNN "Voltage"
 F 6 "X7R" H 3600 5590 50  0000 R CNN "Dielectric"
-F 7 "PN" H 4175 6190 60  0001 C CNN "Digi-Key PN"
+F 7 "1276-1921-1-ND" H 4175 6190 60  0001 C CNN "Digi-Key PN"
 	1    3750 5690
 	1    0    0    -1
@@
 F 0 "R1702" H 3050 4910 50  0000 R CNN
 F 1 "10k" V 3130 4910 50  0000 C CNN
-F 2 "" H 3130 4910 50  0001 C CNN
+F 2 "Resistors_SMD:R_0603" H 3130 4910 50  0001 C CNN
 F 3 "" H 3130 4910 50  0001 C CNN
 F 4 "0603" H 3230 4990 50  0000 L CNN "display_footprint"
 F 5 "1%" H 3230 4910 50  0000 L CNN "Tolerance"
 F 6 "1/10W" H 3240 4830 50  0000 L CNN "Wattage"
-F 7 "PN" H 3430 5310 60  0001 C CNN "Digi-Key PN"
+F 7 "RHM10KADCT-ND" H 3430 5310 60  0001 C CNN "Digi-Key PN"
 	1    3130 4910
 	1    0    0    -1
@@
 F 2 "" H 2060 5890 50  0001 C CNN
 F 3 "" H 2060 5890 50  0001 C CNN
+F 4 "EG2015-ND" H 2060 5690 50  0001 C CNN "Digi-Key PN"
 	1    2060 5690
 	0    -1   -1   0

Commit message: Arranged a few pages of components
Parts:
- J1701: footprint (none) -> Pin_Headers:Pin_Header_Straight_1x02_Pitch2.54mm
Changed lines of the file:
@@
 F 0 "J1701" H 2550 5810 50  0000 C CNN
 F 1 "Ext_SW_Toggle" H 2550 5610 50  0000 C CNN
-F 2 "" H 2500 5710 50  0001 C CNN
+F 2 "Pin_Headers:Pin_Header_Straight_1x02_Pitch2.54mm" H 2500 5710 50  0001 C CNN
 F 3 "~" H 2500 5710 50  0001 C CNN
 	1    2500 5710

Commit message: Nailed down board outline, placed a few sections
Parts:
- Q1701: footprint Package_TO_SOT_SMD:SOT-23 -> TO_SOT_Packages_SMD:SOT-23
Changed lines of the file:
@@
 F 0 "Q1701" H 7360 2655 50  0000 L CNN
 F 1 "2N7002" H 7360 2580 50  0000 L CNN
-F 2 "Package_TO_SOT_SMD:SOT-23" H 7360 2505 50  0001 L CIN
+F 2 "TO_SOT_Packages_SMD:SOT-23" H 7360 2505 50  0001 L CIN
 F 3 "https://www.fairchildsemi.com/datasheets/2N/2N7002.pdf" H 7160 2580 50  0001 L CNN
 F 4 "2N7002NCT-ND" H 0   0   50  0001 C CNN "Digi-Key PN"

Commit message: Placed a lot more parts, netlist cleanup
Other:
- moved on the sheet: Q1701
Changed lines of the file:
@@
 L Custom_Library:R_Custom R?
 U 1 1 5BC28346
-P 6140 2810
+P 6910 2810
 AR Path="/5BB27BA3/5BC28346" Ref="R?"  Part="1"
 AR Path="/5BC25FFE/5BC28346" Ref="R1705"  Part="1"
-F 0 "R1705" H 6060 2810 50  0000 R CNN
-F 1 "10k" V 6140 2810 50  0000 C CNN
-F 2 "Resistors_SMD:R_0603" H 6140 2810 50  0001 C CNN
-F 3 "" H 6140 2810 50  0001 C CNN
-F 4 "0603" H 6240 2890 50  0000 L CNN "display_footprint"
-F 5 "1%" H 6240 2810 50  0000 L CNN "Tolerance"
-F 6 "1/10W" H 6250 2730 50  0000 L CNN "Wattage"
-F 7 "RHM10KADCT-ND" H 6440 3210 60  0001 C CNN "Digi-Key PN"
-	1    6140 2810
-	1    0    0    -1
-$EndComp
-Wire Wire Line
-	6140 2660 6140 2580
+F 0 "R1705" H 6830 2810 50  0000 R CNN
+F 1 "10k" V 6910 2810 50  0000 C CNN
+F 2 "Resistors_SMD:R_0603" H 6910 2810 50  0001 C CNN
+F 3 "" H 6910 2810 50  0001 C CNN
+F 4 "0603" H 7010 2890 50  0000 L CNN "display_footprint"
+F 5 "1%" H 7010 2810 50  0000 L CNN "Tolerance"
+F 6 "1/10W" H 7020 2730 50  0000 L CNN "Wattage"
+F 7 "RHM10KADCT-ND" H 7210 3210 60  0001 C CNN "Digi-Key PN"
+	1    6910 2810
+	1    0    0    -1
+$EndComp
+Wire Wire Line
+	6910 2660 6910 2580
 $Comp
 L power:GND #PWR?
 U 1 1 5BC2834E
-P 6140 2960
+P 6910 2960
 AR Path="/5BB27BA3/5BC2834E" Ref="#PWR?"  Part="1"
 AR Path="/5BC25FFE/5BC2834E" Ref="#PWR01722"  Part="1"
-F 0 "#PWR01722" H 6140 2710 50  0001 C CNN
-F 1 "GND" H 6140 2810 50  0000 C CNN
-F 2 "" H 6140 2960 50  0001 C CNN
-F 3 "" H 6140 2960 50  0001 C CNN
-	1    6140 2960
+F 0 "#PWR01722" H 6910 2710 50  0001 C CNN
+F 1 "GND" H 6910 2810 50  0000 C CNN
+F 2 "" H 6910 2960 50  0001 C CNN
+F 3 "" H 6910 2960 50  0001 C CNN
+	1    6910 2960
 	1    0    0    -1
 $EndComp
@@
 L Transistor_FET:2N7002 Q?
 U 1 1 5BC28354
-P 7160 2580
+P 7640 2580
 AR Path="/5BB27BA3/5BC28354" Ref="Q?"  Part="1"
 AR Path="/5BC25FFE/5BC28354" Ref="Q1701"  Part="1"
-F 0 "Q1701" H 7360 2655 50  0000 L CNN
-F 1 "2N7002" H 7360 2580 50  0000 L CNN
-F 2 "TO_SOT_Packages_SMD:SOT-23" H 7360 2505 50  0001 L CIN
-F 3 "https://www.fairchildsemi.com/datasheets/2N/2N7002.pdf" H 7160 2580 50  0001 L CNN
-F 4 "2N7002NCT-ND" H 0   0   50  0001 C CNN "Digi-Key PN"
-	1    7160 2580
-	1    0    0    -1
-$EndComp
-Text GLabel 7260 2380 1    60   UnSpc ~ 0
+F 0 "Q1701" H 7840 2655 50  0000 L CNN
+F 1 "2N7002" H 7840 2580 50  0000 L CNN
+F 2 "TO_SOT_Packages_SMD:SOT-23" H 7840 2505 50  0001 L CIN
+F 3 "https://www.fairchildsemi.com/datasheets/2N/2N7002.pdf" H 7640 2580 50  0001 L CNN
+F 4 "2N7002NCT-ND" H 480 0   50  0001 C CNN "Digi-Key PN"
+	1    7640 2580
+	1    0    0    -1
+$EndComp
+Text GLabel 7740 2380 1    60   UnSpc ~ 0
 ~MCLR
 $Comp
 L power:GND #PWR?
 U 1 1 5BC2835C
-P 7260 2780
+P 7740 2780
 AR Path="/5BB27BA3/5BC2835C" Ref="#PWR?"  Part="1"
 AR Path="/5BC25FFE/5BC2835C" Ref="#PWR01723"  Part="1"
-F 0 "#PWR01723" H 7260 2530 50  0001 C CNN
-F 1 "GND" H 7260 2630 50  0000 C CNN
-F 2 "" H 7260 2780 50  0001 C CNN
-F 3 "" H 7260 2780 50  0001 C CNN
-	1    7260 2780
+F 0 "#PWR01723" H 7740 2530 50  0001 C CNN
+F 1 "GND" H 7740 2630 50  0000 C CNN
+F 2 "" H 7740 2780 50  0001 C CNN
+F 3 "" H 7740 2780 50  0001 C CNN
+	1    7740 2780
 	-1   0    0    -1
 $EndComp
@@
 L Custom_Library:R_Custom R?
 U 1 1 5BC28366
-P 6760 2580
+P 6200 2580
 AR Path="/5BB31314/5BC28366" Ref="R?"  Part="1"
 AR Path="/5BB27BA3/5BC28366" Ref="R?"  Part="1"
 AR Path="/5BC25FFE/5BC28366" Ref="R1706"  Part="1"
-F 0 "R1706" V 6660 2580 50  0000 C CNN
-F 1 "220" V 6760 2580 50  0000 C CNN
-F 2 "Resistors_SMD:R_0603" H 6760 2580 50  0001 C CNN
-F 3 "" H 6760 2580 50  0001 C CNN
-F 4 "0603" V 6860 2580 50  0000 C CNN "display_footprint"
-F 5 "1%" V 6960 2580 50  0000 C CNN "Tolerance"
-F 6 "1/10W" V 7060 2580 50  0000 C CNN "Wattage"
-F 7 "311-220HRCT-ND" H 7060 2980 60  0001 C CNN "Digi-Key PN"
-	1    6760 2580
+F 0 "R1706" V 6100 2580 50  0000 C CNN
+F 1 "220" V 6200 2580 50  0000 C CNN
+F 2 "Resistors_SMD:R_0603" H 6200 2580 50  0001 C CNN
+F 3 "" H 6200 2580 50  0001 C CNN
+F 4 "0603" V 6300 2580 50  0000 C CNN "display_footprint"
+F 5 "1%" V 6400 2580 50  0000 C CNN "Tolerance"
+F 6 "1/10W" V 6500 2580 50  0000 C CNN "Wattage"
+F 7 "311-220HRCT-ND" H 6500 2980 60  0001 C CNN "Digi-Key PN"
+	1    6200 2580
 	0    1    1    0
 $EndComp
 Wire Wire Line
-	6610 2580 6140 2580
-Wire Wire Line
-	6910 2580 6960 2580
+	6910 2580 7440 2580
 $Comp
 L Custom_Library:R_Custom R?
@@
 Wire Wire Line
 	3990 2980 4050 2980
-Wire Wire Line
-	6140 2580 5050 2580
-Connection ~ 6140 2580
 $Comp
 L Timer:TLC555CPS U1702
@@
 NoConn ~ 2060 5890
 NoConn ~ 2060 5490
+Wire Wire Line
+	6350 2580 6910 2580
+Connection ~ 6910 2580
+Wire Wire Line
+	6050 2580 5050 2580
 $EndSCHEMATC

Commit message: A few routing adjustments and more graphics added to PCB
Parts:
- removed C1701: 10nF, Capacitors_SMD:C_0603, symbol Custom_Library:C_Custom
- removed C1703: 0.1uF, Capacitors_SMD:C_0603, symbol Custom_Library:C_Custom
- removed C1705: 1uF, Capacitors_SMD:C_0805, symbol Custom_Library:C_Custom
- removed Q1701: 2N7002, TO_SOT_Packages_SMD:SOT-23, symbol Transistor_FET:2N7002
- removed R1701, R1705: 10k, Resistors_SMD:R_0603, symbol Custom_Library:R_Custom
- removed R1703: 100k, Resistors_SMD:R_0603, symbol Custom_Library:R_Custom
- removed R1706: 220, Resistors_SMD:R_0603, symbol Custom_Library:R_Custom
- removed U1701: TLC555CPS, Housings_SOIC:SO-8_5.3x6.2mm_Pitch1.27mm, symbol Timer:TLC555CPS
Connections:
- net labels added: ~MRST
- net labels removed: ~MCLR
- wire segments 31 -> 17

Commit message: Serious BOM scrubbing to drive price down
Parts:
- removed C1702: 10nF, Capacitors_SMD:C_0603, symbol Custom_Library:C_Custom
- removed C1704: 0.1uF, Capacitors_SMD:C_0603, symbol Custom_Library:C_Custom
- removed C1706: 1uF, Capacitors_SMD:C_0805, symbol Custom_Library:C_Custom
- removed J1701: Ext_SW_Toggle, Pin_Headers:Pin_Header_Straight_1x02_Pitch2.54mm, symbol Connector_Generic:Conn_02x01
- removed R1702: 10k, Resistors_SMD:R_0603, symbol Custom_Library:R_Custom
- removed R1704: 100k, Resistors_SMD:R_0603, symbol Custom_Library:R_Custom
- removed SW1701: Ext_SW_Toggle, symbol Switch:SW_Push
- removed SW1702: MRESET, Buttons_Switches_THT:SW_PUSH_6mm, symbol Switch:SW_Push
- removed SW1703: SW_Toggle, Buttons_Switches_THT:SW_PUSH_6mm, symbol Switch:SW_Push
- removed U1702: TLC555CPS, Housings_SOIC:SO-8_5.3x6.2mm_Pitch1.27mm, symbol Timer:TLC555CPS
Connections:
- net labels removed: +3.3V, GND, SW_Toggle, ~MRST
- wire segments 17 -> 0
- no-connect marks 2 -> 0
