File: hdw/AC_Power_Meter/Status_LEDs.sch (KiCad schematic (older format))
At the start: 35 parts

Commit message: Added MU logo and titles to all sheets
Other:
- note added: "Status LEDs"

Commit message: Updated MU logo to crisper image
Changed lines of the file:
@@
 Status LEDs
 $Comp
-L Mu_Logo:LOGO #G?
-U 1 1 5BBF9A41
-P 9900 1000
-F 0 "#G?" H 9900 670 60  0001 C CNN
-F 1 "LOGO" H 9900 1330 60  0001 C CNN
-F 2 "" H 9900 1000 50  0001 C CNN
-F 3 "" H 9900 1000 50  0001 C CNN
-	1    9900 1000
+L Custom_Library:MU_Logo #G?
+U 1 1 5BB6AE86
+P 9900 1100
+F 0 "#G?" H 9900 614 60  0001 C CNN
+F 1 "MU_Logo" H 9900 1586 60  0001 C CNN
+F 2 "" H 9900 1100 50  0001 C CNN
+F 3 "" H 9900 1100 50  0001 C CNN
+	1    9900 1100
 	1    0    0    -1
 $EndComp

Commit message: Added pushbuttons sheet, prelim wiring on micro
Connections:
- net labels added: Active
- net labels removed: ~Reset
Changed lines of the file:
@@
 $Descr A 11000 8500
 encoding utf-8
-Sheet 16 16
+Sheet 16 17
 Title ""
 Date ""
@@
 $EndComp
 Text GLabel 1350 3140 0    50   Input ~ 0
-~Reset
+Active
 $Comp
 L Custom_Library:74LVC1G06_Power U?

Commit message: Rewired a few micro symbols, add FMW notes
Parts:
- gave numbers to parts that had none: 35
Connections:
- net labels added: ~Active
- net labels removed: Active

Commit message: Updated most footprints
Parts:
- C1601, C1602, C1603, C1604, C1605, C1606, C1607: footprint (none) -> Capacitors_SMD:C_0603; Digi-Key PN PN -> 490-8020-1-ND
- D1601, D1603, D1605: footprint (none) -> LEDs:LED_0603; Digi-Key PN PN -> 160-1447-1-ND
- D1602, D1604, D1606, D1607: footprint (none) -> LEDs:LED_0603; Digi-Key PN PN -> 160-1446-1-ND
- R1601, R1602, R1605, R1606, R1609, R1610, R1613: footprint (none) -> Resistors_SMD:R_0603; Digi-Key PN PN -> RHM10KADCT-ND
- R1603, R1604, R1607, R1608, R1611, R1612, R1614: footprint (none) -> Resistors_SMD:R_0603; Digi-Key PN PN -> MCT0603-1.00K-CFCT-ND

Commit message: Serious BOM scrubbing to drive price down
Parts:
- removed C1601, C1602, C1603, C1604, C1605, C1606, C1607: 0.1uF, Capacitors_SMD:C_0603, symbol Custom_Library:C_Custom
- removed D1603: Red, LEDs:LED_0603, symbol Custom_Library:LED_ALT_Custom
- removed D1606, D1607: Green, LEDs:LED_0603, symbol Custom_Library:LED_ALT_Custom
- removed R1605, R1610, R1613: 10k, Resistors_SMD:R_0603, symbol Custom_Library:R_Custom
- removed R1607, R1612, R1614: 1k, Resistors_SMD:R_0603, symbol Custom_Library:R_Custom
- removed U1601, U1602, U1603, U1604, U1605, U1606, U1607: 74LVC1G06, TO_SOT_Packages_SMD:SOT-353_SC-70-5, symbol Custom_Library:74LVC1G06_Power
- added Q1401, Q1402, Q1403, Q1404: 2N7002, TO_SOT_Packages_SMD:SOT-23, symbol Transistor_FET:2N7002
- added R1405, R1406, R1407, R1408: 10, Resistors_SMD:R_0603, symbol Custom_Library:R_Custom
Connections:
- net labels removed: ICSP_DETECT, POS12_PGOOD, POS3P3_PGOOD
- wire segments 42 -> 24
